Commit message: Fixed connections to files that moved to other folders

File: mir/mir_description/urdf/mir.urdf.xacro (robot description, xacro)
@@ -3,8 +3,8 @@
        name="mir_100" >
   <!-- MiR100 base -->
-  <xacro:include filename="$(find mir_description)/urdf/include/mir100.urdf.xacro" />
-  <xacro:include filename="$(find mir_description)/urdf/include/common.gazebo.xacro" />
-  <xacro:mir_100 prefix=""/>
-  <xacro:controller_plugin_gazebo robot_namespace=""/>
+  <xacro:include filename="$(find mir_description)/urdf/mir_100/mir_100.urdf.xacro" />
+  <xacro:include filename="$(find mir_description)/urdf/mir_100/mir_100.gazebo.xacro" />
+  <xacro:mir_100 tf_prefix=""/>
+  <!-- <xacro:controller_plugin_gazebo robot_namespace=""/> -->
   <!-- instead of the controller_plugin_gazebo, you can use the diffdrive controller like this:
     <xacro:diff_controller_plugin_gazebo prefix=""

File: mir/mir_description/urdf/mir_100/mir_100.gazebo.xacro (robot description, xacro)
@@ -6,10 +6,10 @@
 	<xacro:macro name="mir_100_gazebo" params="tf_prefix">
 		<!-- Set Gazebo material for the base -->
-		<gazebo reference="${prefix}base_link">
+		<gazebo reference="${tf_prefix}base_link">
 			<material>Gazebo/White</material>
 		</gazebo>
 		<!-- Settings for the IMU of the robot to work in the simulation environment-->
 		<xacro:imu_gazebo link="${tf_prefix}imu_link" imu_topic="imu_data" update_rate="50.0" standard_deviation="${imu_standard_deviation}" />
-		<p3d_base_controller prefix="${prefix}" />
+		<p3d_base_controller prefix="${tf_prefix}" />
 		<!-- wheels -->
 		<xacro:actuated_wheel_gazebo tf_prefix="${tf_prefix}" locationprefix="left"/>
@@ -49,5 +49,5 @@
 					<rosDebugLevel>Debug</rosDebugLevel>
 				</plugin>
-			</gazebo>
-		</xacro:macro> -->
+			</gazebo-->
+	</xacro:macro>
 </robot>

File: mir/mir_description/urdf/mir_100/mir_100.urdf.xacro (robot description, xacro)
@@ -1,7 +1,7 @@
 <?xml version="1.0"?>
 <robot xmlns:xacro="http://ros.org/wiki/xacro">
-	<xacro:include filename="$(find mir_description)/urdf/include/common_properties.urdf.xacro" />
+	<xacro:include filename="$(find mir_description)/urdf/general/common_properties.urdf.xacro" />
 	<xacro:include filename="$(find mir_description)/urdf/mir_100/mir_100_wheels.urdf.xacro" />
-	<xacro:include filename="$(find mir_description)/urdf/include/sick_s300.urdf.xacro" />
+	<xacro:include filename="$(find mir_description)/urdf/general/sick_s300.urdf.xacro" />
 	<xacro:property name="deg_to_rad" value="${(1 / 360) * (2 * pi)}" />
 	<xacro:property name="mir_100_base_mass" value="58.0" />
