Commit message: Added Sick s300 Gazebo to MiR200 gazebo xacro

File: mir/mir_description/urdf/mir_200/mir_200.gazebo.xacro (robot description, xacro)
@@ -44,4 +44,8 @@
 		<!-- -->
 		<p3d_base_controller tf_prefix="${tf_prefix}" />
+		<!-- Add Gazebo xacro for the laser scanner to work in Gazebo-->
+		<!-- Please match there macro calls with the sick_s300 xacro calls in the mir_200.urdf.xacro file-->
+		<xacro:macro name="sick_s300_gazebo" link="front_laser_link" topic="f_scan" tf_prefix="${tf_prefix}"/>
+		<xacro:macro name="sick_s300_gazebo" link="back_laser_link" topic="b_scan" tf_prefix="${tf_prefix}"/>
 		<!-- disabled, because it doesn't make a difference in Gazebo: -->
 		<!-- <xacro:set_all_wheel_frictions tf_prefix="${tf_prefix}"/> -->

Commit message: Update mir_200.gazebo.xacro
Fixed an issue with xacro:macro where the \scan topic would not be published

File: mir/mir_description/urdf/mir_200/mir_200.gazebo.xacro (robot description, xacro)
@@ -47,6 +47,6 @@
 		<!-- Add Gazebo xacro for the laser scanner to work in Gazebo-->
 		<!-- Please match there macro calls with the sick_s300 xacro calls in the mir_200.urdf.xacro file-->
-		<xacro:macro name="sick_s300_gazebo" link="front_laser_link" topic="f_scan" tf_prefix="${tf_prefix}"/>
-		<xacro:macro name="sick_s300_gazebo" link="back_laser_link" topic="b_scan" tf_prefix="${tf_prefix}"/>
+		<xacro:sick_s300_gazebo tf_prefix="${tf_prefix}" link="front_laser_link" topic="f_scan" />
+		<xacro:sick_s300_gazebo tf_prefix="${tf_prefix}" link="back_laser_link" topic="b_scan" />
 		<!-- Add transmissions to wheels -->
 		<xacro:mir_200_wheel_transmissions tf_prefix="${tf_prefix}"/>
