Commit message: changed friction, k-contact and min_depth

File: mir/mir_description/urdf/mir_200/mir_200_wheels.gazebo.xacro (robot description, xacro)
@@ -4,4 +4,20 @@
 		<gazebo reference="${locationprefix}_wheel_link">
 			<material>Gazebo/DarkGrey</material>
+			<collision>
+				<surface>
+				<contact>
+				<ode>
+					<kp>1000.0</kp>
+    				<kd>100.0</kd>
+				</ode>
+				</contact>
+				<friction>
+				<ode>
+					<mu>10000.0</mu>
+    				<mu2>100.0</mu2>
+				</ode>
+				</friction>
+				</surface>
+			</collision>
 		</gazebo>
 	</xacro:macro>
@@ -12,4 +28,21 @@
 		<gazebo reference="${locationprefix}_caster_wheel_link">
 			<material>Gazebo/DarkGrey</material>
+			<collision>
+				<surface>
+				<contact>
+				<ode>
+					<kp>1000000.0</kp>
+    				<kd>100.0</kd>
+					<min_depth>0.001</min_depth>
+				</ode>
+				</contact>
+				<friction>
+				<ode>
+					<mu>0.0</mu>
+    				<mu2>0.0</mu2>
+				</ode>
+				</friction>
+				</surface>
+			</collision>
 		</gazebo>
 	</xacro:macro>
