Commit message: Started removing tf_prefix to implement new and correct camera

File: mir/mir_description/urdf/mir_200/mir_200.urdf.xacro (robot description, xacro)
@@ -23,11 +23,11 @@
 	<xacro:property name="mir_200_caster_wheel_base_dz" value="${mir_200_caster_wheel_radius-mir_200_caster_wheel_dz}" />
 	<xacro:macro name="mir_200" params="tf_prefix">
-		<link name="${tf_prefix}base_footprint" />
-		<joint name="${tf_prefix}base_joint" type="fixed">
-			<parent link="${tf_prefix}base_footprint" />
-			<child link="${tf_prefix}base_link" />
+		<link name="base_footprint" />
+		<joint name="base_joint" type="fixed">
+			<parent link="base_footprint" />
+			<child link="base_link" />
 			<origin xyz="0 0 0" rpy="0 0 0" />
 		</joint>
-		<link name="${tf_prefix}base_link">
+		<link name="base_link">
 		<xacro:box_inertial mass="${mir_200_base_mass}" x="0.9" y="0.58" z="0.3">
 			<origin xyz="${mir_200_act_wheel_dx} 0 0.20" rpy="0 0 0" />
@@ -48,45 +48,45 @@
 		</link>
 		<!-- IMU -->
-		<joint name="${tf_prefix}base_link_to_imu_joint" type="fixed">
-			<parent link="${tf_prefix}base_link" />
-			<child link="${tf_prefix}imu_link" />
+		<joint name="base_link_to_imu_joint" type="fixed">
+			<parent link="base_link" />
+			<child link="imu_link" />
 			<origin xyz="0.0 0.0 0.25" rpy="0 0 0" />  <!-- same as real MiR -->
 		</joint>
-		<link name="${tf_prefix}imu_link" />
+		<link name="imu_link" />
 		<!-- Create an alias for imu_link. This is necessary because the real MiR's
 			TF has imu_link, but the imu_data topic is published in the imu_frame
 			frame. -->
-		<joint name="${tf_prefix}imu_link_to_imu_frame_joint" type="fixed">
-			<parent link="${tf_prefix}imu_link" />
-			<child link="${tf_prefix}imu_frame" />
+		<joint name="imu_link_to_imu_frame_joint" type="fixed">
+			<parent link="imu_link" />
+			<child link="imu_frame" />
 			<origin xyz="0 0 0" rpy="0 0 0" />
 		</joint>
-		<link name="${tf_prefix}imu_frame" />
+		<link name="imu_frame" />
 		<!-- Laser scanners -->
-		<joint name="${tf_prefix}base_link_to_front_laser_joint" type="fixed">
-			<parent link="${tf_prefix}base_link" />
-			<child link="${tf_prefix}front_laser_link" />
+		<joint name="base_link_to_front_laser_joint" type="fixed">
+			<parent link="base_link" />
+			<child link="front_laser_link" />
 			<origin xyz="0.4288 0.2358 0.1914" rpy="0.0 0.0 ${0.25 * pi}" />  <!-- from visually matching up the meshes of the MiR and the laser scanner -->
 		</joint>
 		<xacro:sick_s300 tf_prefix="${tf_prefix}" link="front_laser_link" topic="f_scan" />
-		<joint name="${tf_prefix}base_link_to_back_laser_joint" type="fixed">
-			<parent link="${tf_prefix}base_link" />
-			<child link="${tf_prefix}back_laser_link" />
+		<joint name="base_link_to_back_laser_joint" type="fixed">
+			<parent link="base_link" />
+			<child link="back_laser_link" />
 			<origin xyz="-0.3548 -0.2352 0.1914" rpy="0.0 0.0 ${-0.75 * pi}" />  <!-- from visually matching up the meshes of the MiR and the laser scanner -->
 		</joint>
 		<xacro:sick_s300 tf_prefix="${tf_prefix}" link="back_laser_link" topic="b_scan" />
 		<!-- Ultrasound sensors -->
-		<joint name="${tf_prefix}us_1_joint" type="fixed">   <!-- right ultrasound -->
-			<parent link="${tf_prefix}base_link" />
-			<child link="${tf_prefix}us_1_frame" />
+		<joint name="us_1_joint" type="fixed">   <!-- right ultrasound -->
+			<parent link="base_link" />
+			<child link="us_1_frame" />
 			<origin xyz="0.45 -0.12 0.16 " rpy="0 0 0" />  <!-- from visually matching to the mesh of the MiR -->
 		</joint>
-		<link name="${tf_prefix}us_1_frame" />
-		<joint name="${tf_prefix}us_2_joint" type="fixed">   <!-- left ultrasound -->
-			<parent link="${tf_prefix}base_link" />
-			<child link="${tf_prefix}us_2_frame" />
+		<link name="us_1_frame" />
+		<joint name="us_2_joint" type="fixed">   <!-- left ultrasound -->
+			<parent link="base_link" />
+			<child link="us_2_frame" />
 			<origin xyz="0.45 0.12 0.16 " rpy="0 0 0" />  <!-- from visually matching to the mesh of the MiR -->
 		</joint>
-		<link name="${tf_prefix}us_2_frame" />
+		<link name="us_2_frame" />
 		<!-- wheels -->
 		<xacro:actuated_wheel tf_prefix="${tf_prefix}" locationprefix="left" locationright="-1"/>
@@ -96,11 +96,11 @@
 		<xacro:caster_wheel tf_prefix="${tf_prefix}" locationprefix="bl" locationright="-1" wheel_base_dx="${mir_200_back_caster_wheel_base_dx}"/>
 		<xacro:caster_wheel tf_prefix="${tf_prefix}" locationprefix="br" locationright="1" wheel_base_dx="${mir_200_back_caster_wheel_base_dx}"/>
-		<joint name="${tf_prefix}base_link_surface_joint" type="fixed">
+		<joint name="base_link_surface_joint" type="fixed">
 			<origin xyz="${mir_200_act_wheel_dx} 0 0.352" rpy="0 0 0" />
-			<parent link="${tf_prefix}base_link" />
-			<child link="${tf_prefix}surface" />
+			<parent link="base_link" />
+			<child link="surface" />
 			<axis xyz="0 0 1" />
 		</joint>
-		<link name="${tf_prefix}surface"/>
+		<link name="surface"/>
 		<!-- Camera -->
 		<!--link name="camera_link">
@@ -141,5 +141,5 @@
 		<!--/link-->
 		<!--Realsense_Intel_D435_Camera-->
-		<xacro:sensor_d435 name="camera" topics_ns="camera" parent="${tf_prefix}base_link" publish_pointcloud="true">
+		<xacro:sensor_d435 name="camera" topics_ns="camera" parent="base_link" publish_pointcloud="true">
     		<origin xyz="0.42 0 0.27" rpy="0 0 0" />
   		</xacro:sensor_d435>

Commit message: Replaced copied and old d435 urdf xacro file for new one through a submodule

File: mir/mir_description/urdf/mir_200/mir_200.urdf.xacro (robot description, xacro)
@@ -4,5 +4,5 @@
 	<xacro:include filename="$(find mir_description)/urdf/general/sick_s300.urdf.xacro" />
 	<xacro:include filename="$(find mir_description)/urdf/mir_200/mir_200_wheels.urdf.xacro" />
-	<xacro:include filename="$(find mir_description)/urdf/general/_d435.urdf.xacro" />
+	<xacro:include filename="$(find realsense2_description)/urdf/_d435.urdf.xacro" />
 	<xacro:property name="deg_to_rad" value="${(1 / 360) * (2 * pi)}" />
 	<xacro:property name="mir_200_base_mass" value="58.0" />
@@ -103,4 +103,8 @@
 		</joint>
 		<link name="surface"/>
+		<!--Realsense_Intel_D435_Camera-->
+		<xacro:sensor_d435 name="camera" parent="base_link" use_nominal_extrinsics="true">
+    		<origin xyz="0.42 0 0.27" rpy="0 0 0" />
+  		</xacro:sensor_d435>
 		<!-- Camera -->
 		<!--link name="camera_link">
@@ -140,8 +144,4 @@
 		<link name="camera_link_optical"-->
 		<!--/link-->
-		<!--Realsense_Intel_D435_Camera-->
-		<xacro:sensor_d435 name="camera" topics_ns="camera" parent="base_link" publish_pointcloud="true">
-    		<origin xyz="0.42 0 0.27" rpy="0 0 0" />
-  		</xacro:sensor_d435>
 	</xacro:macro>
 </robot>

Commit message: removed pids again

File: mir/mir_description/urdf/mir_200/mir_200.urdf.xacro (robot description, xacro)
@@ -10,5 +10,5 @@
 	<xacro:property name="mir_200_act_wheel_radius" value="0.0625" />
 	<xacro:property name="mir_200_act_wheel_width" value="0.032" />
-	<xacro:property name="mir_200_act_wheel_mass" value="1.0" />
+	<xacro:property name="mir_200_act_wheel_mass" value="20.0" />
 	<xacro:property name="mir_200_act_wheel_dx" value="0.037646" />
 	<xacro:property name="mir_200_act_wheel_dy" value="0.222604" />

File: mur/mur_description/urdf/mur_620.gazebo.xacro (robot description, xacro)
@@ -8,4 +8,5 @@
 	<!-- UR5 robot arm -->
   	<xacro:include filename="$(find ur_description)/urdf/inc/ur16e_macro.xacro"/>
+	<xacro:include filename="$(find ur_description)/urdf/inc/ur10e_macro.xacro"/>
 	<!-- Include plugin xacros -->
 	<xacro:include filename="$(find mir_description)/urdf/general/plugins.gazebo.xacro" />
@@ -16,16 +17,16 @@
 	<xacro:mir_600_gazebo tf_prefix="$(arg tf_prefix)" robot_namespace="$(arg robot_namespace)"/>
 	<!-- Init the UR5 robot arm macro -->
-	<xacro:ur16e_robot prefix="UR10l/" transmission_hw_interface="hardware_interface/VelocityJointInterface"/>
-	<xacro:ur16e_robot prefix="UR10r/" transmission_hw_interface="hardware_interface/VelocityJointInterface"/>
+	<xacro:ur10e_robot prefix="UR10_l/" transmission_hw_interface="hardware_interface/VelocityJointInterface"/>
+	<xacro:ur10e_robot prefix="UR10_r/" transmission_hw_interface="hardware_interface/VelocityJointInterface"/>
 	<!-- Init the plugins that run the MiR in Gazebo -->
 	<xacro:controller_plugin_gazebo robot_namespace="$(arg robot_namespace)"/>
 	<joint name="plattform_manipulator_joint_l" type="fixed">
 			<parent link="left_lift_top" />
-			<child link="UR10l/base_link" />
+			<child link="UR10_l/base_link" />
 			<origin xyz="0.0 0.0 0.555" rpy="0 0 0" />
 	</joint>
 	<joint name="plattform_manipulator_joint_r" type="fixed">
 			<parent link="right_lift_top" />
-			<child link="UR10r/base_link" />
+			<child link="UR10_r/base_link" />
 			<origin xyz="0.0 0.0 0.555" rpy="0 0 0" />
 	</joint>
