Commit message: Completely removed tf_prefix from the hw urdf file

File: mir/mir_description/urdf/general/sick_s300.urdf.xacro (robot description, xacro)
@@ -6,6 +6,6 @@
 	<xacro:property name="laser_z" value="0.185" />
 	<xacro:property name="laser_mass" value="2.0" />
-	<xacro:macro name="sick_s300" params="tf_prefix link topic">
-		<link name="${tf_prefix}${link}">
+	<xacro:macro name="sick_s300" params="link topic">
+		<link name="${link}">
 			<visual>
 				<origin xyz="0.0 0.0 0.0" rpy="${pi} 0 0" />

File: mir/mir_description/urdf/mir_200/mir_200.urdf.xacro (robot description, xacro)
@@ -22,5 +22,5 @@
 	<xacro:property name="mir_200_caster_wheel_base_dy" value="0.203" />
 	<xacro:property name="mir_200_caster_wheel_base_dz" value="${mir_200_caster_wheel_radius-mir_200_caster_wheel_dz}" />
-	<xacro:macro name="mir_200" params="tf_prefix">
+	<xacro:macro name="mir_200">
 		<link name="base_footprint" />
 		<joint name="base_joint" type="fixed">
@@ -69,5 +69,5 @@
 			<origin xyz="0.4288 0.2358 0.1914" rpy="0.0 0.0 ${0.25 * pi}" />  <!-- from visually matching up the meshes of the MiR and the laser scanner -->
 		</joint>
-		<xacro:sick_s300 tf_prefix="${tf_prefix}" link="front_laser_link" topic="f_scan" />
+		<xacro:sick_s300 link="front_laser_link" topic="f_scan" />
 		<joint name="base_link_to_back_laser_joint" type="fixed">
 			<parent link="base_link" />
@@ -75,5 +75,5 @@
 			<origin xyz="-0.3548 -0.2352 0.1914" rpy="0.0 0.0 ${-0.75 * pi}" />  <!-- from visually matching up the meshes of the MiR and the laser scanner -->
 		</joint>
-		<xacro:sick_s300 tf_prefix="${tf_prefix}" link="back_laser_link" topic="b_scan" />
+		<xacro:sick_s300 link="back_laser_link" topic="b_scan" />
 		<!-- Ultrasound sensors -->
 		<joint name="us_1_joint" type="fixed">   <!-- right ultrasound -->
@@ -90,10 +90,10 @@
 		<link name="us_2_frame" />
 		<!-- wheels -->
-		<xacro:actuated_wheel tf_prefix="${tf_prefix}" locationprefix="left" locationright="-1"/>
-		<xacro:actuated_wheel tf_prefix="${tf_prefix}" locationprefix="right" locationright="1"/>
-		<xacro:caster_wheel tf_prefix="${tf_prefix}" locationprefix="fl" locationright="-1" wheel_base_dx="${mir_200_front_caster_wheel_base_dx}"/>
-		<xacro:caster_wheel tf_prefix="${tf_prefix}" locationprefix="fr" locationright="1" wheel_base_dx="${mir_200_front_caster_wheel_base_dx}"/>
-		<xacro:caster_wheel tf_prefix="${tf_prefix}" locationprefix="bl" locationright="-1" wheel_base_dx="${mir_200_back_caster_wheel_base_dx}"/>
-		<xacro:caster_wheel tf_prefix="${tf_prefix}" locationprefix="br" locationright="1" wheel_base_dx="${mir_200_back_caster_wheel_base_dx}"/>
+		<xacro:actuated_wheel locationprefix="left" locationright="-1"/>
+		<xacro:actuated_wheel locationprefix="right" locationright="1"/>
+		<xacro:caster_wheel locationprefix="fl" locationright="-1" wheel_base_dx="${mir_200_front_caster_wheel_base_dx}"/>
+		<xacro:caster_wheel locationprefix="fr" locationright="1" wheel_base_dx="${mir_200_front_caster_wheel_base_dx}"/>
+		<xacro:caster_wheel locationprefix="bl" locationright="-1" wheel_base_dx="${mir_200_back_caster_wheel_base_dx}"/>
+		<xacro:caster_wheel locationprefix="br" locationright="1" wheel_base_dx="${mir_200_back_caster_wheel_base_dx}"/>
 		<joint name="base_link_surface_joint" type="fixed">
 			<origin xyz="${mir_200_act_wheel_dx} 0 0.352" rpy="0 0 0" />

File: mir/mir_description/urdf/mir_200/mir_200_wheels.urdf.xacro (robot description, xacro)
@@ -2,13 +2,13 @@
 <robot xmlns:xacro="http://ros.org/wiki/xacro">
 	<xacro:include filename="$(find mir_description)/urdf/general/common_properties.urdf.xacro" />
-	<xacro:macro name="actuated_wheel" params="tf_prefix locationprefix locationright">
-		<joint name="${tf_prefix}${locationprefix}_wheel_joint" type="continuous">
+	<xacro:macro name="actuated_wheel" params="locationprefix locationright">
+		<joint name="${locationprefix}_wheel_joint" type="continuous">
 			<origin xyz="0.0 ${-mir_200_act_wheel_dy * locationright} ${mir_200_act_wheel_radius}" rpy="0 0 0" />
-			<parent link="${tf_prefix}base_link" />
-			<child link="${tf_prefix}${locationprefix}_wheel_link" />
+			<parent link="base_link" />
+			<child link="${locationprefix}_wheel_link" />
 			<axis xyz="0 1 0" />
 			<limit effort="200" velocity="20.0" />
 		</joint>
-		<link name="${tf_prefix}${locationprefix}_wheel_link">
+		<link name="${locationprefix}_wheel_link">
 			<xacro:cylinder_inertial mass="${mir_200_act_wheel_mass}" radius="${mir_200_act_wheel_radius}" length="${mir_200_act_wheel_width}">
 				<origin xyz="0 0 0" rpy="${0.5 * pi} 0 0" />
@@ -29,14 +29,14 @@
 		</link>
 	</xacro:macro>
-	<xacro:macro name="caster_wheel" params="tf_prefix locationprefix locationright wheel_base_dx">
+	<xacro:macro name="caster_wheel" params="locationprefix locationright wheel_base_dx">
 		<!-- caster hub -->
-		<joint name="${tf_prefix}${locationprefix}_caster_rotation_joint" type="continuous">
+		<joint name="${locationprefix}_caster_rotation_joint" type="continuous">
 			<origin xyz="${wheel_base_dx} ${-mir_200_caster_wheel_base_dy * locationright} ${mir_200_caster_wheel_base_dz}" rpy="0 0 0" />
-			<parent link="${tf_prefix}base_link" />
-			<child link="${tf_prefix}${locationprefix}_caster_rotation_link" />
+			<parent link="base_link" />
+			<child link="${locationprefix}_caster_rotation_link" />
 			<axis xyz="0 0 1" />
 			<dynamics damping="0.01" friction="0.0"/>
 		</joint>
-		<link name="${tf_prefix}${locationprefix}_caster_rotation_link">
+		<link name="${locationprefix}_caster_rotation_link">
 		<inertial>
 			<!-- <origin xyz="0 0 -0.042500000044" rpy="${0.5 * pi} ${24 * deg_to_rad} ${1.5 * pi}" /> -->
@@ -66,11 +66,11 @@
 		</link>
 		<!-- caster wheel -->
-		<joint name="${tf_prefix}${locationprefix}_caster_wheel_joint" type="continuous">
+		<joint name="${locationprefix}_caster_wheel_joint" type="continuous">
 			<origin xyz="${mir_200_caster_wheel_dx} ${-mir_200_caster_wheel_dy * locationright} ${mir_200_caster_wheel_dz}" rpy="0 0 0" />
-			<parent link="${tf_prefix}${locationprefix}_caster_rotation_link" />
-			<child link="${tf_prefix}${locationprefix}_caster_wheel_link" />
+			<parent link="${locationprefix}_caster_rotation_link" />
+			<child link="${locationprefix}_caster_wheel_link" />
 			<axis xyz="0 1 0" />
 		</joint>
-		<link name="${tf_prefix}${locationprefix}_caster_wheel_link">
+		<link name="${locationprefix}_caster_wheel_link">
 			<xacro:cylinder_inertial mass="${mir_200_caster_wheel_mass}" radius="${mir_200_caster_wheel_radius}" length="${mir_200_caster_wheel_width}">
 				<origin xyz="0 0 0" rpy="${0.5 * pi} 0 0" />
