Commit message: Working D435 camera for multiple robots

File: mir/mir_description/urdf/general/_d435.gazebo.xacro (robot description, xacro)
@@ -6,5 +6,5 @@
 -->
 <robot xmlns:xacro="http://ros.org/wiki/xacro">
-  <xacro:macro name="gazebo_d435" params="camera_name reference_link tf_prefix robot_namespace topics_ns depth_optical_frame color_optical_frame infrared1_optical_frame infrared2_optical_frame publish_pointcloud:=true" >
+  <xacro:macro name="gazebo_d435" params="camera_name reference_link topics_ns depth_optical_frame color_optical_frame infrared1_optical_frame infrared2_optical_frame publish_pointcloud:=true" >
     <!-- Load parameters to model's main link-->
     <xacro:property name="deg_to_rad" value="0.01745329251994329577" />
@@ -113,5 +113,5 @@
     <!-- tf_prefix is necessary for the configuration of the plugin as it looks like the plugin doesnt use the robot_state_publishers tf_prefix-->
     <gazebo>
-      <plugin name="${robot_namespace}/${topics_ns}" filename="librealsense_gazebo_plugin.so">
+      <plugin name="${topics_ns}" filename="librealsense_gazebo_plugin.so">
         <prefix>${camera_name}</prefix>
         <depthUpdateRate>30.0</depthUpdateRate>
@@ -126,8 +126,8 @@
         <infrared2TopicName>infra2/image_raw</infrared2TopicName>
         <infrared2CameraInfoTopicName>infra2/camera_info</infrared2CameraInfoTopicName>
-        <colorOpticalframeName>${tf_prefix}/${color_optical_frame}</colorOpticalframeName>
-        <depthOpticalframeName>${tf_prefix}/${depth_optical_frame}</depthOpticalframeName>
-        <infrared1OpticalframeName>${tf_prefix}/${infrared1_optical_frame}</infrared1OpticalframeName>
-        <infrared2OpticalframeName>${tf_prefix}/${infrared2_optical_frame}</infrared2OpticalframeName>
+        <colorOpticalframeName>${color_optical_frame}</colorOpticalframeName>
+        <depthOpticalframeName>${depth_optical_frame}</depthOpticalframeName>
+        <infrared1OpticalframeName>${infrared1_optical_frame}</infrared1OpticalframeName>
+        <infrared2OpticalframeName>${infrared2_optical_frame}</infrared2OpticalframeName>
         <rangeMinDepth>0.2</rangeMinDepth>
         <rangeMaxDepth>10.0</rangeMaxDepth>

File: mir/mir_description/urdf/mir_200/mir_200.gazebo.xacro (robot description, xacro)
@@ -32,5 +32,5 @@
 		</gazebo-->
 		<!-- Settings for the camera of the robot to work in the simulation environment-->
-    	<xacro:gazebo_d435 camera_name="camera" reference_link="camera_link" tf_prefix="${tf_prefix}" robot_namespace="${robot_namespace}" topics_ns="camera" depth_optical_frame="camera_depth_optical_frame" color_optical_frame="camera_color_optical_frame" infrared1_optical_frame="camera_left_ir_optical_frame" infrared2_optical_frame="camera_right_ir_optical_frame" publish_pointcloud="true"/>
+    	<xacro:gazebo_d435 camera_name="${robot_namespace}_camera" reference_link="camera_link" topics_ns="${robot_namespace}/camera" depth_optical_frame="${tf_prefix}/camera_depth_optical_frame" color_optical_frame="${tf_prefix}/camera_color_optical_frame" infrared1_optical_frame="${tf_prefix}/camera_left_ir_optical_frame" infrared2_optical_frame="${tf_prefix}/camera_right_ir_optical_frame" publish_pointcloud="true"/>
 		<!-- Set Gazebo material for the base -->
 		<gazebo reference="base_link">
