Commit message: Added meshes for match logo Added match logo to both sides of the MiR200

File: mir/mir_description/urdf/general/common_properties.urdf.xacro (robot description, xacro)
@@ -50,4 +50,9 @@
 		</material>
 	</xacro:property>
+	<xacro:property name="material_match_green">
+		<material name="match_green">
+			<color rgba="${176.0/255.0} ${203.0/255.0} ${33.0/255.0} 1"/>
+		</material>
+	</xacro:property>
 	<!-- #################### inertials with origin #################### -->
 	<!-- see https://secure.wikimedia.org/wikipedia/en/wiki/List_of_moment_of_inertia_tensors -->

File: mir/mir_description/urdf/mir_200/mir_200.urdf.xacro (robot description, xacro)
@@ -4,4 +4,5 @@
 	<xacro:include filename="$(find mir_description)/urdf/general/sick_s300.urdf.xacro" />
 	<xacro:include filename="$(find mir_description)/urdf/mir_200/mir_200_wheels.urdf.xacro" />
+	<xacro:include filename="$(find mir_description)/urdf/general/match_logo.urdf.xacro" />
 	<xacro:include filename="$(find realsense2_description)/urdf/_d435.urdf.xacro" />
 	<xacro:property name="deg_to_rad" value="${(1 / 360) * (2 * pi)}" />
@@ -22,4 +23,7 @@
 	<xacro:property name="mir_200_caster_wheel_base_dy" value="0.203" />
 	<xacro:property name="mir_200_caster_wheel_base_dz" value="${mir_200_caster_wheel_radius-mir_200_caster_wheel_dz}" />
+	<xacro:property name="mir_200_match_logo_dx" value="0.0" />
+	<xacro:property name="mir_200_match_logo_dy" value="0.2724435" />
+	<xacro:property name="mir_200_match_logo_dz" value="0.27" />
 	<xacro:macro name="mir_200">
 		<link name="base_footprint" />
@@ -30,20 +34,20 @@
 		</joint>
 		<link name="base_link">
-		<xacro:box_inertial mass="${mir_200_base_mass}" x="0.9" y="0.58" z="0.3">
-			<origin xyz="${mir_200_act_wheel_dx} 0 0.20" rpy="0 0 0" />
-		</xacro:box_inertial>
-		<visual>
-			<origin xyz="${mir_200_act_wheel_dx} 0 0" rpy="0 0 0" />
-			<geometry>
-				<mesh filename="package://mir_description/meshes/visual/MIR200_base.stl" />
-			</geometry>
-			<xacro:insert_block name="material_white" />
-		</visual>
-		<collision>
-			<origin xyz="${mir_200_act_wheel_dx} 0 0" rpy="0 0 0" />
-			<geometry>
-				<mesh filename="package://mir_description/meshes/collision/MIR200_base.stl" />
-			</geometry>
-		</collision>
+			<xacro:box_inertial mass="${mir_200_base_mass}" x="0.9" y="0.58" z="0.3">
+				<origin xyz="${mir_200_act_wheel_dx} 0 0.20" rpy="0 0 0" />
+			</xacro:box_inertial>
+			<visual>
+				<origin xyz="${mir_200_act_wheel_dx} 0 0" rpy="0 0 0" />
+				<geometry>
+					<mesh filename="package://mir_description/meshes/visual/MIR200_base.stl" />
+				</geometry>
+				<xacro:insert_block name="material_white" />
+			</visual>
+			<collision>
+				<origin xyz="${mir_200_act_wheel_dx} 0 0" rpy="0 0 0" />
+				<geometry>
+					<mesh filename="package://mir_description/meshes/collision/MIR200_base.stl" />
+				</geometry>
+			</collision>
 		</link>
 		<!-- IMU -->
@@ -107,4 +111,7 @@
     		<origin xyz="0.42 0 0.27" rpy="0 0 0" />
   		</xacro:sensor_d435>
+		<!-- Insert a match logo on both sides of the mobile robot -->
+		<xacro:match_logo parent="base_link" locationprefix="left" location_dx="${mir_200_match_logo_dx}" location_dy="${mir_200_match_logo_dy}" location_dz="${mir_200_match_logo_dz}"/>
+		<xacro:match_logo parent="base_link" locationprefix="right" location_dx="${mir_200_match_logo_dx}" location_dy="${-1 * mir_200_match_logo_dy}" location_dz="${mir_200_match_logo_dz}" orientation="${pi}"/>
 		<!-- Camera -->
 		<!--link name="camera_link">
