Commit message: Fixed namespace problems with the gazebo plugins

File: mir/mir_description/urdf/general/imu.gazebo.xacro (robot description, xacro)
@@ -10,5 +10,5 @@
 			<xacro:property name="imu_frame" value="$(arg tf_prefix)/imu_frame" />
 	</xacro:unless>
-	<xacro:macro name="imu_gazebo" params="link imu_topic update_rate standard_deviation">
+	<xacro:macro name="imu_gazebo" params="link robot_namespace imu_topic update_rate standard_deviation">
 		<gazebo reference="${link}">
 			<gravity>true</gravity>
@@ -19,4 +19,5 @@
 				<topic>__default_topic__</topic>
 				<plugin filename="libgazebo_ros_imu_sensor.so" name="imu_plugin">
+					<robotNamespace>/${robot_namespace}</robotNamespace>
 					<topicName>${imu_topic}</topicName>
 					<bodyName>${link}</bodyName>

File: mir/mir_description/urdf/general/plugins.gazebo.xacro (robot description, xacro)
@@ -5,5 +5,5 @@
 			<plugin name="gazebo_ros_control" filename="libgazebo_ros_control.so">
 				<xacro:unless value="${robot_namespace == ''}">
-					<robotNamespace>($robot_namespace)</robotNamespace>
+					<robotNamespace>/${robot_namespace}</robotNamespace>
 				</xacro:unless>
 				<controlPeriod>0.001</controlPeriod>

File: mir/mir_description/urdf/general/sick_s300.gazebo.xacro (robot description, xacro)
@@ -2,5 +2,5 @@
 <robot xmlns:xacro="http://ros.org/wiki/xacro">
 	<xacro:include filename="$(find mir_description)/urdf/general/common_properties.urdf.xacro" />
-	<xacro:macro name="sick_s300_gazebo" params="tf_prefix link topic">
+	<xacro:macro name="sick_s300_gazebo" params="tf_prefix link robot_namespace topic">
 		<gazebo reference="${tf_prefix}${link}">
 			<xacro:insert_block name="material_black" />
@@ -34,4 +34,5 @@
 				<plugin name="gazebo_ros_${link}_controller" filename="libgazebo_ros_laser.so">
 					<!-- no tf_prefix, plugin always uses a tf_prefix (if none is set it uses robotNamespace) -->
+					<robotNamespace>/${robot_namespace}</robotNamespace>
 					<frameName>${link}</frameName>
 					<topicName>${topic}</topicName>

File: mir/mir_description/urdf/mir_200/mir_200.gazebo.xacro (robot description, xacro)
@@ -6,5 +6,5 @@
 	<xacro:include filename="$(find mir_description)/urdf/general/plugins.gazebo.xacro" />
 	<xacro:property name="imu_standard_deviation" value="0.00017" />
-	<xacro:macro name="mir_200_gazebo" params="tf_prefix">
+	<xacro:macro name="mir_200_gazebo" params="tf_prefix robot_namespace">
 		<!-- Settings for the camera of the robot to work in the simulation environment-->
 		<gazebo reference="camera_link">
@@ -42,11 +42,11 @@
 		<xacro:caster_wheel_gazebo tf_prefix="${tf_prefix}" locationprefix="br"/>
 		<!-- Settings for the IMU of the robot to work in the simulation environment-->
-		<xacro:imu_gazebo link="${tf_prefix}imu_link" imu_topic="imu_data" update_rate="50.0" standard_deviation="${imu_standard_deviation}" />
+		<xacro:imu_gazebo link="${tf_prefix}imu_link" robot_namespace="${robot_namespace}" imu_topic="imu_data" update_rate="50.0" standard_deviation="${imu_standard_deviation}" />
 		<!--  -->
 		<!-- <p3d_base_controller tf_prefix="${tf_prefix}" /> -->
 		<!-- Add Gazebo xacro for the laser scanner to work in Gazebo-->
 		<!-- Please match there macro calls with the sick_s300 xacro calls in the mir_200.urdf.xacro file-->
-		<xacro:sick_s300_gazebo tf_prefix="${tf_prefix}" link="front_laser_link" topic="f_scan" />
-		<xacro:sick_s300_gazebo tf_prefix="${tf_prefix}" link="back_laser_link" topic="b_scan" />
+		<xacro:sick_s300_gazebo tf_prefix="${tf_prefix}" link="front_laser_link" robot_namespace="${robot_namespace}" topic="f_scan" />
+		<xacro:sick_s300_gazebo tf_prefix="${tf_prefix}" link="back_laser_link" robot_namespace="${robot_namespace}" topic="b_scan" />
 		<!-- Add transmissions to wheels -->
 		<xacro:mir_200_wheel_transmissions tf_prefix="${tf_prefix}"/>

Commit message: Fixed namespace problem when using one mir with no namespace Fixed using model_name instead of tf_prefix Improved formatting

File: mir/mir_description/urdf/general/imu.gazebo.xacro (robot description, xacro)
@@ -19,5 +19,5 @@
 				<topic>__default_topic__</topic>
 				<plugin filename="libgazebo_ros_imu_sensor.so" name="imu_plugin">
-					<robotNamespace>/${robot_namespace}</robotNamespace>
+					<robotNamespace>${robot_namespace}</robotNamespace>
 					<topicName>${imu_topic}</topicName>
 					<bodyName>${link}</bodyName>

File: mir/mir_description/urdf/general/plugins.gazebo.xacro (robot description, xacro)
@@ -5,5 +5,5 @@
 			<plugin name="gazebo_ros_control" filename="libgazebo_ros_control.so">
 				<xacro:unless value="${robot_namespace == ''}">
-					<robotNamespace>/${robot_namespace}</robotNamespace>
+					<robotNamespace>${robot_namespace}</robotNamespace>
 				</xacro:unless>
 				<controlPeriod>0.001</controlPeriod>

File: mir/mir_description/urdf/general/sick_s300.gazebo.xacro (robot description, xacro)
@@ -34,5 +34,5 @@
 				<plugin name="gazebo_ros_${link}_controller" filename="libgazebo_ros_laser.so">
 					<!-- no tf_prefix, plugin always uses a tf_prefix (if none is set it uses robotNamespace) -->
-					<robotNamespace>/${robot_namespace}</robotNamespace>
+					<robotNamespace>${robot_namespace}</robotNamespace>
 					<frameName>${link}</frameName>
 					<topicName>${topic}</topicName>

File: mir/mir_description/urdf/mir_200/mir_200.gazebo.xacro (robot description, xacro)
@@ -8,29 +8,25 @@
 	<xacro:property name="imu_standard_deviation" value="0.00017" />
 	<xacro:macro name="mir_200_gazebo" params="tf_prefix robot_namespace">
+		<!-- Predefine some values that are necessary later. It is important to differenciate between empty and not empty robot_namespace and tf_prefix -->
+		<xacro:if value="${robot_namespace == ''}">
+			<xacro:property name="robot_namespace_slashed" value="/" />
+		</xacro:if>
+		<xacro:unless value="${robot_namespace == ''}">
+				<xacro:property name="robot_namespace_slashed" value="${robot_namespace}/" />
+		</xacro:unless>
+		<xacro:if value="${tf_prefix == ''}">
+			<xacro:property name="tf_prefix_slashed" value="" />
+		</xacro:if>
+		<xacro:unless value="${tf_prefix == ''}">
+				<xacro:property name="tf_prefix_slashed" value="${tf_prefix}/" />
+		</xacro:unless>
+		<xacro:if value="${robot_namespace == ''}">
+			<xacro:property name="robot_namespace_underscored" value="" />
+		</xacro:if>
+		<xacro:unless value="${robot_namespace == ''}">
+				<xacro:property name="robot_namespace_underscored" value="${robot_namespace}_" />
+		</xacro:unless>
 		<!-- Settings for the camera of the robot to work in the simulation environment-->
-		<!--gazebo reference="camera_link">
-			<sensor type="depth" name="camera">
-			<plugin name="kinect_camera_controller" filename="libgazebo_ros_openni_kinect.so">
-				<cameraName>camera</cameraName>
-				<alwaysOn>true</alwaysOn>
-				<updateRate>10</updateRate>
-				<imageTopicName>rgb/image_raw</imageTopicName>
-				<depthImageTopicName>depth/image_raw</depthImageTopicName>
-				<pointCloudTopicName>depth/points</pointCloudTopicName>
-				<cameraInfoTopicName>rgb/camera_info</cameraInfoTopicName>
-				<depthImageCameraInfoTopicName>depth/camera_info</depthImageCameraInfoTopicName>
-				<frameName>camera_link_optical</frameName>
-				<baseline>0.1</baseline>
-				<distortion_k1>0.0</distortion_k1>
-				<distortion_k2>0.0</distortion_k2>
-				<distortion_k3>0.0</distortion_k3>
-				<distortion_t1>0.0</distortion_t1>
-				<distortion_t2>0.0</distortion_t2>
-				<pointCloudCutoff>0.4</pointCloudCutoff>
-			</plugin>
-			</sensor>
-		</gazebo-->
-		<!-- Settings for the camera of the robot to work in the simulation environment-->
-    	<xacro:gazebo_d435 camera_name="${robot_namespace}_camera" reference_link="camera_link" topics_ns="${robot_namespace}/camera" depth_optical_frame="${tf_prefix}/camera_depth_optical_frame" color_optical_frame="${tf_prefix}/camera_color_optical_frame" infrared1_optical_frame="${tf_prefix}/camera_left_ir_optical_frame" infrared2_optical_frame="${tf_prefix}/camera_right_ir_optical_frame" publish_pointcloud="true"/>
+    	<xacro:gazebo_d435 camera_name="${robot_namespace_underscored}camera" reference_link="camera_link" topics_ns="${robot_namespace_slashed}camera" depth_optical_frame="${tf_prefix_slashed}camera_depth_optical_frame" color_optical_frame="${tf_prefix_slashed}camera_color_optical_frame" infrared1_optical_frame="${tf_prefix_slashed}camera_left_ir_optical_frame" infrared2_optical_frame="${tf_prefix_slashed}camera_right_ir_optical_frame" publish_pointcloud="true"/>
 		<!-- Set Gazebo material for the base -->
 		<gazebo reference="base_link">
@@ -45,11 +41,9 @@
 		<xacro:caster_wheel_gazebo locationprefix="br"/>
 		<!-- Settings for the IMU of the robot to work in the simulation environment-->
-		<xacro:imu_gazebo link="imu_link" robot_namespace="${robot_namespace}" imu_topic="imu_data" update_rate="50.0" standard_deviation="${imu_standard_deviation}" />
-		<!--  -->
-		<!-- <p3d_base_controller tf_prefix="${tf_prefix}" /> -->
+		<xacro:imu_gazebo link="imu_link" robot_namespace="${robot_namespace_slashed}" imu_topic="imu_data" update_rate="50.0" standard_deviation="${imu_standard_deviation}" />
 		<!-- Add Gazebo xacro for the laser scanner to work in Gazebo -->
 		<!-- Please match there macro calls with the sick_s300 xacro calls in the mir_200.urdf.xacro file-->
-		<xacro:sick_s300_gazebo link="front_laser_link" robot_namespace="${robot_namespace}" topic="f_scan" />
-		<xacro:sick_s300_gazebo link="back_laser_link" robot_namespace="${robot_namespace}" topic="b_scan" />
+		<xacro:sick_s300_gazebo link="front_laser_link" robot_namespace="${robot_namespace_slashed}" topic="f_scan" />
+		<xacro:sick_s300_gazebo link="back_laser_link" robot_namespace="${robot_namespace_slashed}" topic="b_scan" />
 		<!-- Add transmissions to wheels -->
 		<xacro:mir_200_wheel_transmissions/>
@@ -98,4 +92,28 @@
 			<xacro:set_wheel_friction link="${prefix}br_caster_wheel_link" friction="1"/>
 		</xacro:macro> -->
+		<!-- <p3d_base_controller tf_prefix="${tf_prefix}" /> -->
+		<!-- Settings for the camera of the robot to work in the simulation environment-->
+		<!--gazebo reference="camera_link">
+			<sensor type="depth" name="camera">
+			<plugin name="kinect_camera_controller" filename="libgazebo_ros_openni_kinect.so">
+				<cameraName>camera</cameraName>
+				<alwaysOn>true</alwaysOn>
+				<updateRate>10</updateRate>
+				<imageTopicName>rgb/image_raw</imageTopicName>
+				<depthImageTopicName>depth/image_raw</depthImageTopicName>
+				<pointCloudTopicName>depth/points</pointCloudTopicName>
+				<cameraInfoTopicName>rgb/camera_info</cameraInfoTopicName>
+				<depthImageCameraInfoTopicName>depth/camera_info</depthImageCameraInfoTopicName>
+				<frameName>camera_link_optical</frameName>
+				<baseline>0.1</baseline>
+				<distortion_k1>0.0</distortion_k1>
+				<distortion_k2>0.0</distortion_k2>
+				<distortion_k3>0.0</distortion_k3>
+				<distortion_t1>0.0</distortion_t1>
+				<distortion_t2>0.0</distortion_t2>
+				<pointCloudCutoff>0.4</pointCloudCutoff>
+			</plugin>
+			</sensor>
+		</gazebo-->
 	</xacro:macro>
 </robot>
