Commit message: Cleaned up files further - better separation between common files

File: mir/mir_description/urdf/general/plugins.gazebo.xacro (robot description, xacro)
@@ -12,5 +12,6 @@
 		</gazebo>
 	</xacro:macro>
-	<xacro:macro name="p3d_base_controller" params="prefix">
+	<!-- This controller is deprecated and forbidden in Noetic -->
+	<!-- <xacro:macro name="p3d_base_controller" params="prefix">
 		<gazebo>
 		<plugin name="p3d_base_controller" filename="libgazebo_ros_p3d.so">
@@ -25,20 +26,4 @@
 		</plugin>
 		</gazebo>
-	</xacro:macro>
-	<!-- <xacro:macro name="set_wheel_friction" params="link friction">
-		<gazebo reference="${link}">
-			<mu1 value="${friction}"/>
-			<mu2 value="${friction}"/>
-			<kp value="10000000.0"/>
-			<kd value="1.0"/>
-		</gazebo>
-	</xacro:macro>
-	<xacro:macro name="set_all_wheel_frictions" params="prefix">
-		<xacro:set_wheel_friction link="${prefix}left_wheel_link" friction="200"/>
-		<xacro:set_wheel_friction link="${prefix}right_wheel_link" friction="200"/>
-		<xacro:set_wheel_friction link="${prefix}fl_caster_wheel_link" friction="1"/>
-		<xacro:set_wheel_friction link="${prefix}fr_caster_wheel_link" friction="1"/>
-		<xacro:set_wheel_friction link="${prefix}bl_caster_wheel_link" friction="1"/>
-		<xacro:set_wheel_friction link="${prefix}br_caster_wheel_link" friction="1"/>
 	</xacro:macro> -->
 </robot>

File: mir/mir_description/urdf/mir_200/mir_200.gazebo.xacro (robot description, xacro)
@@ -4,4 +4,5 @@
 	<xacro:include filename="$(find mir_description)/urdf/general/sick_s300.gazebo.xacro" />
 	<xacro:include filename="$(find mir_description)/urdf/general/imu.gazebo.xacro" />
+	<xacro:include filename="$(find mir_description)/urdf/general/plugins.gazebo.xacro" />
 	<xacro:property name="imu_standard_deviation" value="0.00017" />
 	<xacro:macro name="mir_200_gazebo" params="tf_prefix">
@@ -42,10 +43,12 @@
 		<!-- Settings for the IMU of the robot to work in the simulation environment-->
 		<xacro:imu_gazebo link="${tf_prefix}imu_link" imu_topic="imu_data" update_rate="50.0" standard_deviation="${imu_standard_deviation}" />
-		<!-- -->
-		<p3d_base_controller tf_prefix="${tf_prefix}" />
+		<!--  -->
+		<!-- <p3d_base_controller tf_prefix="${tf_prefix}" /> -->
 		<!-- Add Gazebo xacro for the laser scanner to work in Gazebo-->
 		<!-- Please match there macro calls with the sick_s300 xacro calls in the mir_200.urdf.xacro file-->
 		<xacro:macro name="sick_s300_gazebo" link="front_laser_link" topic="f_scan" tf_prefix="${tf_prefix}"/>
 		<xacro:macro name="sick_s300_gazebo" link="back_laser_link" topic="b_scan" tf_prefix="${tf_prefix}"/>
+		<!-- Add transmissions to wheels -->
+		<xacro:mir_200_wheel_transmissions tf_prefix="${tf_prefix}"/>
 		<!-- disabled, because it doesn't make a difference in Gazebo: -->
 		<!-- <xacro:set_all_wheel_frictions tf_prefix="${tf_prefix}"/> -->

File: mir/mir_description/urdf/mir_200/mir_200.urdf.xacro (robot description, xacro)
@@ -102,5 +102,4 @@
 		</joint>
 		<link name="${tf_prefix}surface"/>
-		<xacro:mir_200_wheel_transmissions tf_prefix="${tf_prefix}"/>
 		<!-- Camera -->
 		<link name="camera_link">

File: mir/mir_description/urdf/mir_200/mir_200_wheels.gazebo.xacro (robot description, xacro)
@@ -14,3 +14,19 @@
 		</gazebo>
 	</xacro:macro>
+	<xacro:macro name="mir_200_wheel_transmission" params="tf_prefix locationprefix">
+		<transmission name="${tf_prefix}${locationprefix}_wheel_trans">
+		<type>transmission_interface/SimpleTransmission</type>
+		<joint name="${tf_prefix}${locationprefix}_wheel_joint">
+			<hardwareInterface>hardware_interface/VelocityJointInterface</hardwareInterface>
+		</joint>
+		<actuator name="${tf_prefix}${locationprefix}_wheel_motor">
+			<hardwareInterface>hardware_interface/VelocityJointInterface</hardwareInterface>
+			<mechanicalReduction>1</mechanicalReduction>
+		</actuator>
+		</transmission>
+	</xacro:macro>
+	<xacro:macro name="mir_200_wheel_transmissions" params="tf_prefix">
+		<xacro:mir_200_wheel_transmission tf_prefix="${tf_prefix}" locationprefix="left"/>
+		<xacro:mir_200_wheel_transmission tf_prefix="${tf_prefix}" locationprefix="right"/>
+	</xacro:macro>
 </robot>

File: mir/mir_description/urdf/mir_200/mir_200_wheels.urdf.xacro (robot description, xacro)
@@ -91,19 +91,3 @@
 		</link>
 	</xacro:macro>
-	<xacro:macro name="mir_200_wheel_transmission" params="tf_prefix locationprefix">
-		<transmission name="${tf_prefix}${locationprefix}_wheel_trans">
-		<type>transmission_interface/SimpleTransmission</type>
-		<joint name="${tf_prefix}${locationprefix}_wheel_joint">
-			<hardwareInterface>hardware_interface/VelocityJointInterface</hardwareInterface>
-		</joint>
-		<actuator name="${tf_prefix}${locationprefix}_wheel_motor">
-			<hardwareInterface>hardware_interface/VelocityJointInterface</hardwareInterface>
-			<mechanicalReduction>1</mechanicalReduction>
-		</actuator>
-		</transmission>
-	</xacro:macro>
-	<xacro:macro name="mir_200_wheel_transmissions" params="tf_prefix">
-		<xacro:mir_200_wheel_transmission tf_prefix="${tf_prefix}" locationprefix="left"/>
-		<xacro:mir_200_wheel_transmission tf_prefix="${tf_prefix}" locationprefix="right"/>
-	</xacro:macro>
 </robot>

Commit message: Added ground truth plugin to mir platforms

File: mir/mir_description/urdf/general/plugins.gazebo.xacro (robot description, xacro)
@@ -13,17 +13,19 @@
 	</xacro:macro>
 	<!-- This controller is deprecated and forbidden in Noetic -->
-	<!-- <xacro:macro name="p3d_base_controller" params="prefix">
+	<!-- This controller publishes the ground truth pose -->
+	<xacro:macro name="p3d_base_controller" params="robot_namespace">
 		<gazebo>
-		<plugin name="p3d_base_controller" filename="libgazebo_ros_p3d.so">
-			<alwaysOn>true</alwaysOn>
-			<updateRate>50.0</updateRate>
-			<bodyName>${prefix}base_footprint</bodyName>
-			<topicName>base_pose_ground_truth</topicName>
-			<gaussianNoise>0.01</gaussianNoise>
-			<frameName>map</frameName>
-			<xyzOffsets>0 0 0</xyzOffsets>
-			<rpyOffsets>0 0 0</rpyOffsets>
-		</plugin>
+			<plugin name="p3d_base_controller" filename="libgazebo_ros_p3d.so">
+				<robotNamespace>${robot_namespace}</robotNamespace>
+				<alwaysOn>true</alwaysOn>
+				<updateRate>50.0</updateRate>
+				<bodyName>base_footprint</bodyName>
+				<topicName>ground_truth</topicName>
+				<gaussianNoise>0.01</gaussianNoise>
+				<frameName>map</frameName>
+				<xyzOffsets>0 0 0</xyzOffsets>
+				<rpyOffsets>0 0 0</rpyOffsets>
+			</plugin>
 		</gazebo>
-	</xacro:macro> -->
+	</xacro:macro>
 </robot>
