Commit message: First version of new MiR200 urdf/xacro files

File: mir/mir_description/urdf/general/sick_s300.gazebo.xacro (robot description, xacro)
@@ -1,6 +1,6 @@
 <?xml version="1.0"?>
 <robot xmlns:xacro="http://ros.org/wiki/xacro">
-	<xacro:include filename="$(find mir_description)/urdf/include/common_properties.urdf.xacro" />
-	<!-- <xacro:macro name="sick_s300_gazebo" params="link topic tf_prefix"> -->
+	<xacro:include filename="$(find mir_description)/urdf/general/common_properties.urdf.xacro" />
+	<xacro:macro name="sick_s300_gazebo" params="link topic tf_prefix">
 		<gazebo reference="${tf_prefix}${link}">
 			<xacro:insert_block name="material_black" />
@@ -39,4 +39,4 @@
 			</sensor>
 		</gazebo>
-	<!-- </xacro:macro> -->
+	</xacro:macro>
 </robot>

File: mir/mir_description/urdf/general/sick_s300.urdf.xacro (robot description, xacro)
@@ -1,5 +1,5 @@
 <?xml version="1.0"?>
 <robot xmlns:xacro="http://ros.org/wiki/xacro">
-	<xacro:include filename="$(find mir_description)/urdf/include/common_properties.urdf.xacro" />
+	<xacro:include filename="$(find mir_description)/urdf/general/common_properties.urdf.xacro" />
 	<xacro:property name="laser_x" value="0.156" />
 	<xacro:property name="laser_y" value="0.155" />

File: mir/mir_description/urdf/mir_200/mir_200.gazebo.xacro (robot description, xacro)
@@ -1,8 +1,5 @@
 <?xml version="1.0"?>
-<robot xmlns:controller="http://playerstage.sourceforge.net/gazebo/xmlschema/#controller"
-		xmlns:interface="http://playerstage.sourceforge.net/gazebo/xmlschema/#interface"
-		xmlns:sensor="http://playerstage.sourceforge.net/gazebo/xmlschema/#sensor"
-		xmlns:xacro="http://ros.org/wiki/xacro">
-	<xacro:include filename="$(find mir_description)/urdf/mir_200/mir_200.urdf.xacro" />
+<robot xmlns:xacro="http://wiki.ros.org/xacro">
+	<!-- <xacro:include filename="$(find mir_description)/urdf/mir_200/mir_200.urdf.xacro" /> -->
 	<xacro:include filename="$(find mir_description)/urdf/mir_200/mir_200_wheels.gazebo.xacro" />
 	<xacro:include filename="$(find mir_description)/urdf/general/sick_s300.gazebo.xacro" />
@@ -11,5 +8,5 @@
 	<xacro:macro name="mir_200_gazebo" params="tf_prefix">
 		<!-- Call MiR200 xacro to get base robot model loaded-->
-		<xacro:mir_200 tf_prefix="${tf_prefix}">
+		<!-- <xacro:mir_200 tf_prefix="${tf_prefix}"> -->
 		<!-- Settings for the camera of the robot to work in the simulation environment-->
 		<gazebo reference="camera_link">
@@ -40,12 +37,12 @@
 		</gazebo>
 		<!-- Set gazebo material for the wheels -->
-		<xacro:actuated_wheel tf_prefix="${tf_prefix}" locationtf_prefix="left" locationright="-1"/>
-		<xacro:actuated_wheel tf_prefix="${tf_prefix}" locationtf_prefix="right" locationright="1"/>
-		<xacro:caster_wheel tf_prefix="${tf_prefix}" locationtf_prefix="fl" locationright="-1" wheel_base_dx="${mir_200_front_caster_wheel_base_dx}"/>
-		<xacro:caster_wheel tf_prefix="${tf_prefix}" locationtf_prefix="fr" locationright="1" wheel_base_dx="${mir_200_front_caster_wheel_base_dx}"/>
-		<xacro:caster_wheel tf_prefix="${tf_prefix}" locationtf_prefix="bl" locationright="-1" wheel_base_dx="${mir_200_back_caster_wheel_base_dx}"/>
-		<xacro:caster_wheel tf_prefix="${tf_prefix}" locationtf_prefix="br" locationright="1" wheel_base_dx="${mir_200_back_caster_wheel_base_dx}"/>
+		<xacro:actuated_wheel_gazebo tf_prefix="${tf_prefix}" locationprefix="left"/>
+		<xacro:actuated_wheel_gazebo tf_prefix="${tf_prefix}" locationprefix="right"/>
+		<xacro:caster_wheel_gazebo tf_prefix="${tf_prefix}" locationprefix="fl"/>
+		<xacro:caster_wheel_gazebo tf_prefix="${tf_prefix}" locationprefix="fr"/>
+		<xacro:caster_wheel_gazebo tf_prefix="${tf_prefix}" locationprefix="bl"/>
+		<xacro:caster_wheel_gazebo tf_prefix="${tf_prefix}" locationprefix="br"/>
 		<!-- Settings for the IMU of the robot to work in the simulation environment-->
-		<xacro:imu_gazebo link="${tf_prefix}imu_link" imu_topic="imu_data" update_rate="50.0" stdev="${imu_standard_deviation}" />
+		<xacro:imu_gazebo link="${tf_prefix}imu_link" imu_topic="imu_data" update_rate="50.0" standard_deviation="${imu_standard_deviation}" />
 		<!-- -->
 		<p3d_base_controller tf_prefix="${tf_prefix}" />
@@ -94,4 +91,4 @@
 			<xacro:set_wheel_friction link="${prefix}br_caster_wheel_link" friction="1"/>
 		</xacro:macro> -->
-	<xacro:macro>
+	</xacro:macro>
 </robot>

File: mir/mir_description/urdf/mir_200/mir_200.urdf.xacro (robot description, xacro)
@@ -89,10 +89,10 @@
 		<link name="${tf_prefix}us_2_frame" />
 		<!-- wheels -->
-		<xacro:actuated_wheel tf_prefix="${tf_prefix}" locationtf_prefix="left" locationright="-1"/>
-		<xacro:actuated_wheel tf_prefix="${tf_prefix}" locationtf_prefix="right" locationright="1"/>
-		<xacro:caster_wheel tf_prefix="${tf_prefix}" locationtf_prefix="fl" locationright="-1" wheel_base_dx="${mir_200_front_caster_wheel_base_dx}"/>
-		<xacro:caster_wheel tf_prefix="${tf_prefix}" locationtf_prefix="fr" locationright="1" wheel_base_dx="${mir_200_front_caster_wheel_base_dx}"/>
-		<xacro:caster_wheel tf_prefix="${tf_prefix}" locationtf_prefix="bl" locationright="-1" wheel_base_dx="${mir_200_back_caster_wheel_base_dx}"/>
-		<xacro:caster_wheel tf_prefix="${tf_prefix}" locationtf_prefix="br" locationright="1" wheel_base_dx="${mir_200_back_caster_wheel_base_dx}"/>
+		<xacro:actuated_wheel tf_prefix="${tf_prefix}" locationprefix="left" locationright="-1"/>
+		<xacro:actuated_wheel tf_prefix="${tf_prefix}" locationprefix="right" locationright="1"/>
+		<xacro:caster_wheel tf_prefix="${tf_prefix}" locationprefix="fl" locationright="-1" wheel_base_dx="${mir_200_front_caster_wheel_base_dx}"/>
+		<xacro:caster_wheel tf_prefix="${tf_prefix}" locationprefix="fr" locationright="1" wheel_base_dx="${mir_200_front_caster_wheel_base_dx}"/>
+		<xacro:caster_wheel tf_prefix="${tf_prefix}" locationprefix="bl" locationright="-1" wheel_base_dx="${mir_200_back_caster_wheel_base_dx}"/>
+		<xacro:caster_wheel tf_prefix="${tf_prefix}" locationprefix="br" locationright="1" wheel_base_dx="${mir_200_back_caster_wheel_base_dx}"/>
 		<joint name="${tf_prefix}base_link_surface_joint" type="fixed">
 			<origin xyz="${mir_200_act_wheel_dx} 0 0.352" rpy="0 0 0" />

Commit message: Added MiR100 urdf files

File: mir/mir_description/urdf/general/sick_s300.gazebo.xacro (robot description, xacro)
@@ -2,5 +2,5 @@
 <robot xmlns:xacro="http://ros.org/wiki/xacro">
 	<xacro:include filename="$(find mir_description)/urdf/general/common_properties.urdf.xacro" />
-	<xacro:macro name="sick_s300_gazebo" params="link topic tf_prefix">
+	<xacro:macro name="sick_s300_gazebo" params="tf_prefix link topic">
 		<gazebo reference="${tf_prefix}${link}">
 			<xacro:insert_block name="material_black" />

File: mir/mir_description/urdf/general/sick_s300.urdf.xacro (robot description, xacro)
@@ -6,5 +6,5 @@
 	<xacro:property name="laser_z" value="0.185" />
 	<xacro:property name="laser_mass" value="2.0" />
-	<xacro:macro name="sick_s300" params="link topic tf_prefix">
+	<xacro:macro name="sick_s300" params="tf_prefix link topic">
 		<link name="${tf_prefix}${link}">
 			<visual>

File: mir/mir_description/urdf/mir_100/mir_100.gazebo.xacro (robot description, xacro)
@@ -2,4 +2,5 @@
 <robot xmlns:xacro="http://ros.org/wiki/xacro">
 	<xacro:include filename="$(find mir_description)/urdf/general/imu.gazebo.xacro" />
+	<xacro:include filename="$(find mir_description)/urdf/general/sick_s300.gazebo.xacro" />
 	<xacro:property name="imu_standard_deviation" value="0.00017" />
 	<xacro:macro name="mir_100_gazebo" params="tf_prefix">
@@ -18,4 +19,8 @@
 		<xacro:caster_wheel_gazebo tf_prefix="${tf_prefix}" locationprefix="bl"/>
 		<xacro:caster_wheel_gazebo tf_prefix="${tf_prefix}" locationprefix="br"/>
+		<!-- Add Gazebo xacro for the laser scanner to work in Gazebo-->
+		<!-- Please match there macro calls with the sick_s300 xacro calls in the mir_200.urdf.xacro file-->
+		<xacro:sick_s300_gazebo tf_prefix="${tf_prefix}" link="front_laser_link" topic="f_scan"/>
+		<xacro:sick_s300_gazebo tf_prefix="${tf_prefix}" link="back_laser_link" topic="b_scan"/>
 		<!-- This part of the file looks like it is not necessary for the correct function of the urdf files.-->
 		<!-- Remove this part in a second iteration when all functions are working like they are supposed to be-->

Commit message: Added new camera. Currently not working for multi robot applications. Next commit will be

File: mir/mir_description/urdf/general/sick_s300.gazebo.xacro (robot description, xacro)
@@ -2,5 +2,5 @@
 <robot xmlns:xacro="http://ros.org/wiki/xacro">
 	<xacro:include filename="$(find mir_description)/urdf/general/common_properties.urdf.xacro" />
-	<xacro:macro name="sick_s300_gazebo" params="tf_prefix link robot_namespace topic">
+	<xacro:macro name="sick_s300_gazebo" params="tf_prefix link topic robot_namespace">
 		<gazebo reference="${tf_prefix}${link}">
 			<xacro:insert_block name="material_black" />

File: mir/mir_description/urdf/mir_200/mir_200.gazebo.xacro (robot description, xacro)
@@ -5,8 +5,9 @@
 	<xacro:include filename="$(find mir_description)/urdf/general/imu.gazebo.xacro" />
 	<xacro:include filename="$(find mir_description)/urdf/general/plugins.gazebo.xacro" />
+	<xacro:include filename="$(find mir_description)/urdf/general/_d435.gazebo.xacro" />
 	<xacro:property name="imu_standard_deviation" value="0.00017" />
 	<xacro:macro name="mir_200_gazebo" params="tf_prefix robot_namespace">
 		<!-- Settings for the camera of the robot to work in the simulation environment-->
-		<gazebo reference="camera_link">
+		<!--gazebo reference="camera_link">
 			<sensor type="depth" name="camera">
 			<plugin name="kinect_camera_controller" filename="libgazebo_ros_openni_kinect.so">
@@ -29,5 +30,7 @@
 			</plugin>
 			</sensor>
-		</gazebo>
+		</gazebo-->
+		<!-- Settings for the camera of the robot to work in the simulation environment-->
+    	<xacro:gazebo_d435 camera_name="camera" reference_link="camera_link" tf_prefix="${tf_prefix}" robot_namespace="${robot_namespace}" topics_ns="camera" depth_optical_frame="camera_depth_optical_frame" color_optical_frame="camera_color_optical_frame" infrared1_optical_frame="camera_left_ir_optical_frame" infrared2_optical_frame="camera_right_ir_optical_frame" publish_pointcloud="true"/>
 		<!-- Set Gazebo material for the base -->
 		<gazebo reference="${tf_prefix}base_link">
@@ -45,5 +48,5 @@
 		<!--  -->
 		<!-- <p3d_base_controller tf_prefix="${tf_prefix}" /> -->
-		<!-- Add Gazebo xacro for the laser scanner to work in Gazebo-->
+		<!-- Add Gazebo xacro for the laser scanner to work in Gazebo -->
 		<!-- Please match there macro calls with the sick_s300 xacro calls in the mir_200.urdf.xacro file-->
 		<xacro:sick_s300_gazebo tf_prefix="${tf_prefix}" link="front_laser_link" robot_namespace="${robot_namespace}" topic="f_scan" />

File: mir/mir_description/urdf/mir_200/mir_200.urdf.xacro (robot description, xacro)
@@ -4,4 +4,5 @@
 	<xacro:include filename="$(find mir_description)/urdf/general/sick_s300.urdf.xacro" />
 	<xacro:include filename="$(find mir_description)/urdf/mir_200/mir_200_wheels.urdf.xacro" />
+	<xacro:include filename="$(find mir_description)/urdf/general/_d435.urdf.xacro" />
 	<xacro:property name="deg_to_rad" value="${(1 / 360) * (2 * pi)}" />
 	<xacro:property name="mir_200_base_mass" value="58.0" />
@@ -103,5 +104,5 @@
 		<link name="${tf_prefix}surface"/>
 		<!-- Camera -->
-		<link name="camera_link">
+		<!--link name="camera_link">
 		<collision>
 			<origin xyz="0 0 0" rpy="0 0 0"/>
@@ -124,19 +125,23 @@
 		<joint name="camera_joint" type="fixed">
 			<axis xyz="0 1 0" />
-			<origin xyz="0.42 0 0.27" rpy="0 0.2 0"/> <!--set the position of the realsense-->
-			<parent link="${tf_prefix}base_link"/>
+			<origin xyz="0.42 0 0.27" rpy="0 0.2 0"/--> <!--set the position of the realsense-->
+			<!--parent link="${tf_prefix}base_link"/>
 			<child link="camera_link"/>
-		</joint>
+		</joint-->
 		<!-- generate an optical frame http://www.ros.org/reps/rep-0103.html#suffix-frames
 			so that ros and opencv can operate on the camera frame correctly -->
-		<joint name="camera_optical_joint" type="fixed">
+		<!--joint name="camera_optical_joint" type="fixed"-->
 			<!-- these values have to be these values otherwise the gazebo camera image
 				won't be aligned properly with the frame it is supposedly originating from -->
-			<origin xyz="0 0 0" rpy="-1.5708 0 -1.5708"/>
+			<!--origin xyz="0 0 0" rpy="-1.5708 0 -1.5708"/>
 			<parent link="camera_link"/>
 			<child link="camera_link_optical"/>
 		</joint>
-		<link name="camera_link_optical">
-		</link>
+		<link name="camera_link_optical"-->
+		<!--/link-->
+		<!--Realsense_Intel_D435_Camera-->
+		<xacro:sensor_d435 name="camera" topics_ns="camera" parent="${tf_prefix}base_link" publish_pointcloud="true">
+    		<origin xyz="0.42 0 0.27" rpy="0 0 0" />
+  		</xacro:sensor_d435>
 	</xacro:macro>
 </robot>

Commit message: Removed all unnecessary tf_prefix from the gazebo mir200 urdf

File: mir/mir_description/urdf/general/sick_s300.gazebo.xacro (robot description, xacro)
@@ -2,8 +2,8 @@
 <robot xmlns:xacro="http://ros.org/wiki/xacro">
 	<xacro:include filename="$(find mir_description)/urdf/general/common_properties.urdf.xacro" />
-	<xacro:macro name="sick_s300_gazebo" params="tf_prefix link topic robot_namespace">
-		<gazebo reference="${tf_prefix}${link}">
+	<xacro:macro name="sick_s300_gazebo" params="link topic robot_namespace">
+		<gazebo reference="${link}">
 			<xacro:insert_block name="material_black" />
-			<sensor type="ray" name="${tf_prefix}${link}">
+			<sensor type="ray" name="${link}">
 				<pose>0 0 0 0 0 0</pose>
 				<visualize>false</visualize>

File: mir/mir_description/urdf/mir_200/mir_200.gazebo.xacro (robot description, xacro)
@@ -34,24 +34,24 @@
     	<xacro:gazebo_d435 camera_name="camera" reference_link="camera_link" tf_prefix="${tf_prefix}" robot_namespace="${robot_namespace}" topics_ns="camera" depth_optical_frame="camera_depth_optical_frame" color_optical_frame="camera_color_optical_frame" infrared1_optical_frame="camera_left_ir_optical_frame" infrared2_optical_frame="camera_right_ir_optical_frame" publish_pointcloud="true"/>
 		<!-- Set Gazebo material for the base -->
-		<gazebo reference="${tf_prefix}base_link">
+		<gazebo reference="base_link">
 			<material>Gazebo/LightGrey</material>
 		</gazebo>
 		<!-- Set gazebo material for the wheels -->
-		<xacro:actuated_wheel_gazebo tf_prefix="${tf_prefix}" locationprefix="left"/>
-		<xacro:actuated_wheel_gazebo tf_prefix="${tf_prefix}" locationprefix="right"/>
-		<xacro:caster_wheel_gazebo tf_prefix="${tf_prefix}" locationprefix="fl"/>
-		<xacro:caster_wheel_gazebo tf_prefix="${tf_prefix}" locationprefix="fr"/>
-		<xacro:caster_wheel_gazebo tf_prefix="${tf_prefix}" locationprefix="bl"/>
-		<xacro:caster_wheel_gazebo tf_prefix="${tf_prefix}" locationprefix="br"/>
+		<xacro:actuated_wheel_gazebo locationprefix="left"/>
+		<xacro:actuated_wheel_gazebo locationprefix="right"/>
+		<xacro:caster_wheel_gazebo locationprefix="fl"/>
+		<xacro:caster_wheel_gazebo locationprefix="fr"/>
+		<xacro:caster_wheel_gazebo locationprefix="bl"/>
+		<xacro:caster_wheel_gazebo locationprefix="br"/>
 		<!-- Settings for the IMU of the robot to work in the simulation environment-->
-		<xacro:imu_gazebo link="${tf_prefix}imu_link" robot_namespace="${robot_namespace}" imu_topic="imu_data" update_rate="50.0" standard_deviation="${imu_standard_deviation}" />
+		<xacro:imu_gazebo link="imu_link" robot_namespace="${robot_namespace}" imu_topic="imu_data" update_rate="50.0" standard_deviation="${imu_standard_deviation}" />
 		<!--  -->
 		<!-- <p3d_base_controller tf_prefix="${tf_prefix}" /> -->
 		<!-- Add Gazebo xacro for the laser scanner to work in Gazebo -->
 		<!-- Please match there macro calls with the sick_s300 xacro calls in the mir_200.urdf.xacro file-->
-		<xacro:sick_s300_gazebo tf_prefix="${tf_prefix}" link="front_laser_link" robot_namespace="${robot_namespace}" topic="f_scan" />
-		<xacro:sick_s300_gazebo tf_prefix="${tf_prefix}" link="back_laser_link" robot_namespace="${robot_namespace}" topic="b_scan" />
+		<xacro:sick_s300_gazebo link="front_laser_link" robot_namespace="${robot_namespace}" topic="f_scan" />
+		<xacro:sick_s300_gazebo link="back_laser_link" robot_namespace="${robot_namespace}" topic="b_scan" />
 		<!-- Add transmissions to wheels -->
-		<xacro:mir_200_wheel_transmissions tf_prefix="${tf_prefix}"/>
+		<xacro:mir_200_wheel_transmissions/>
 		<!-- disabled, because it doesn't make a difference in Gazebo: -->
 		<!-- <xacro:set_all_wheel_frictions tf_prefix="${tf_prefix}"/> -->

File: mir/mir_description/urdf/mir_200/mir_200_wheels.gazebo.xacro (robot description, xacro)
@@ -1,24 +1,24 @@
 <?xml version="1.0"?>
 <robot xmlns:xacro="http://ros.org/wiki/xacro">
-	<xacro:macro name="actuated_wheel_gazebo" params="tf_prefix locationprefix">
-		<gazebo reference="${tf_prefix}${locationprefix}_wheel_link">
+	<xacro:macro name="actuated_wheel_gazebo" params="locationprefix">
+		<gazebo reference="${locationprefix}_wheel_link">
 			<material>Gazebo/DarkGrey</material>
 		</gazebo>
 	</xacro:macro>
-	<xacro:macro name="caster_wheel_gazebo" params="tf_prefix locationprefix">
-		<gazebo reference="${tf_prefix}${locationprefix}_caster_rotation_link">
+	<xacro:macro name="caster_wheel_gazebo" params="locationprefix">
+		<gazebo reference="${locationprefix}_caster_rotation_link">
 			<material>Gazebo/Grey</material>
 		</gazebo>
-		<gazebo reference="${tf_prefix}${locationprefix}_caster_wheel_link">
+		<gazebo reference="${locationprefix}_caster_wheel_link">
 			<material>Gazebo/DarkGrey</material>
 		</gazebo>
 	</xacro:macro>
-	<xacro:macro name="mir_200_wheel_transmission" params="tf_prefix locationprefix">
-		<transmission name="${tf_prefix}${locationprefix}_wheel_trans">
+	<xacro:macro name="mir_200_wheel_transmission" params="locationprefix">
+		<transmission name="${locationprefix}_wheel_trans">
 		<type>transmission_interface/SimpleTransmission</type>
-		<joint name="${tf_prefix}${locationprefix}_wheel_joint">
+		<joint name="${locationprefix}_wheel_joint">
 			<hardwareInterface>hardware_interface/VelocityJointInterface</hardwareInterface>
 		</joint>
-		<actuator name="${tf_prefix}${locationprefix}_wheel_motor">
+		<actuator name="${locationprefix}_wheel_motor">
 			<hardwareInterface>hardware_interface/VelocityJointInterface</hardwareInterface>
 			<mechanicalReduction>1</mechanicalReduction>
@@ -26,7 +26,7 @@
 		</transmission>
 	</xacro:macro>
-	<xacro:macro name="mir_200_wheel_transmissions" params="tf_prefix">
-		<xacro:mir_200_wheel_transmission tf_prefix="${tf_prefix}" locationprefix="left"/>
-		<xacro:mir_200_wheel_transmission tf_prefix="${tf_prefix}" locationprefix="right"/>
+	<xacro:macro name="mir_200_wheel_transmissions" params="">
+		<xacro:mir_200_wheel_transmission locationprefix="left"/>
+		<xacro:mir_200_wheel_transmission locationprefix="right"/>
 	</xacro:macro>
 </robot>

Commit message: fixed missing tf_prefix under noetic

File: mir/mir_description/urdf/general/sick_s300.gazebo.xacro (robot description, xacro)
@@ -2,5 +2,5 @@
 <robot xmlns:xacro="http://ros.org/wiki/xacro">
 	<xacro:include filename="$(find mir_description)/urdf/general/common_properties.urdf.xacro" />
-	<xacro:macro name="sick_s300_gazebo" params="link topic robot_namespace">
+	<xacro:macro name="sick_s300_gazebo" params="link topic robot_namespace tf_prefix">
 		<gazebo reference="${link}">
 			<xacro:insert_block name="material_black" />
@@ -35,5 +35,5 @@
 					<!-- no tf_prefix, plugin always uses a tf_prefix (if none is set it uses robotNamespace) -->
 					<robotNamespace>${robot_namespace}</robotNamespace>
-					<frameName>${link}</frameName>
+					<frameName>${tf_prefix}${link}</frameName>
 					<topicName>${topic}</topicName>
 				</plugin>

File: mir/mir_description/urdf/mir_100/mir_100.gazebo.xacro (robot description, xacro)
@@ -44,6 +44,6 @@
 		<!-- Add Gazebo xacro for the laser scanner to work in Gazebo -->
 		<!-- Please match there macro calls with the sick_s300 xacro calls in the mir_100.urdf.xacro file-->
-		<xacro:sick_s300_gazebo link="front_laser_link" robot_namespace="${robot_namespace_slashed}" topic="f_scan" />
-		<xacro:sick_s300_gazebo link="back_laser_link" robot_namespace="${robot_namespace_slashed}" topic="b_scan" />
+		<xacro:sick_s300_gazebo link="front_laser_link" robot_namespace="${robot_namespace_slashed}" topic="f_scan" tf_prefix="{tf_prefix_slashed}" />
+		<xacro:sick_s300_gazebo link="back_laser_link" robot_namespace="${robot_namespace_slashed}" topic="b_scan" tf_prefix="{tf_prefix_slashed}"/>
 		<!-- Settings for the camera of the robot to work in the simulation environment-->
     	<xacro:gazebo_d435 camera_name="${robot_namespace_underscored}camera" reference_link="camera_link" topics_ns="${robot_namespace_slashed}camera" depth_optical_frame="${tf_prefix_slashed}camera_depth_optical_frame" color_optical_frame="${tf_prefix_slashed}camera_color_optical_frame" infrared1_optical_frame="${tf_prefix_slashed}camera_left_ir_optical_frame" infrared2_optical_frame="${tf_prefix_slashed}camera_right_ir_optical_frame" publish_pointcloud="true"/>

File: mir/mir_description/urdf/mir_200/mir_200.gazebo.xacro (robot description, xacro)
@@ -44,6 +44,6 @@
 		<!-- Add Gazebo xacro for the laser scanner to work in Gazebo -->
 		<!-- Please match there macro calls with the sick_s300 xacro calls in the mir_200.urdf.xacro file-->
-		<xacro:sick_s300_gazebo link="front_laser_link" robot_namespace="${robot_namespace_slashed}" topic="f_scan" />
-		<xacro:sick_s300_gazebo link="back_laser_link" robot_namespace="${robot_namespace_slashed}" topic="b_scan" />
+		<xacro:sick_s300_gazebo link="front_laser_link" robot_namespace="${robot_namespace_slashed}" topic="f_scan" tf_prefix="${tf_prefix_slashed}"/>
+		<xacro:sick_s300_gazebo link="back_laser_link" robot_namespace="${robot_namespace_slashed}" topic="b_scan" tf_prefix="${tf_prefix_slashed}"/>
 		<!-- Settings for the camera of the robot to work in the simulation environment-->
     	<xacro:gazebo_d435 camera_name="${robot_namespace_underscored}camera" reference_link="camera_link" topics_ns="${robot_namespace_slashed}camera" depth_optical_frame="${tf_prefix_slashed}camera_depth_optical_frame" color_optical_frame="${tf_prefix_slashed}camera_color_optical_frame" infrared1_optical_frame="${tf_prefix_slashed}camera_left_ir_optical_frame" infrared2_optical_frame="${tf_prefix_slashed}camera_right_ir_optical_frame" publish_pointcloud="true"/>
