Commit message: Reworked MuR205 and got it working - Deleted tf_prefix from mir_200.urdf - Reimplemented mur_205.gazebo.urdf - Updated ur_robot and ur_ros_driver - Created package for examples with mur205 - Implemented first mur_205 example - reworked mur.launch as it didnt work - Adjusted all moveit files to new repo

File: mur/mur_description/urdf/mur_205.gazebo.urdf (robot description, URDF)
Before this commit: robot mur205, 0 links, 1 joints
Joints:
- joint plattform_manipulator_joint: child ur/base_link -> UR5/base_link; parent mir/base_link -> base_link
