Commit message: moved gripper to seperate package

File: mur/mur_description/urdf/mur_620.gazebo.xacro (robot description, xacro)
@@ -13,5 +13,5 @@
 	<xacro:p3d_base_controller robot_namespace="$(arg robot_namespace)"/>
 	<!-- include gripper -->
-	<xacro:include filename="$(find mur_description)/urdf/inc/schunk_emh_rp_045.urdf.xacro"/>
+	<xacro:include filename="$(find schunk_emh_rp_45)/urdf/schunk_emh_rp_045.urdf.xacro"/>
 	<!-- Init the MiR200 marco that is also used for the hardware -->
 	<xacro:mir_600 />

File: tools/schunk_emh_rp_45/urdf/schunk_emh_rp_045.urdf.xacro (robot description, xacro)
@@ -11,5 +11,5 @@
 				<origin xyz="0 0 0.128" rpy="${-pi * 0.5} 0 0" />
 				<geometry>
-					<mesh filename="package://mur_description/meshes/visual/schunk_emh_rp_045.stl" scale="0.001 0.001 0.001"/>
+					<mesh filename="package://schunk_emh_rp_45/meshes/visual/schunk_emh_rp_045.stl" scale="0.001 0.001 0.001"/>
 				</geometry>
 				<xacro:insert_block name="material_white" />
@@ -18,5 +18,5 @@
 				<origin xyz="0 0 0" rpy="0 0 0" />
 				<geometry>
-					<mesh filename="package://mur_description/meshes/collision/schunk_emh_rp_045.stl" scale="0.001 0.001 0.001" />
+					<mesh filename="package://schunk_emh_rp_45/meshes/collision/schunk_emh_rp_045.stl" scale="0.001 0.001 0.001" />
 				</geometry>
 			</collision>

Commit message: hw working with moveit

File: mur/mur_description/urdf/mur_620.gazebo.xacro (robot description, xacro)
@@ -5,4 +5,6 @@
 	<xacro:arg name="use_lift" default='true'/>
 	<xacro:property name="use_lift" value="$(arg use_lift)"/>
+	<xacro:arg name="sim" default='true'/>
+	<xacro:property name="sim" value="$(arg sim)"/>
 	<!-- MiR200 base -->
 	<xacro:include filename="$(find mir_description)/urdf/mir_600/mir_600.urdf.xacro" />
@@ -17,5 +19,7 @@
 	<xacro:p3d_base_controller robot_namespace="$(arg robot_namespace)"/>
 	<!-- include gripper -->
-	<xacro:include filename="$(find schunk_emh_rp_45)/urdf/schunk_emh_rp_045.urdf.xacro"/>
+	<xacro:if value="${sim}">
+		<xacro:include filename="$(find schunk_emh_rp_45)/urdf/schunk_emh_rp_045.urdf.xacro"/>
+	</xacro:if>
 	<!-- Init the MiR200 marco that is also used for the hardware -->
 	<xacro:mir_600 />
@@ -23,8 +27,8 @@
 	<xacro:mir_600_gazebo tf_prefix="$(arg tf_prefix)" robot_namespace="$(arg robot_namespace)"/>
 	<!-- Init the UR5 robot arm macro -->
-	<!-- <xacro:ur10e_robot prefix="UR10_l/" transmission_hw_interface="hardware_interface/VelocityJointInterface"/>
-	<xacro:ur10e_robot prefix="UR10_r/" transmission_hw_interface="hardware_interface/VelocityJointInterface"/> -->
-	<xacro:ur10e_robot prefix="UR10_l/" transmission_hw_interface="hardware_interface/PositionJointInterface"/>
-	<xacro:ur10e_robot prefix="UR10_r/" transmission_hw_interface="hardware_interface/PositionJointInterface"/>
+	<xacro:ur10e_robot prefix="UR10_l/" transmission_hw_interface="hardware_interface/VelocityJointInterface"/>
+	<xacro:ur10e_robot prefix="UR10_r/" transmission_hw_interface="hardware_interface/VelocityJointInterface"/>
+	<!-- <xacro:ur10e_robot prefix="UR10_l/" transmission_hw_interface="hardware_interface/PositionJointInterface"/>
+	<xacro:ur10e_robot prefix="UR10_r/" transmission_hw_interface="hardware_interface/PositionJointInterface"/> -->
 	<!-- Init the plugins that run the MiR in Gazebo -->
 	<xacro:controller_plugin_gazebo robot_namespace="$(arg robot_namespace)"/>
@@ -40,5 +44,5 @@
 				<parent link="right_lift_top" />
 				<child link="UR10_r/base_link" />
-				<origin xyz="0.0 0.0 0.555" rpy="0 0 0" />
+				<origin xyz="0.0 0.0 0.555" rpy="0 0 3.14159265" />
 		</joint>
 	</xacro:if>
@@ -55,6 +59,8 @@
 		</joint>
 	</xacro:unless>
-	<xacro:schunk_emh_rp_045 tf_prefix="UR10_r"	tool_link="UR10_r/flange"/>
-	<xacro:schunk_emh_rp_045 tf_prefix="UR10_l"	tool_link="UR10_l/flange"/>
+	<xacro:if value="${sim}">
+		<xacro:schunk_emh_rp_045 tf_prefix="UR10_r"	tool_link="UR10_r/flange"/>
+		<xacro:schunk_emh_rp_045 tf_prefix="UR10_l"	tool_link="UR10_l/flange"/>
+	</xacro:if>
 	<!-- <gazebo>
 		<plugin name="gazebo_ros_control" filename="libgazebo_ros_control.so">

Commit message: add frame base_ideal to have same rotation as mir (and for calibration purposes)

File: mur/mur_description/urdf/mur_620.gazebo.xacro (robot description, xacro)
@@ -33,4 +33,7 @@
 	<!-- Init the plugins that run the MiR in Gazebo -->
 	<xacro:controller_plugin_gazebo robot_namespace="$(arg robot_namespace)"/>
+	<!-- virtual link rotated to show in same direction like mir  -->
+	<link name="UR10_l/base_ideal" />
+	<link name="UR10_r/base_ideal" />
 	<!-- Init the lift macro -->
 	<xacro:if value="${use_lift}">
@@ -38,11 +41,11 @@
 		<joint name="plattform_manipulator_joint_l" type="fixed">
 				<parent link="left_lift_top" />
-				<child link="UR10_l/base_link" />
+				<child link="UR10_l/base_ideal" />
 				<origin xyz="0.0 0.0 0.555" rpy="0 0 0" />
 		</joint>
 		<joint name="plattform_manipulator_joint_r" type="fixed">
 				<parent link="right_lift_top" />
-				<child link="UR10_r/base_link" />
-				<origin xyz="0.0 0.0 0.555" rpy="0 0 3.14159265" />
+				<child link="UR10_r/base_ideal" />
+				<origin xyz="0.0 0.0 0.555" rpy="0 0 0" />
 		</joint>
 	</xacro:if>
@@ -50,13 +53,24 @@
 		<joint name="plattform_manipulator_joint_l" type="fixed">
 			<parent link="left_lift_bottom" />
-			<child link="UR10_l/base_link" />
+			<child link="UR10_l/base_ideal" />
 			<origin xyz="0.0 0.0 0.555" rpy="0 0 0" />
 		</joint>
 		<joint name="plattform_manipulator_joint_r" type="fixed">
 			<parent link="right_lift_bottom" />
-			<child link="UR10_r/base_link" />
-			<origin xyz="0.0 0.0 0.555" rpy="0 0 3.14159265" />
+			<child link="UR10_r/base_ideal" />
+			<origin xyz="0.0 0.0 0.555" rpy="0 0 0" />
 		</joint>
 	</xacro:unless>
+	<!-- Because one arm is mounted backwards. TODO: use calibrated pose -->
+	<joint name="plattform_ur_calibration_joint_l" type="fixed">
+			<parent link="UR10_l/base_ideal" />
+			<child link="UR10_l/base_link" />
+			<origin xyz="0.0 0.0 0.0" rpy="0 0 0" />
+	</joint>
+	<joint name="plattform_ur_calibration_joint_r" type="fixed">
+			<parent link="UR10_r/base_ideal" />
+			<child link="UR10_r/base_link" />
+			<origin xyz="0.0 0.0 0.0" rpy="0 0 3.14159265" />
+	</joint>
 	<xacro:if value="${sim}">
 		<xacro:schunk_emh_rp_045 tf_prefix="UR10_r"	tool_link="UR10_r/flange"/>

Commit message: added args to change cailbrated pose

File: mur/mur_description/urdf/mur_620.gazebo.xacro (robot description, xacro)
@@ -7,4 +7,12 @@
 	<xacro:arg name="sim" default='true'/>
 	<xacro:property name="sim" value="$(arg sim)"/>
+	<xacro:arg name="ur_l_xyz" default='0 0 0'/>
+	<xacro:arg name="ur_l_rpy" default='0 0 0'/>
+	<xacro:property name="ur_l_xyz" value="$(arg ur_l_xyz)"/>
+	<xacro:property name="ur_l_rpy" value="$(arg ur_l_rpy)"/>
+	<xacro:arg name="ur_r_xyz" default='0 0 0'/>
+	<xacro:arg name="ur_r_rpy" default='0 0 0'/>
+	<xacro:property name="ur_r_xyz" value="$(arg ur_r_xyz)"/>
+	<xacro:property name="ur_r_rpy" value="$(arg ur_r_rpy)"/>
 	<!-- MiR200 base -->
 	<xacro:include filename="$(find mir_description)/urdf/mir_600/mir_600.urdf.xacro" />
@@ -66,10 +74,10 @@
 			<parent link="UR10_l/base_ideal" />
 			<child link="UR10_l/base_link" />
-			<origin xyz="0.0 0.0 0.0" rpy="0 0 0" />
+			<origin xyz="${ur_l_xyz}" rpy="${ur_l_rpy}" /> <!-- 0 0 0" -->
 	</joint>
 	<joint name="plattform_ur_calibration_joint_r" type="fixed">
 			<parent link="UR10_r/base_ideal" />
 			<child link="UR10_r/base_link" />
-			<origin xyz="0.0 0.0 0.0" rpy="0 0 3.14159265" />
+			<origin xyz="${ur_r_xyz}" rpy="${ur_r_rpy}" /> <!-- 0 0 3.14159265" -->
 	</joint>
 	<xacro:if value="${sim}">

Commit message: Refactor bauschaum_ee integration: update URDF and launch files, add collision mesh, and adjust localization settings

File: mur/mur_description/urdf/mur_620.gazebo.xacro (robot description, xacro)
@@ -33,6 +33,9 @@
 		<xacro:include filename="$(find schunk_emh_rp_45)/urdf/schunk_emh_rp_045.urdf.xacro"/>
 		<xacro:include filename="$(find keyence_lj_x)/urdf/keyence_lj_x.urdf.xacro"/>
+		<xacro:include filename="$(find bauschaum_ee)/urdf/bauschaum_ee.urdf.gazebo.xacro"/>
+	</xacro:if>
+	<xacro:unless value="${sim}">
 		<xacro:include filename="$(find bauschaum_ee)/urdf/bauschaum_ee.urdf.xacro"/>
-	</xacro:if>
+	</xacro:unless>
 	<!-- Init the MiR200 marco that is also used for the hardware -->
 	<xacro:mir_600 />
@@ -86,17 +89,15 @@
 			<origin xyz="${ur_r_xyz}" rpy="${ur_r_rpy}" /> <!-- 0 0 3.14159265" -->
 	</joint>
-	<xacro:if value="${sim}">
-		<xacro:if value="${tool == 'schunk_emh_rp_045'}">
-			<xacro:schunk_emh_rp_045 tf_prefix="UR10_r"	tool_link="UR10_r/flange"/>
-			<xacro:schunk_emh_rp_045 tf_prefix="UR10_l"	tool_link="UR10_l/flange"/>
-		</xacro:if>
-		<xacro:if value="${tool == 'keyence_line_laser'}">
-			<xacro:keyence_lj_x tf_prefix="UR10_r"	tool_link="UR10_r/flange"/>
-			<xacro:keyence_lj_x tf_prefix="UR10_l"	tool_link="UR10_l/flange"/>
-		</xacro:if>
-		<xacro:if value="${tool == 'bauschaum_ee'}">
-			<xacro:bauschaum_ee tf_prefix="UR10_r"	tool_link="UR10_r/flange"/>
-			<xacro:bauschaum_ee  tf_prefix="UR10_l"	tool_link="UR10_l/flange"/>
-		</xacro:if>
+	<xacro:if value="${tool == 'schunk_emh_rp_045'}">
+		<xacro:schunk_emh_rp_045 tf_prefix="UR10_r"	tool_link="UR10_r/flange"/>
+		<xacro:schunk_emh_rp_045 tf_prefix="UR10_l"	tool_link="UR10_l/flange"/>
+	</xacro:if>
+	<xacro:if value="${tool == 'keyence_line_laser'}">
+		<xacro:keyence_lj_x tf_prefix="UR10_r"	tool_link="UR10_r/flange"/>
+		<xacro:keyence_lj_x tf_prefix="UR10_l"	tool_link="UR10_l/flange"/>
+	</xacro:if>
+	<xacro:if value="${tool == 'bauschaum_ee'}">
+		<xacro:bauschaum_ee tf_prefix="UR10_r"	tool_link="UR10_r/tool0"/>
+		<xacro:bauschaum_ee  tf_prefix="UR10_l"	tool_link="UR10_l/tool0"/>
 	</xacro:if>
     <!-- <xacro:include filename="$(find print_sim)/urdf/keyence_line_laser.gazebo.xacro" />

File: mur/mur_moveit_config/config/mur620.srdf.xacro (robot description, xacro)
@@ -109,4 +109,6 @@
     <passive_joint name="fr_caster_rotation_joint" />
     <passive_joint name="fr_caster_wheel_joint" />
+    <passive_joint name="$(arg prefix)_l/gripper_joint"/>
+    <passive_joint name="$(arg prefix)_r/gripper_joint"/>
     <!--GROUP STATES: Purpose: Define a named state for a particular group, in terms of joint values. This is useful to define states like 'folded arms'-->
     <group_state name="Home_custom" group="UR_arm_l">
@@ -229,8 +231,8 @@
     </group_state>
     <!--END EFFECTOR: Purpose: Represent information about an end effector.-->
-    <end_effector name="hand_l" parent_link="$(arg prefix)_l/tool0" group="UR_arm_l"/>
-	<end_effector name="hand_r" parent_link="$(arg prefix)_r/tool0" group="UR_arm_r"/>
-	<end_effector name="hand_l_both" parent_link="$(arg prefix)_l/tool0" group="UR_arm_both"/>
-	<end_effector name="hand_r_both" parent_link="$(arg prefix)_r/tool0" group="UR_arm_both"/>
+    <end_effector name="hand_l" parent_link="$(arg prefix)_l/gripper" group="UR_arm_l"/>
+	<end_effector name="hand_r" parent_link="$(arg prefix)_r/gripper" group="UR_arm_r"/>
+	<end_effector name="hand_l_both" parent_link="$(arg prefix)_l/gripper" group="UR_arm_both"/>
+	<end_effector name="hand_r_both" parent_link="$(arg prefix)_r/gripper" group="UR_arm_both"/>
     <!--DISABLE COLLISIONS: By default it is assumed that any link of the robot could potentially come into collision with any other link in the robot. This tag disables collision checking between a specified pair of links. -->
 	<disable_collisions link1="$(arg prefix)_l/base_link_inertia" link2="$(arg prefix)_l/shoulder_link" reason="Adjacent"/>

File: tools/bauschaum_ee/urdf/bauschaum_ee.urdf.gazebo.xacro (robot description, xacro)
@@ -26,11 +26,8 @@
 				<xacro:insert_block name="material_white" />
 			</visual>
-			<collision>
-				<origin xyz="0.0 0.0 0" rpy="0 ${pi * 0.5} ${pi * 0.0}" />
-				<geometry>
-					<mesh filename="package://bauschaum_ee/meshes/collision/bauschaum_ee.stl" scale="0.001 0.001 0.001"/>
-				</geometry>
-			</collision>
 		</link>
+		<gazebo reference="${tf_prefix}/tcp">
+			<material>Gazebo/DarkGrey</material>
+		</gazebo>
 		<!-- the ft_sensor plugin will not work with fixed joints. This is why a prismatic joint with very small limits is added -->
 		<joint name="${tf_prefix}/tcp_joint" type="prismatic">
@@ -41,4 +38,43 @@
    			<limit effort="1000" lower="-0.0001" upper="0.0001" velocity="10"/>
 		</joint>
+		<!-- Gazebo Plugin for Line Laser -->
+		<gazebo reference="${tf_prefix}/gripper">
+			<sensor type="ray" name="line_laser">
+			<pose>0 0 0 0.0 0 0</pose>
+			<visualize>true</visualize>
+			<update_rate>20.0</update_rate>
+			<ray>
+				<scan>
+				<!-- Horizontal range parameters -->
+				<horizontal>
+					<samples>1000</samples> <!-- Number of laser beams -->
+					<resolution>1</resolution>
+					<min_angle>-0.27317277996474193</min_angle> <!-- Start angle in radians -->
+					<max_angle>0.27317277996474193</max_angle> <!-- End angle in radians -->
+				</horizontal>
+				<!-- Vertical range parameters (set min and max equal for a line) -->
+				<vertical>
+					<samples>1</samples> <!-- Single vertical beam -->
+					<min_angle>0.0</min_angle>
+					<max_angle>0.0</max_angle>
+				</vertical>
+				</scan>
+				<range>
+				<min>0.285</min> <!-- Minimum range in meters -->
+				<max>0.600</max> <!-- Maximum range in meters -->
+				<resolution>0.0001707329874779637</resolution> <!-- Range resolution -->
+				</range>
+				<noise>
+				<type>gaussian</type>
+				<mean>0.00005</mean>
+				<stddev>0.0005</stddev>
+				</noise>
+			</ray>
+			<plugin name="gazebo_ros_laser" filename="libgazebo_ros_laser.so">
+				<topicName>${tf_prefix}/line_laser/scan</topicName> <!-- ROS topic -->
+				<frameName>mur620a/${tf_prefix}/gripper</frameName> <!-- Frame for the laser -->
+			</plugin>
+			</sensor>
+		</gazebo>
 	</xacro:macro>
 </robot>
