Commit message: corrected mesh path

File: general_hardware_helper/keyence_scanner/urdf/7200.urdf (robot description, URDF)
Before this commit: robot myfirst, 1 links, 0 joints
Links:
- link sensor_frame: geometry collision mesh filename=package://keyence_scanner/meshes/collision/lj_v7200.stl; visual mesh filename=package://keyence_scanner/meshes/visual/lj_v7200.dae
