Commit message: Split the files in differernt folders Started splitting hw and sim (gazebo) parts Started removing unnecessary descriptions

File: mir/mir_description/urdf/mir_100/mir_100.gazebo.xacro (robot description, xacro)
@@ -1,5 +1,5 @@
 <?xml version="1.0"?>
 <robot xmlns:xacro="http://ros.org/wiki/xacro">
-  <xacro:macro name="diff_controller_plugin_gazebo" params="prefix left_wheel_joint right_wheel_joint wheel_separation wheel_radius">
+  <!-- <xacro:macro name="diff_controller_plugin_gazebo" params="prefix left_wheel_joint right_wheel_joint wheel_separation wheel_radius">
     <gazebo>
       <plugin name="diff_drive_controller" filename="libgazebo_ros_diff_drive.so">
@@ -24,5 +24,5 @@
       </plugin>
     </gazebo>
-  </xacro:macro>
+  </xacro:macro> -->
   <xacro:macro name="set_wheel_friction" params="link friction">
     <gazebo reference="${link}">
@@ -41,5 +41,5 @@
     <xacro:set_wheel_friction link="${prefix}br_caster_wheel_link" friction="1"/>
   </xacro:macro>
-  <xacro:macro name="p3d_base_controller" params="prefix">
+  <!-- <xacro:macro name="p3d_base_controller" params="prefix">
     <gazebo>
       <plugin name="p3d_base_controller" filename="libgazebo_ros_p3d.so">
@@ -54,27 +54,4 @@
       </plugin>
     </gazebo>
-  </xacro:macro>
-    <!-- camera -->
-    <gazebo reference="camera_link">
-      <sensor type="depth" name="camera">
-        <plugin name="kinect_camera_controller" filename="libgazebo_ros_openni_kinect.so">
-          <cameraName>camera</cameraName>
-          <alwaysOn>true</alwaysOn>
-          <updateRate>10</updateRate>
-          <imageTopicName>rgb/image_raw</imageTopicName>
-          <depthImageTopicName>depth/image_raw</depthImageTopicName>
-          <pointCloudTopicName>depth/points</pointCloudTopicName>
-          <cameraInfoTopicName>rgb/camera_info</cameraInfoTopicName>
-          <depthImageCameraInfoTopicName>depth/camera_info</depthImageCameraInfoTopicName>
-          <frameName>camera_link_optical</frameName>
-          <baseline>0.1</baseline>
-          <distortion_k1>0.0</distortion_k1>
-          <distortion_k2>0.0</distortion_k2>
-          <distortion_k3>0.0</distortion_k3>
-          <distortion_t1>0.0</distortion_t1>
-          <distortion_t2>0.0</distortion_t2>
-          <pointCloudCutoff>0.4</pointCloudCutoff>
-        </plugin>
-      </sensor>
-    </gazebo>
+  </xacro:macro> -->
 </robot>

File: mir/mir_description/urdf/mir_200/mir_200.gazebo.xacro (robot description, xacro)
@@ -1,5 +1,5 @@
 <?xml version="1.0"?>
 <robot xmlns:xacro="http://ros.org/wiki/xacro">
-  <xacro:macro name="diff_controller_plugin_gazebo" params="prefix left_wheel_joint right_wheel_joint wheel_separation wheel_radius">
+  <!-- <xacro:macro name="diff_controller_plugin_gazebo" params="prefix left_wheel_joint right_wheel_joint wheel_separation wheel_radius">
     <gazebo>
       <plugin name="diff_drive_controller" filename="libgazebo_ros_diff_drive.so">
@@ -24,5 +24,5 @@
       </plugin>
     </gazebo>
-  </xacro:macro>
+  </xacro:macro> -->
   <xacro:macro name="set_wheel_friction" params="link friction">
     <gazebo reference="${link}">
@@ -41,5 +41,5 @@
     <xacro:set_wheel_friction link="${prefix}br_caster_wheel_link" friction="1"/>
   </xacro:macro>
-  <xacro:macro name="p3d_base_controller" params="prefix">
+  <!-- <xacro:macro name="p3d_base_controller" params="prefix">
     <gazebo>
       <plugin name="p3d_base_controller" filename="libgazebo_ros_p3d.so">
@@ -54,4 +54,27 @@
       </plugin>
     </gazebo>
-  </xacro:macro>
+  </xacro:macro> -->
+    <!-- camera -->
+    <gazebo reference="camera_link">
+      <sensor type="depth" name="camera">
+        <plugin name="kinect_camera_controller" filename="libgazebo_ros_openni_kinect.so">
+          <cameraName>camera</cameraName>
+          <alwaysOn>true</alwaysOn>
+          <updateRate>10</updateRate>
+          <imageTopicName>rgb/image_raw</imageTopicName>
+          <depthImageTopicName>depth/image_raw</depthImageTopicName>
+          <pointCloudTopicName>depth/points</pointCloudTopicName>
+          <cameraInfoTopicName>rgb/camera_info</cameraInfoTopicName>
+          <depthImageCameraInfoTopicName>depth/camera_info</depthImageCameraInfoTopicName>
+          <frameName>camera_link_optical</frameName>
+          <baseline>0.1</baseline>
+          <distortion_k1>0.0</distortion_k1>
+          <distortion_k2>0.0</distortion_k2>
+          <distortion_k3>0.0</distortion_k3>
+          <distortion_t1>0.0</distortion_t1>
+          <distortion_t2>0.0</distortion_t2>
+          <pointCloudCutoff>0.4</pointCloudCutoff>
+        </plugin>
+      </sensor>
+    </gazebo>
 </robot>

Commit message: Added separate launch files for the MiR100 and MiR200 Started separating the MiR100 from the gazebo parts

File: mir/mir_description/urdf/mir_100/mir_100.gazebo.xacro (robot description, xacro)
@@ -1,29 +1,36 @@
 <?xml version="1.0"?>
 <robot xmlns:xacro="http://ros.org/wiki/xacro">
-	<!-- This part of the file looks like it is not necessary for the correct function of the urdf files.-->
-	<!-- Remove this part in a second iteration when all functions are working like they are supposed to be-->
-	<!-- <xacro:macro name="diff_controller_plugin_gazebo" params="prefix left_wheel_joint right_wheel_joint wheel_separation wheel_radius">
-		<gazebo>
-			<plugin name="diff_drive_controller" filename="libgazebo_ros_diff_drive.so">
-				<legacyMode>false</legacyMode>
-				<alwaysOn>true</alwaysOn>
-				<updateRate>1000.0</updateRate>
-				<leftJoint>${left_wheel_joint}</leftJoint>
-				<rightJoint>${right_wheel_joint}</rightJoint>
-				<wheelSeparation>${wheel_separation}</wheelSeparation>
-				<wheelDiameter>${2*wheel_radius}</wheelDiameter>
-				<wheelTorque>10</wheelTorque>
-				<publishTf>1</publishTf>
-				<odometryFrame>map</odometryFrame>
-				<commandTopic>mobile_base_controller/cmd_vel</commandTopic>
-				<odometryTopic>mobile_base_controller/odom</odometryTopic>
-				<robotBaseFrame>base_footprint</robotBaseFrame>
-				<wheelAcceleration>2.8</wheelAcceleration>
-				<publishWheelJointState>true</publishWheelJointState>
-				<publishWheelTF>false</publishWheelTF>
-				<odometrySource>world</odometrySource>
-				<rosDebugLevel>Debug</rosDebugLevel>
-			</plugin>
+	<xacro:macro name="mir_100_gazebo" params="tf_prefix">
+		<!-- Set Gazebo material for the base -->
+		<gazebo reference="${prefix}base_link">
+			<material>Gazebo/White</material>
 		</gazebo>
-	</xacro:macro> -->
+		<!-- Settings for the IMU of the robot to work in the simulation environment-->
+		<xacro:imu_gazebo link="${prefix}imu_link" imu_topic="imu_data" update_rate="50.0" stdev="${imu_stdev}" />
+		<!-- This part of the file looks like it is not necessary for the correct function of the urdf files.-->
+		<!-- Remove this part in a second iteration when all functions are working like they are supposed to be-->
+		<!-- <xacro:macro name="diff_controller_plugin_gazebo" params="prefix left_wheel_joint right_wheel_joint wheel_separation wheel_radius">
+			<gazebo>
+				<plugin name="diff_drive_controller" filename="libgazebo_ros_diff_drive.so">
+					<legacyMode>false</legacyMode>
+					<alwaysOn>true</alwaysOn>
+					<updateRate>1000.0</updateRate>
+					<leftJoint>${left_wheel_joint}</leftJoint>
+					<rightJoint>${right_wheel_joint}</rightJoint>
+					<wheelSeparation>${wheel_separation}</wheelSeparation>
+					<wheelDiameter>${2*wheel_radius}</wheelDiameter>
+					<wheelTorque>10</wheelTorque>
+					<publishTf>1</publishTf>
+					<odometryFrame>map</odometryFrame>
+					<commandTopic>mobile_base_controller/cmd_vel</commandTopic>
+					<odometryTopic>mobile_base_controller/odom</odometryTopic>
+					<robotBaseFrame>base_footprint</robotBaseFrame>
+					<wheelAcceleration>2.8</wheelAcceleration>
+					<publishWheelJointState>true</publishWheelJointState>
+					<publishWheelTF>false</publishWheelTF>
+					<odometrySource>world</odometrySource>
+					<rosDebugLevel>Debug</rosDebugLevel>
+				</plugin>
+			</gazebo>
+		</xacro:macro> -->
 </robot>

File: mir/mir_description/urdf/mir_100/mir_100.urdf.xacro (robot description, xacro)
@@ -32,24 +32,21 @@
 		</joint>
 		<link name="${prefix}base_link">
-		<xacro:box_inertial mass="${mir_100_base_mass}" x="0.9" y="0.58" z="0.3">
-			<origin xyz="${mir_100_act_wheel_dx} 0 0.20" rpy="0 0 0" />
-		</xacro:box_inertial>
-		<visual>
-			<origin xyz="${mir_100_act_wheel_dx} 0 0" rpy="0 0 0" />
-			<geometry>
-				<mesh filename="package://mir_description/meshes/visual/mir_100_base.stl" />
-			</geometry>
-			<xacro:insert_block name="material_white" />
-		</visual>
-		<collision>
-			<origin xyz="${mir_100_act_wheel_dx} 0 0" rpy="0 0 0" />
-			<geometry>
-				<mesh filename="package://mir_description/meshes/collision/mir_100_base.stl" />
-			</geometry>
-		</collision>
+			<xacro:box_inertial mass="${mir_100_base_mass}" x="0.9" y="0.58" z="0.3">
+				<origin xyz="${mir_100_act_wheel_dx} 0 0.20" rpy="0 0 0" />
+			</xacro:box_inertial>
+			<visual>
+				<origin xyz="${mir_100_act_wheel_dx} 0 0" rpy="0 0 0" />
+				<geometry>
+					<mesh filename="package://mir_description/meshes/visual/mir_100_base.stl" />
+				</geometry>
+				<xacro:insert_block name="material_white" />
+			</visual>
+			<collision>
+				<origin xyz="${mir_100_act_wheel_dx} 0 0" rpy="0 0 0" />
+				<geometry>
+					<mesh filename="package://mir_description/meshes/collision/mir_100_base.stl" />
+				</geometry>
+			</collision>
 		</link>
-			<gazebo reference="${prefix}base_link">
-			<material>Gazebo/White</material>
-		</gazebo>
 		<!-- IMU -->
 		<joint name="${prefix}base_link_to_imu_joint" type="fixed">
@@ -59,5 +56,4 @@
 		</joint>
 		<link name="${prefix}imu_link" />
-		<xacro:imu_gazebo link="${prefix}imu_link" imu_topic="imu_data" update_rate="50.0" stdev="${imu_stdev}" />
 		<!-- Create an alias for imu_link. This is necessary because the real MiR's
 			TF has imu_link, but the imu_data topic is published in the imu_frame

File: mir/mir_description/urdf/mir_200/mir_200.gazebo.xacro (robot description, xacro)
@@ -1,5 +1,4 @@
 <?xml version="1.0"?>
 <robot xmlns:xacro="http://wiki.ros.org/xacro">
-	<!-- <xacro:include filename="$(find mir_description)/urdf/mir_200/mir_200.urdf.xacro" /> -->
 	<xacro:include filename="$(find mir_description)/urdf/mir_200/mir_200_wheels.gazebo.xacro" />
 	<xacro:include filename="$(find mir_description)/urdf/general/sick_s300.gazebo.xacro" />
@@ -7,6 +6,4 @@
 	<xacro:property name="imu_standard_deviation" value="0.00017" />
 	<xacro:macro name="mir_200_gazebo" params="tf_prefix">
-		<!-- Call MiR200 xacro to get base robot model loaded-->
-		<!-- <xacro:mir_200 tf_prefix="${tf_prefix}"> -->
 		<!-- Settings for the camera of the robot to work in the simulation environment-->
 		<gazebo reference="camera_link">
