Commit message: More separation of MiR100 urdf.xacro and gazebo.xacro

File: mir/mir_description/urdf/mir_100/mir_100.gazebo.xacro (robot description, xacro)
@@ -1,4 +1,6 @@
 <?xml version="1.0"?>
 <robot xmlns:xacro="http://ros.org/wiki/xacro">
+	<xacro:include filename="$(find mir_description)/urdf/general/imu.gazebo.xacro" />
+	<xacro:property name="imu_standard_deviation" value="0.00017" />
 	<xacro:macro name="mir_100_gazebo" params="tf_prefix">
 		<!-- Set Gazebo material for the base -->
@@ -7,7 +9,17 @@
 		</gazebo>
 		<!-- Settings for the IMU of the robot to work in the simulation environment-->
-		<xacro:imu_gazebo link="${prefix}imu_link" imu_topic="imu_data" update_rate="50.0" stdev="${imu_stdev}" />
+		<xacro:imu_gazebo link="${tf_prefix}imu_link" imu_topic="imu_data" update_rate="50.0" standard_deviation="${imu_standard_deviation}" />
+		<p3d_base_controller prefix="${prefix}" />
+		<!-- wheels -->
+		<xacro:actuated_wheel_gazebo tf_prefix="${tf_prefix}" locationprefix="left"/>
+		<xacro:actuated_wheel_gazebo tf_prefix="${tf_prefix}" locationprefix="right"/>
+		<xacro:caster_wheel_gazebo tf_prefix="${tf_prefix}" locationprefix="fl"/>
+		<xacro:caster_wheel_gazebo tf_prefix="${tf_prefix}" locationprefix="fr"/>
+		<xacro:caster_wheel_gazebo tf_prefix="${tf_prefix}" locationprefix="bl"/>
+		<xacro:caster_wheel_gazebo tf_prefix="${tf_prefix}" locationprefix="br"/>
 		<!-- This part of the file looks like it is not necessary for the correct function of the urdf files.-->
 		<!-- Remove this part in a second iteration when all functions are working like they are supposed to be-->
+		<!-- disabled, because it doesn't make a difference in Gazebo: -->
+		<!-- <xacro:set_all_wheel_frictions prefix="${prefix}"/> -->
 		<!-- <xacro:macro name="diff_controller_plugin_gazebo" params="prefix left_wheel_joint right_wheel_joint wheel_separation wheel_radius">
 			<gazebo>

File: mir/mir_description/urdf/mir_100/mir_100.urdf.xacro (robot description, xacro)
@@ -2,9 +2,7 @@
 <robot xmlns:xacro="http://ros.org/wiki/xacro">
 	<xacro:include filename="$(find mir_description)/urdf/include/common_properties.urdf.xacro" />
-	<xacro:include filename="$(find mir_description)/urdf/include/imu.gazebo.urdf.xacro" />
-	<xacro:include filename="$(find mir_description)/urdf/include/mir_100.gazebo.xacro" />
-	<xacro:include filename="$(find mir_description)/urdf/include/mir_100.transmission.xacro" />
+	<xacro:include filename="$(find mir_description)/urdf/mir_100/mir_100_wheels.urdf.xacro" />
 	<xacro:include filename="$(find mir_description)/urdf/include/sick_s300.urdf.xacro" />
-	<xacro:property name="deg_to_rad" value="0.017453293" />
+	<xacro:property name="deg_to_rad" value="${(1 / 360) * (2 * pi)}" />
 	<xacro:property name="mir_100_base_mass" value="58.0" />
 	<xacro:property name="mir_100_act_wheel_radius" value="0.0625" />
@@ -23,13 +21,12 @@
 	<xacro:property name="mir_100_caster_wheel_base_dy" value="0.203" />
 	<xacro:property name="mir_100_caster_wheel_base_dz" value="${mir_100_caster_wheel_radius-mir_100_caster_wheel_dz}" />
-	<xacro:property name="imu_stdev" value="0.00017" />
-	<xacro:macro name="mir_100" params="prefix">
-		<link name="${prefix}base_footprint" />
-		<joint name="${prefix}base_joint" type="fixed">
-			<parent link="${prefix}base_footprint" />
-			<child link="${prefix}base_link" />
+	<xacro:macro name="mir_100" params="tf_prefix">
+		<link name="${tf_prefix}base_footprint" />
+		<joint name="${tf_prefix}base_joint" type="fixed">
+			<parent link="${tf_prefix}base_footprint" />
+			<child link="${tf_prefix}base_link" />
 			<origin xyz="0 0 0" rpy="0 0 0" />
 		</joint>
-		<link name="${prefix}base_link">
+		<link name="${tf_prefix}base_link">
 			<xacro:box_inertial mass="${mir_100_base_mass}" x="0.9" y="0.58" z="0.3">
 				<origin xyz="${mir_100_act_wheel_dx} 0 0.20" rpy="0 0 0" />
@@ -50,63 +47,60 @@
 		</link>
 		<!-- IMU -->
-		<joint name="${prefix}base_link_to_imu_joint" type="fixed">
-			<parent link="${prefix}base_link" />
-			<child link="${prefix}imu_link" />
+		<joint name="${tf_prefix}base_link_to_imu_joint" type="fixed">
+			<parent link="${tf_prefix}base_link" />
+			<child link="${tf_prefix}imu_link" />
 			<origin xyz="0.0 0.0 0.25" rpy="0 0 0" />  <!-- same as real MiR -->
 		</joint>
-		<link name="${prefix}imu_link" />
+		<link name="${tf_prefix}imu_link" />
 		<!-- Create an alias for imu_link. This is necessary because the real MiR's
 			TF has imu_link, but the imu_data topic is published in the imu_frame
 			frame. -->
-		<joint name="${prefix}imu_link_to_imu_frame_joint" type="fixed">
-			<parent link="${prefix}imu_link" />
-			<child link="${prefix}imu_frame" />
+		<joint name="${tf_prefix}imu_link_to_imu_frame_joint" type="fixed">
+			<parent link="${tf_prefix}imu_link" />
+			<child link="${tf_prefix}imu_frame" />
 			<origin xyz="0 0 0" rpy="0 0 0" />
 		</joint>
-		<link name="${prefix}imu_frame" />
+		<link name="${tf_prefix}imu_frame" />
 		<!-- Laser scanners -->
-		<joint name="${prefix}base_link_to_front_laser_joint" type="fixed">
-			<parent link="${prefix}base_link" />
-			<child link="${prefix}front_laser_link" />
+		<joint name="${tf_prefix}base_link_to_front_laser_joint" type="fixed">
+			<parent link="${tf_prefix}base_link" />
+			<child link="${tf_prefix}front_laser_link" />
 			<origin xyz="0.4288 0.2358 0.1914" rpy="0.0 0.0 ${0.25 * pi}" />  <!-- from visually matching up the meshes of the MiR and the laser scanner -->
 		</joint>
-		<xacro:sick_s300 prefix="${prefix}" link="front_laser_link" topic="f_scan" />
-		<joint name="${prefix}base_link_to_back_laser_joint" type="fixed">
-			<parent link="${prefix}base_link" />
-			<child link="${prefix}back_laser_link" />
+		<xacro:sick_s300 tf_prefix="${tf_prefix}" link="front_laser_link" topic="f_scan" />
+		<joint name="${tf_prefix}base_link_to_back_laser_joint" type="fixed">
+			<parent link="${tf_prefix}base_link" />
+			<child link="${tf_prefix}back_laser_link" />
 			<origin xyz="-0.3548 -0.2352 0.1914" rpy="0.0 0.0 ${-0.75 * pi}" />  <!-- from visually matching up the meshes of the MiR and the laser scanner -->
 		</joint>
-		<xacro:sick_s300 prefix="${prefix}" link="back_laser_link" topic="b_scan" />
+		<xacro:sick_s300 tf_prefix="${tf_prefix}" link="back_laser_link" topic="b_scan" />
 		<!-- Ultrasound sensors -->
-		<joint name="${prefix}us_1_joint" type="fixed">   <!-- right ultrasound -->
-			<parent link="${prefix}base_link" />
-			<child link="${prefix}us_1_frame" />
+		<joint name="${tf_prefix}us_1_joint" type="fixed">   <!-- right ultrasound -->
+			<parent link="${tf_prefix}base_link" />
+			<child link="${tf_prefix}us_1_frame" />
 			<origin xyz="0.45 -0.12 0.16 " rpy="0 0 0" />  <!-- from visually matching to the mesh of the MiR -->
 		</joint>
-		<link name="${prefix}us_1_frame" />
-		<joint name="${prefix}us_2_joint" type="fixed">   <!-- left ultrasound -->
-			<parent link="${prefix}base_link" />
-			<child link="${prefix}us_2_frame" />
+		<link name="${tf_prefix}us_1_frame" />
+		<joint name="${tf_prefix}us_2_joint" type="fixed">   <!-- left ultrasound -->
+			<parent link="${tf_prefix}base_link" />
+			<child link="${tf_prefix}us_2_frame" />
 			<origin xyz="0.45 0.12 0.16 " rpy="0 0 0" />  <!-- from visually matching to the mesh of the MiR -->
 		</joint>
-		<link name="${prefix}us_2_frame" />
+		<link name="${tf_prefix}us_2_frame" />
 		<!-- wheels -->
-		<xacro:actuated_wheel prefix="${prefix}" locationprefix="left" locationright="-1"/>
-		<xacro:actuated_wheel prefix="${prefix}" locationprefix="right" locationright="1"/>
-		<xacro:caster_wheel prefix="${prefix}" locationprefix="fl" locationright="-1" wheel_base_dx="${mir_100_front_caster_wheel_base_dx}"/>
-		<xacro:caster_wheel prefix="${prefix}" locationprefix="fr" locationright="1" wheel_base_dx="${mir_100_front_caster_wheel_base_dx}"/>
-		<xacro:caster_wheel prefix="${prefix}" locationprefix="bl" locationright="-1" wheel_base_dx="${mir_100_back_caster_wheel_base_dx}"/>
-		<xacro:caster_wheel prefix="${prefix}" locationprefix="br" locationright="1" wheel_base_dx="${mir_100_back_caster_wheel_base_dx}"/>
-		<joint name="${prefix}base_link_surface_joint" type="fixed">
+		<xacro:actuated_wheel tf_prefix="${tf_prefix}" locationprefix="left" locationright="-1"/>
+		<xacro:actuated_wheel tf_prefix="${tf_prefix}" locationprefix="right" locationright="1"/>
+		<xacro:caster_wheel tf_prefix="${tf_prefix}" locationprefix="fl" locationright="-1" wheel_base_dx="${mir_100_front_caster_wheel_base_dx}"/>
+		<xacro:caster_wheel tf_prefix="${tf_prefix}" locationprefix="fr" locationright="1" wheel_base_dx="${mir_100_front_caster_wheel_base_dx}"/>
+		<xacro:caster_wheel tf_prefix="${tf_prefix}" locationprefix="bl" locationright="-1" wheel_base_dx="${mir_100_back_caster_wheel_base_dx}"/>
+		<xacro:caster_wheel tf_prefix="${tf_prefix}" locationprefix="br" locationright="1" wheel_base_dx="${mir_100_back_caster_wheel_base_dx}"/>
+		<joint name="${tf_prefix}base_link_surface_joint" type="fixed">
 			<origin xyz="${mir_100_act_wheel_dx} 0 0.352" rpy="0 0 0" />
-			<parent link="${prefix}base_link" />
-			<child link="${prefix}surface" />
+			<parent link="${tf_prefix}base_link" />
+			<child link="${tf_prefix}surface" />
 			<axis xyz="0 0 1" />
 		</joint>
-		<link name="${prefix}surface"/>
-		<xacro:mir_100_wheel_transmissions prefix="${prefix}"/>
-		<!-- disabled, because it doesn't make a difference in Gazebo: -->
-		<!-- <xacro:set_all_wheel_frictions prefix="${prefix}"/> -->
-		<p3d_base_controller prefix="${prefix}" />
+		<link name="${tf_prefix}surface"/>
+		<xacro:mir_100_wheel_transmissions tf_prefix="${tf_prefix}"/>
 	</xacro:macro>
 </robot>

File: mir/mir_description/urdf/mir_100/mir_100_wheels.urdf.xacro (robot description, xacro)
@@ -1,13 +1,13 @@
 <?xml version="1.0"?>
 <robot xmlns:xacro="http://ros.org/wiki/xacro">
-	<xacro:macro name="actuated_wheel" params="prefix locationprefix locationright">
-		<joint name="${prefix}${locationprefix}_wheel_joint" type="continuous">
+	<xacro:macro name="actuated_wheel" params="tf_prefix locationprefix locationright">
+		<joint name="${tf_prefix}${locationprefix}_wheel_joint" type="continuous">
 		<origin xyz="0.0 ${-mir_100_act_wheel_dy * locationright} ${mir_100_act_wheel_radius}" rpy="0 0 0" />
-		<parent link="${prefix}base_link" />
-		<child link="${prefix}${locationprefix}_wheel_link" />
+		<parent link="${tf_prefix}base_link" />
+		<child link="${tf_prefix}${locationprefix}_wheel_link" />
 		<axis xyz="0 1 0" />
 		<limit effort="100" velocity="20.0" />
 		</joint>
-		<link name="${prefix}${locationprefix}_wheel_link">
+		<link name="${tf_prefix}${locationprefix}_wheel_link">
 		<xacro:cylinder_inertial mass="${mir_100_act_wheel_mass}" radius="${mir_100_act_wheel_radius}" length="${mir_100_act_wheel_width}">
 			<origin xyz="0 0 0" rpy="${0.5 * pi} 0 0" />
@@ -27,18 +27,18 @@
 		</collision>
 		</link>
-		<gazebo reference="${prefix}${locationprefix}_wheel_link">
+		<gazebo reference="${tf_prefix}${locationprefix}_wheel_link">
 		<material>Gazebo/DarkGrey</material>
 		</gazebo>
 	</xacro:macro>
-	<xacro:macro name="caster_wheel" params="prefix locationprefix locationright wheel_base_dx">
+	<xacro:macro name="caster_wheel" params="tf_prefix locationprefix locationright wheel_base_dx">
 		<!-- caster hub -->
-		<joint name="${prefix}${locationprefix}_caster_rotation_joint" type="continuous">
+		<joint name="${tf_prefix}${locationprefix}_caster_rotation_joint" type="continuous">
 		<origin xyz="${wheel_base_dx} ${-mir_100_caster_wheel_base_dy * locationright} ${mir_100_caster_wheel_base_dz}" rpy="0 0 0" />
-		<parent link="${prefix}base_link" />
-		<child link="${prefix}${locationprefix}_caster_rotation_link" />
+		<parent link="${tf_prefix}base_link" />
+		<child link="${tf_prefix}${locationprefix}_caster_rotation_link" />
 		<axis xyz="0 0 1" />
 		<dynamics damping="0.01" friction="0.0"/>
 		</joint>
-		<link name="${prefix}${locationprefix}_caster_rotation_link">
+		<link name="${tf_prefix}${locationprefix}_caster_rotation_link">
 		<inertial>
 			<!-- <origin xyz="0 0 -0.042500000044" rpy="${0.5 * pi} ${24 * deg_to_rad} ${1.5 * pi}" /> -->
@@ -67,15 +67,15 @@
 		</collision>
 		</link>
-		<gazebo reference="${prefix}${locationprefix}_caster_rotation_link">
+		<gazebo reference="${tf_prefix}${locationprefix}_caster_rotation_link">
 		<material>Gazebo/Grey</material>
 		</gazebo>
 		<!-- caster wheel -->
-		<joint name="${prefix}${locationprefix}_caster_wheel_joint" type="continuous">
+		<joint name="${tf_prefix}${locationprefix}_caster_wheel_joint" type="continuous">
 		<origin xyz="${mir_100_caster_wheel_dx} ${-mir_100_caster_wheel_dy * locationright} ${mir_100_caster_wheel_dz}" rpy="0 0 0" />
-		<parent link="${prefix}${locationprefix}_caster_rotation_link" />
-		<child link="${prefix}${locationprefix}_caster_wheel_link" />
+		<parent link="${tf_prefix}${locationprefix}_caster_rotation_link" />
+		<child link="${tf_prefix}${locationprefix}_caster_wheel_link" />
 		<axis xyz="0 1 0" />
 		</joint>
-		<link name="${prefix}${locationprefix}_caster_wheel_link">
+		<link name="${tf_prefix}${locationprefix}_caster_wheel_link">
 		<xacro:cylinder_inertial mass="${mir_100_caster_wheel_mass}" radius="${mir_100_caster_wheel_radius}" length="${mir_100_caster_wheel_width}">
 			<origin xyz="0 0 0" rpy="${0.5 * pi} 0 0" />
@@ -95,15 +95,15 @@
 		</collision>
 		</link>
-		<gazebo reference="${prefix}${locationprefix}_caster_wheel_link">
+		<gazebo reference="${tf_prefix}${locationprefix}_caster_wheel_link">
 		<material>Gazebo/DarkGrey</material>
 		</gazebo>
 	</xacro:macro>
-	<xacro:macro name="mir_100_wheel_transmission" params="prefix locationprefix">
-		<transmission name="${prefix}${locationprefix}_wheel_trans">
+	<xacro:macro name="mir_100_wheel_transmission" params="tf_prefix locationprefix">
+		<transmission name="${tf_prefix}${locationprefix}_wheel_trans">
 			<type>transmission_interface/SimpleTransmission</type>
-			<joint name="${prefix}${locationprefix}_wheel_joint">
+			<joint name="${tf_prefix}${locationprefix}_wheel_joint">
 				<hardwareInterface>hardware_interface/VelocityJointInterface</hardwareInterface>
 			</joint>
-			<actuator name="${prefix}${locationprefix}_wheel_motor">
+			<actuator name="${tf_prefix}${locationprefix}_wheel_motor">
 				<hardwareInterface>hardware_interface/VelocityJointInterface</hardwareInterface>
 				<mechanicalReduction>1</mechanicalReduction>
@@ -111,7 +111,7 @@
 		</transmission>
 	</xacro:macro>
-	<xacro:macro name="mir_100_wheel_transmissions" params="prefix">
-		<xacro:mir_100_wheel_transmission prefix="${prefix}" locationprefix="left"/>
-		<xacro:mir_100_wheel_transmission prefix="${prefix}" locationprefix="right"/>
+	<xacro:macro name="mir_100_wheel_transmissions" params="tf_prefix">
+		<xacro:mir_100_wheel_transmission tf_prefix="${tf_prefix}" locationprefix="left"/>
+		<xacro:mir_100_wheel_transmission tf_prefix="${tf_prefix}" locationprefix="right"/>
 	</xacro:macro>
 </robot>
