Commit message: Finished MiR100 files to be usable and complete - Renamed MiR200 stl for naming conventions - Removed tf_prefix from all MiR100 files - Added mir100 gazebo urdf info - copied new code from mir200 gazebo xacro to mir100 - Added sick300, new camera and match logo to mir100 - Refactored mir200 xacro file - Added single mir 100 launch and multi mir 100 launch example - Added mir_100.launch in mir_launch_sim for easy spawning of a robot

File: mir/mir_description/urdf/mir_100/mir_100.gazebo.xacro (robot description, xacro)
@@ -1,26 +1,51 @@
 <?xml version="1.0"?>
-<robot xmlns:xacro="http://ros.org/wiki/xacro">
+<robot xmlns:xacro="http://wiki.ros.org/xacro">
+	<xacro:include filename="$(find mir_description)/urdf/mir_100/mir_100_wheels.gazebo.xacro" />
+	<xacro:include filename="$(find mir_description)/urdf/general/sick_s300.gazebo.xacro" />
 	<xacro:include filename="$(find mir_description)/urdf/general/imu.gazebo.xacro" />
-	<xacro:include filename="$(find mir_description)/urdf/general/sick_s300.gazebo.xacro" />
+	<xacro:include filename="$(find mir_description)/urdf/general/plugins.gazebo.xacro" />
+	<xacro:include filename="$(find mir_description)/urdf/general/_d435.gazebo.xacro" />
 	<xacro:property name="imu_standard_deviation" value="0.00017" />
-	<xacro:macro name="mir_100_gazebo" params="tf_prefix">
+	<xacro:macro name="mir_100_gazebo" params="tf_prefix robot_namespace">
+		<!-- Predefine some values that are necessary later. It is important to differenciate between empty and not empty robot_namespace and tf_prefix -->
+		<xacro:if value="${robot_namespace == ''}">
+			<xacro:property name="robot_namespace_slashed" value="/" />
+		</xacro:if>
+		<xacro:unless value="${robot_namespace == ''}">
+				<xacro:property name="robot_namespace_slashed" value="${robot_namespace}/" />
+		</xacro:unless>
+		<xacro:if value="${tf_prefix == ''}">
+			<xacro:property name="tf_prefix_slashed" value="" />
+		</xacro:if>
+		<xacro:unless value="${tf_prefix == ''}">
+				<xacro:property name="tf_prefix_slashed" value="${tf_prefix}/" />
+		</xacro:unless>
+		<xacro:if value="${robot_namespace == ''}">
+			<xacro:property name="robot_namespace_underscored" value="" />
+		</xacro:if>
+		<xacro:unless value="${robot_namespace == ''}">
+				<xacro:property name="robot_namespace_underscored" value="${robot_namespace}_" />
+		</xacro:unless>
 		<!-- Set Gazebo material for the base -->
-		<gazebo reference="${tf_prefix}base_link">
+		<gazebo reference="base_link">
 			<material>Gazebo/White</material>
 		</gazebo>
+		<!-- Set gazebo material for the wheels -->
+		<xacro:actuated_wheel_gazebo locationprefix="left"/>
+		<xacro:actuated_wheel_gazebo locationprefix="right"/>
+		<xacro:caster_wheel_gazebo locationprefix="fl"/>
+		<xacro:caster_wheel_gazebo locationprefix="fr"/>
+		<xacro:caster_wheel_gazebo locationprefix="bl"/>
+		<xacro:caster_wheel_gazebo locationprefix="br"/>
+		<!-- Add transmissions to wheels -->
+		<xacro:mir_100_wheel_transmissions/>
 		<!-- Settings for the IMU of the robot to work in the simulation environment-->
-		<xacro:imu_gazebo link="${tf_prefix}imu_link" imu_topic="imu_data" update_rate="50.0" standard_deviation="${imu_standard_deviation}" />
-		<p3d_base_controller prefix="${tf_prefix}" />
-		<!-- wheels -->
-		<xacro:actuated_wheel_gazebo tf_prefix="${tf_prefix}" locationprefix="left"/>
-		<xacro:actuated_wheel_gazebo tf_prefix="${tf_prefix}" locationprefix="right"/>
-		<xacro:caster_wheel_gazebo tf_prefix="${tf_prefix}" locationprefix="fl"/>
-		<xacro:caster_wheel_gazebo tf_prefix="${tf_prefix}" locationprefix="fr"/>
-		<xacro:caster_wheel_gazebo tf_prefix="${tf_prefix}" locationprefix="bl"/>
-		<xacro:caster_wheel_gazebo tf_prefix="${tf_prefix}" locationprefix="br"/>
-		<!-- Add Gazebo xacro for the laser scanner to work in Gazebo-->
-		<!-- Please match there macro calls with the sick_s300 xacro calls in the mir_200.urdf.xacro file-->
-		<xacro:sick_s300_gazebo tf_prefix="${tf_prefix}" link="front_laser_link" topic="f_scan"/>
-		<xacro:sick_s300_gazebo tf_prefix="${tf_prefix}" link="back_laser_link" topic="b_scan"/>
+		<xacro:imu_gazebo link="imu_link" robot_namespace="${robot_namespace_slashed}" imu_topic="imu_data" update_rate="50.0" standard_deviation="${imu_standard_deviation}" />
+		<!-- Add Gazebo xacro for the laser scanner to work in Gazebo -->
+		<!-- Please match there macro calls with the sick_s300 xacro calls in the mir_100.urdf.xacro file-->
+		<xacro:sick_s300_gazebo link="front_laser_link" robot_namespace="${robot_namespace_slashed}" topic="f_scan" />
+		<xacro:sick_s300_gazebo link="back_laser_link" robot_namespace="${robot_namespace_slashed}" topic="b_scan" />
+		<!-- Settings for the camera of the robot to work in the simulation environment-->
+    	<xacro:gazebo_d435 camera_name="${robot_namespace_underscored}camera" reference_link="camera_link" topics_ns="${robot_namespace_slashed}camera" depth_optical_frame="${tf_prefix_slashed}camera_depth_optical_frame" color_optical_frame="${tf_prefix_slashed}camera_color_optical_frame" infrared1_optical_frame="${tf_prefix_slashed}camera_left_ir_optical_frame" infrared2_optical_frame="${tf_prefix_slashed}camera_right_ir_optical_frame" publish_pointcloud="true"/>
 		<!-- This part of the file looks like it is not necessary for the correct function of the urdf files.-->
 		<!-- Remove this part in a second iteration when all functions are working like they are supposed to be-->
@@ -28,26 +53,27 @@
 		<!-- <xacro:set_all_wheel_frictions prefix="${prefix}"/> -->
 		<!-- <xacro:macro name="diff_controller_plugin_gazebo" params="prefix left_wheel_joint right_wheel_joint wheel_separation wheel_radius">
-			<gazebo>
-				<plugin name="diff_drive_controller" filename="libgazebo_ros_diff_drive.so">
-					<legacyMode>false</legacyMode>
-					<alwaysOn>true</alwaysOn>
-					<updateRate>1000.0</updateRate>
-					<leftJoint>${left_wheel_joint}</leftJoint>
-					<rightJoint>${right_wheel_joint}</rightJoint>
-					<wheelSeparation>${wheel_separation}</wheelSeparation>
-					<wheelDiameter>${2*wheel_radius}</wheelDiameter>
-					<wheelTorque>10</wheelTorque>
-					<publishTf>1</publishTf>
-					<odometryFrame>map</odometryFrame>
-					<commandTopic>mobile_base_controller/cmd_vel</commandTopic>
-					<odometryTopic>mobile_base_controller/odom</odometryTopic>
-					<robotBaseFrame>base_footprint</robotBaseFrame>
-					<wheelAcceleration>2.8</wheelAcceleration>
-					<publishWheelJointState>true</publishWheelJointState>
-					<publishWheelTF>false</publishWheelTF>
-					<odometrySource>world</odometrySource>
-					<rosDebugLevel>Debug</rosDebugLevel>
-				</plugin>
-			</gazebo-->
+		<gazebo>
+			<plugin name="diff_drive_controller" filename="libgazebo_ros_diff_drive.so">
+				<legacyMode>false</legacyMode>
+				<alwaysOn>true</alwaysOn>
+				<updateRate>1000.0</updateRate>
+				<leftJoint>${left_wheel_joint}</leftJoint>
+				<rightJoint>${right_wheel_joint}</rightJoint>
+				<wheelSeparation>${wheel_separation}</wheelSeparation>
+				<wheelDiameter>${2*wheel_radius}</wheelDiameter>
+				<wheelTorque>10</wheelTorque>
+				<publishTf>1</publishTf>
+				<odometryFrame>map</odometryFrame>
+				<commandTopic>mobile_base_controller/cmd_vel</commandTopic>
+				<odometryTopic>mobile_base_controller/odom</odometryTopic>
+				<robotBaseFrame>base_footprint</robotBaseFrame>
+				<wheelAcceleration>2.8</wheelAcceleration>
+				<publishWheelJointState>true</publishWheelJointState>
+				<publishWheelTF>false</publishWheelTF>
+				<odometrySource>world</odometrySource>
+				<rosDebugLevel>Debug</rosDebugLevel>
+			</plugin>
+		</gazebo-->
+		<!-- <p3d_base_controller prefix="${tf_prefix}" /> -->
 	</xacro:macro>
 </robot>

File: mir/mir_description/urdf/mir_100/mir_100.urdf.xacro (robot description, xacro)
@@ -2,6 +2,8 @@
 <robot xmlns:xacro="http://ros.org/wiki/xacro">
 	<xacro:include filename="$(find mir_description)/urdf/general/common_properties.urdf.xacro" />
+	<xacro:include filename="$(find mir_description)/urdf/general/sick_s300.urdf.xacro" />
 	<xacro:include filename="$(find mir_description)/urdf/mir_100/mir_100_wheels.urdf.xacro" />
-	<xacro:include filename="$(find mir_description)/urdf/general/sick_s300.urdf.xacro" />
+	<xacro:include filename="$(find mir_description)/urdf/general/match_logo.urdf.xacro" />
+	<xacro:include filename="$(find realsense2_description)/urdf/_d435.urdf.xacro" />
 	<xacro:property name="deg_to_rad" value="${(1 / 360) * (2 * pi)}" />
 	<xacro:property name="mir_100_base_mass" value="58.0" />
@@ -21,12 +23,15 @@
 	<xacro:property name="mir_100_caster_wheel_base_dy" value="0.203" />
 	<xacro:property name="mir_100_caster_wheel_base_dz" value="${mir_100_caster_wheel_radius-mir_100_caster_wheel_dz}" />
-	<xacro:macro name="mir_100" params="tf_prefix">
-		<link name="${tf_prefix}base_footprint" />
-		<joint name="${tf_prefix}base_joint" type="fixed">
-			<parent link="${tf_prefix}base_footprint" />
-			<child link="${tf_prefix}base_link" />
+	<xacro:property name="mir_100_match_logo_dx" value="0.0" />
+	<xacro:property name="mir_100_match_logo_dy" value="0.2724435" />
+	<xacro:property name="mir_100_match_logo_dz" value="0.27" />
+	<xacro:macro name="mir_100">
+		<link name="base_footprint" />
+		<joint name="base_joint" type="fixed">
+			<parent link="base_footprint" />
+			<child link="base_link" />
 			<origin xyz="0 0 0" rpy="0 0 0" />
 		</joint>
-		<link name="${tf_prefix}base_link">
+		<link name="base_link">
 			<xacro:box_inertial mass="${mir_100_base_mass}" x="0.9" y="0.58" z="0.3">
 				<origin xyz="${mir_100_act_wheel_dx} 0 0.20" rpy="0 0 0" />
@@ -47,60 +52,66 @@
 		</link>
 		<!-- IMU -->
-		<joint name="${tf_prefix}base_link_to_imu_joint" type="fixed">
-			<parent link="${tf_prefix}base_link" />
-			<child link="${tf_prefix}imu_link" />
+		<joint name="base_link_to_imu_joint" type="fixed">
+			<parent link="base_link" />
+			<child link="imu_link" />
 			<origin xyz="0.0 0.0 0.25" rpy="0 0 0" />  <!-- same as real MiR -->
 		</joint>
-		<link name="${tf_prefix}imu_link" />
+		<link name="imu_link" />
 		<!-- Create an alias for imu_link. This is necessary because the real MiR's
 			TF has imu_link, but the imu_data topic is published in the imu_frame
 			frame. -->
-		<joint name="${tf_prefix}imu_link_to_imu_frame_joint" type="fixed">
-			<parent link="${tf_prefix}imu_link" />
-			<child link="${tf_prefix}imu_frame" />
+		<joint name="imu_link_to_imu_frame_joint" type="fixed">
+			<parent link="imu_link" />
+			<child link="imu_frame" />
 			<origin xyz="0 0 0" rpy="0 0 0" />
 		</joint>
-		<link name="${tf_prefix}imu_frame" />
+		<link name="imu_frame" />
 		<!-- Laser scanners -->
-		<joint name="${tf_prefix}base_link_to_front_laser_joint" type="fixed">
-			<parent link="${tf_prefix}base_link" />
-			<child link="${tf_prefix}front_laser_link" />
+		<joint name="base_link_to_front_laser_joint" type="fixed">
+			<parent link="base_link" />
+			<child link="front_laser_link" />
 			<origin xyz="0.4288 0.2358 0.1914" rpy="0.0 0.0 ${0.25 * pi}" />  <!-- from visually matching up the meshes of the MiR and the laser scanner -->
 		</joint>
-		<xacro:sick_s300 tf_prefix="${tf_prefix}" link="front_laser_link" topic="f_scan" />
-		<joint name="${tf_prefix}base_link_to_back_laser_joint" type="fixed">
-			<parent link="${tf_prefix}base_link" />
-			<child link="${tf_prefix}back_laser_link" />
+		<xacro:sick_s300 link="front_laser_link" topic="f_scan" />
+		<joint name="base_link_to_back_laser_joint" type="fixed">
+			<parent link="base_link" />
+			<child link="back_laser_link" />
 			<origin xyz="-0.3548 -0.2352 0.1914" rpy="0.0 0.0 ${-0.75 * pi}" />  <!-- from visually matching up the meshes of the MiR and the laser scanner -->
 		</joint>
-		<xacro:sick_s300 tf_prefix="${tf_prefix}" link="back_laser_link" topic="b_scan" />
+		<xacro:sick_s300 link="back_laser_link" topic="b_scan" />
 		<!-- Ultrasound sensors -->
-		<joint name="${tf_prefix}us_1_joint" type="fixed">   <!-- right ultrasound -->
-			<parent link="${tf_prefix}base_link" />
-			<child link="${tf_prefix}us_1_frame" />
+		<joint name="us_1_joint" type="fixed">   <!-- right ultrasound -->
+			<parent link="base_link" />
+			<child link="us_1_frame" />
 			<origin xyz="0.45 -0.12 0.16 " rpy="0 0 0" />  <!-- from visually matching to the mesh of the MiR -->
 		</joint>
-		<link name="${tf_prefix}us_1_frame" />
-		<joint name="${tf_prefix}us_2_joint" type="fixed">   <!-- left ultrasound -->
-			<parent link="${tf_prefix}base_link" />
-			<child link="${tf_prefix}us_2_frame" />
+		<link name="us_1_frame" />
+		<joint name="us_2_joint" type="fixed">   <!-- left ultrasound -->
+			<parent link="base_link" />
+			<child link="us_2_frame" />
 			<origin xyz="0.45 0.12 0.16 " rpy="0 0 0" />  <!-- from visually matching to the mesh of the MiR -->
 		</joint>
-		<link name="${tf_prefix}us_2_frame" />
+		<link name="us_2_frame" />
 		<!-- wheels -->
-		<xacro:actuated_wheel tf_prefix="${tf_prefix}" locationprefix="left" locationright="-1"/>
-		<xacro:actuated_wheel tf_prefix="${tf_prefix}" locationprefix="right" locationright="1"/>
-		<xacro:caster_wheel tf_prefix="${tf_prefix}" locationprefix="fl" locationright="-1" wheel_base_dx="${mir_100_front_caster_wheel_base_dx}"/>
-		<xacro:caster_wheel tf_prefix="${tf_prefix}" locationprefix="fr" locationright="1" wheel_base_dx="${mir_100_front_caster_wheel_base_dx}"/>
-		<xacro:caster_wheel tf_prefix="${tf_prefix}" locationprefix="bl" locationright="-1" wheel_base_dx="${mir_100_back_caster_wheel_base_dx}"/>
-		<xacro:caster_wheel tf_prefix="${tf_prefix}" locationprefix="br" locationright="1" wheel_base_dx="${mir_100_back_caster_wheel_base_dx}"/>
-		<joint name="${tf_prefix}base_link_surface_joint" type="fixed">
+		<xacro:actuated_wheel locationprefix="left" locationright="-1"/>
+		<xacro:actuated_wheel locationprefix="right" locationright="1"/>
+		<xacro:caster_wheel locationprefix="fl" locationright="-1" wheel_base_dx="${mir_100_front_caster_wheel_base_dx}"/>
+		<xacro:caster_wheel locationprefix="fr" locationright="1" wheel_base_dx="${mir_100_front_caster_wheel_base_dx}"/>
+		<xacro:caster_wheel locationprefix="bl" locationright="-1" wheel_base_dx="${mir_100_back_caster_wheel_base_dx}"/>
+		<xacro:caster_wheel locationprefix="br" locationright="1" wheel_base_dx="${mir_100_back_caster_wheel_base_dx}"/>
+		<joint name="base_link_surface_joint" type="fixed">
 			<origin xyz="${mir_100_act_wheel_dx} 0 0.352" rpy="0 0 0" />
-			<parent link="${tf_prefix}base_link" />
-			<child link="${tf_prefix}surface" />
+			<parent link="base_link" />
+			<child link="surface" />
 			<axis xyz="0 0 1" />
 		</joint>
-		<link name="${tf_prefix}surface"/>
-		<xacro:mir_100_wheel_transmissions tf_prefix="${tf_prefix}"/>
+		<link name="surface"/>
+		<!--Realsense_Intel_D435_Camera-->
+		<xacro:sensor_d435 name="camera" parent="base_link" use_nominal_extrinsics="true">
+    		<origin xyz="0.42 0 0.27" rpy="0 0 0" />
+  		</xacro:sensor_d435>
+		<!-- Insert a match logo on both sides of the mobile robot -->
+		<xacro:match_logo parent="base_link" locationprefix="left" location_dx="${mir_100_match_logo_dx}" location_dy="${mir_100_match_logo_dy}" location_dz="${mir_100_match_logo_dz}"/>
+		<xacro:match_logo parent="base_link" locationprefix="right" location_dx="${mir_100_match_logo_dx}" location_dy="${-1 * mir_100_match_logo_dy}" location_dz="${mir_100_match_logo_dz}" orientation="${pi}"/>
 	</xacro:macro>
 </robot>

File: mir/mir_description/urdf/mir_100/mir_100_wheels.gazebo.xacro (robot description, xacro)
@@ -1,14 +1,14 @@
 <?xml version="1.0"?>
 <robot xmlns:xacro="http://ros.org/wiki/xacro">
-	<xacro:macro name="actuated_wheel_gazebo" params="tf_prefix locationprefix">
-		<gazebo reference="${tf_prefix}${locationprefix}_wheel_link">
+	<xacro:macro name="actuated_wheel_gazebo" params="locationprefix">
+		<gazebo reference="${locationprefix}_wheel_link">
 			<material>Gazebo/DarkGrey</material>
 		</gazebo>
 	</xacro:macro>
-	<xacro:macro name="caster_wheel_gazebo" params="tf_prefix locationprefix">
-		<gazebo reference="${tf_prefix}${locationprefix}_caster_rotation_link">
+	<xacro:macro name="caster_wheel_gazebo" params="locationprefix">
+		<gazebo reference="${locationprefix}_caster_rotation_link">
 			<material>Gazebo/Grey</material>
 		</gazebo>
-		<gazebo reference="${tf_prefix}${locationprefix}_caster_wheel_link">
+		<gazebo reference="${locationprefix}_caster_wheel_link">
 			<material>Gazebo/DarkGrey</material>
 		</gazebo>

File: mir/mir_description/urdf/mir_100/mir_100_wheels.urdf.xacro (robot description, xacro)
@@ -1,13 +1,13 @@
 <?xml version="1.0"?>
 <robot xmlns:xacro="http://ros.org/wiki/xacro">
-	<xacro:macro name="actuated_wheel" params="tf_prefix locationprefix locationright">
-		<joint name="${tf_prefix}${locationprefix}_wheel_joint" type="continuous">
+	<xacro:macro name="actuated_wheel" params="locationprefix locationright">
+		<joint name="${locationprefix}_wheel_joint" type="continuous">
 		<origin xyz="0.0 ${-mir_100_act_wheel_dy * locationright} ${mir_100_act_wheel_radius}" rpy="0 0 0" />
-		<parent link="${tf_prefix}base_link" />
-		<child link="${tf_prefix}${locationprefix}_wheel_link" />
+		<parent link="base_link" />
+		<child link="${locationprefix}_wheel_link" />
 		<axis xyz="0 1 0" />
 		<limit effort="100" velocity="20.0" />
 		</joint>
-		<link name="${tf_prefix}${locationprefix}_wheel_link">
+		<link name="${locationprefix}_wheel_link">
 		<xacro:cylinder_inertial mass="${mir_100_act_wheel_mass}" radius="${mir_100_act_wheel_radius}" length="${mir_100_act_wheel_width}">
 			<origin xyz="0 0 0" rpy="${0.5 * pi} 0 0" />
@@ -27,18 +27,18 @@
 		</collision>
 		</link>
-		<gazebo reference="${tf_prefix}${locationprefix}_wheel_link">
+		<gazebo reference="${locationprefix}_wheel_link">
 		<material>Gazebo/DarkGrey</material>
 		</gazebo>
 	</xacro:macro>
-	<xacro:macro name="caster_wheel" params="tf_prefix locationprefix locationright wheel_base_dx">
+	<xacro:macro name="caster_wheel" params="locationprefix locationright wheel_base_dx">
 		<!-- caster hub -->
-		<joint name="${tf_prefix}${locationprefix}_caster_rotation_joint" type="continuous">
+		<joint name="${locationprefix}_caster_rotation_joint" type="continuous">
 		<origin xyz="${wheel_base_dx} ${-mir_100_caster_wheel_base_dy * locationright} ${mir_100_caster_wheel_base_dz}" rpy="0 0 0" />
-		<parent link="${tf_prefix}base_link" />
-		<child link="${tf_prefix}${locationprefix}_caster_rotation_link" />
+		<parent link="base_link" />
+		<child link="${locationprefix}_caster_rotation_link" />
 		<axis xyz="0 0 1" />
 		<dynamics damping="0.01" friction="0.0"/>
 		</joint>
-		<link name="${tf_prefix}${locationprefix}_caster_rotation_link">
+		<link name="${locationprefix}_caster_rotation_link">
 		<inertial>
 			<!-- <origin xyz="0 0 -0.042500000044" rpy="${0.5 * pi} ${24 * deg_to_rad} ${1.5 * pi}" /> -->
@@ -67,15 +67,15 @@
 		</collision>
 		</link>
-		<gazebo reference="${tf_prefix}${locationprefix}_caster_rotation_link">
+		<gazebo reference="${locationprefix}_caster_rotation_link">
 		<material>Gazebo/Grey</material>
 		</gazebo>
 		<!-- caster wheel -->
-		<joint name="${tf_prefix}${locationprefix}_caster_wheel_joint" type="continuous">
+		<joint name="${locationprefix}_caster_wheel_joint" type="continuous">
 		<origin xyz="${mir_100_caster_wheel_dx} ${-mir_100_caster_wheel_dy * locationright} ${mir_100_caster_wheel_dz}" rpy="0 0 0" />
-		<parent link="${tf_prefix}${locationprefix}_caster_rotation_link" />
-		<child link="${tf_prefix}${locationprefix}_caster_wheel_link" />
+		<parent link="${locationprefix}_caster_rotation_link" />
+		<child link="${locationprefix}_caster_wheel_link" />
 		<axis xyz="0 1 0" />
 		</joint>
-		<link name="${tf_prefix}${locationprefix}_caster_wheel_link">
+		<link name="${locationprefix}_caster_wheel_link">
 		<xacro:cylinder_inertial mass="${mir_100_caster_wheel_mass}" radius="${mir_100_caster_wheel_radius}" length="${mir_100_caster_wheel_width}">
 			<origin xyz="0 0 0" rpy="${0.5 * pi} 0 0" />
@@ -95,15 +95,15 @@
 		</collision>
 		</link>
-		<gazebo reference="${tf_prefix}${locationprefix}_caster_wheel_link">
+		<gazebo reference="${locationprefix}_caster_wheel_link">
 		<material>Gazebo/DarkGrey</material>
 		</gazebo>
 	</xacro:macro>
-	<xacro:macro name="mir_100_wheel_transmission" params="tf_prefix locationprefix">
-		<transmission name="${tf_prefix}${locationprefix}_wheel_trans">
+	<xacro:macro name="mir_100_wheel_transmission" params="locationprefix">
+		<transmission name="${locationprefix}_wheel_trans">
 			<type>transmission_interface/SimpleTransmission</type>
-			<joint name="${tf_prefix}${locationprefix}_wheel_joint">
+			<joint name="${locationprefix}_wheel_joint">
 				<hardwareInterface>hardware_interface/VelocityJointInterface</hardwareInterface>
 			</joint>
-			<actuator name="${tf_prefix}${locationprefix}_wheel_motor">
+			<actuator name="${locationprefix}_wheel_motor">
 				<hardwareInterface>hardware_interface/VelocityJointInterface</hardwareInterface>
 				<mechanicalReduction>1</mechanicalReduction>
@@ -111,7 +111,7 @@
 		</transmission>
 	</xacro:macro>
-	<xacro:macro name="mir_100_wheel_transmissions" params="tf_prefix">
-		<xacro:mir_100_wheel_transmission tf_prefix="${tf_prefix}" locationprefix="left"/>
-		<xacro:mir_100_wheel_transmission tf_prefix="${tf_prefix}" locationprefix="right"/>
+	<xacro:macro name="mir_100_wheel_transmissions">
+		<xacro:mir_100_wheel_transmission locationprefix="left"/>
+		<xacro:mir_100_wheel_transmission locationprefix="right"/>
 	</xacro:macro>
 </robot>
