Commit message: Finished MiR100 files to be usable and complete - Renamed MiR200 stl for naming conventions - Removed tf_prefix from all MiR100 files - Added mir100 gazebo urdf info - copied new code from mir200 gazebo xacro to mir100 - Added sick300, new camera and match logo to mir100 - Refactored mir200 xacro file - Added single mir 100 launch and multi mir 100 launch example - Added mir_100.launch in mir_launch_sim for easy spawning of a robot

File: mir/mir_description/urdf/mir_200/mir_200.gazebo.xacro (robot description, xacro)
@@ -27,9 +27,7 @@
 				<xacro:property name="robot_namespace_underscored" value="${robot_namespace}_" />
 		</xacro:unless>
-		<!-- Settings for the camera of the robot to work in the simulation environment-->
-    	<xacro:gazebo_d435 camera_name="${robot_namespace_underscored}camera" reference_link="camera_link" topics_ns="${robot_namespace_slashed}camera" depth_optical_frame="${tf_prefix_slashed}camera_depth_optical_frame" color_optical_frame="${tf_prefix_slashed}camera_color_optical_frame" infrared1_optical_frame="${tf_prefix_slashed}camera_left_ir_optical_frame" infrared2_optical_frame="${tf_prefix_slashed}camera_right_ir_optical_frame" publish_pointcloud="true"/>
 		<!-- Set Gazebo material for the base -->
 		<gazebo reference="base_link">
-			<material>Gazebo/LightGrey</material>
+			<material>Gazebo/Grey</material>
 		</gazebo>
 		<!-- Set gazebo material for the wheels -->
@@ -40,4 +38,6 @@
 		<xacro:caster_wheel_gazebo locationprefix="bl"/>
 		<xacro:caster_wheel_gazebo locationprefix="br"/>
+		<!-- Add transmissions to wheels -->
+		<xacro:mir_200_wheel_transmissions/>
 		<!-- Settings for the IMU of the robot to work in the simulation environment-->
 		<xacro:imu_gazebo link="imu_link" robot_namespace="${robot_namespace_slashed}" imu_topic="imu_data" update_rate="50.0" standard_deviation="${imu_standard_deviation}" />
@@ -46,6 +46,6 @@
 		<xacro:sick_s300_gazebo link="front_laser_link" robot_namespace="${robot_namespace_slashed}" topic="f_scan" />
 		<xacro:sick_s300_gazebo link="back_laser_link" robot_namespace="${robot_namespace_slashed}" topic="b_scan" />
-		<!-- Add transmissions to wheels -->
-		<xacro:mir_200_wheel_transmissions/>
+		<!-- Settings for the camera of the robot to work in the simulation environment-->
+    	<xacro:gazebo_d435 camera_name="${robot_namespace_underscored}camera" reference_link="camera_link" topics_ns="${robot_namespace_slashed}camera" depth_optical_frame="${tf_prefix_slashed}camera_depth_optical_frame" color_optical_frame="${tf_prefix_slashed}camera_color_optical_frame" infrared1_optical_frame="${tf_prefix_slashed}camera_left_ir_optical_frame" infrared2_optical_frame="${tf_prefix_slashed}camera_right_ir_optical_frame" publish_pointcloud="true"/>
 		<!-- disabled, because it doesn't make a difference in Gazebo: -->
 		<!-- <xacro:set_all_wheel_frictions tf_prefix="${tf_prefix}"/> -->

File: mir/mir_description/urdf/mir_200/mir_200.urdf.xacro (robot description, xacro)
@@ -40,5 +40,5 @@
 				<origin xyz="${mir_200_act_wheel_dx} 0 0" rpy="0 0 0" />
 				<geometry>
-					<mesh filename="package://mir_description/meshes/visual/MIR200_base.stl" />
+					<mesh filename="package://mir_description/meshes/visual/mir_200_base.stl" />
 				</geometry>
 				<xacro:insert_block name="material_white" />
@@ -47,5 +47,5 @@
 				<origin xyz="${mir_200_act_wheel_dx} 0 0" rpy="0 0 0" />
 				<geometry>
-					<mesh filename="package://mir_description/meshes/collision/MIR200_base.stl" />
+					<mesh filename="package://mir_description/meshes/collision/mir_200_base.stl" />
 				</geometry>
 			</collision>

Commit message: Removed commented code as the urdf compiler includes it somehow and produces an error

File: mir/mir_description/urdf/mir_100/mir_100.gazebo.xacro (robot description, xacro)
@@ -48,32 +48,4 @@
 		<!-- Settings for the camera of the robot to work in the simulation environment-->
     	<xacro:gazebo_d435 camera_name="${robot_namespace_underscored}camera" reference_link="camera_link" topics_ns="${robot_namespace_slashed}camera" depth_optical_frame="${tf_prefix_slashed}camera_depth_optical_frame" color_optical_frame="${tf_prefix_slashed}camera_color_optical_frame" infrared1_optical_frame="${tf_prefix_slashed}camera_left_ir_optical_frame" infrared2_optical_frame="${tf_prefix_slashed}camera_right_ir_optical_frame" publish_pointcloud="true"/>
-		<!-- This part of the file looks like it is not necessary for the correct function of the urdf files.-->
-		<!-- Remove this part in a second iteration when all functions are working like they are supposed to be-->
-		<!-- disabled, because it doesn't make a difference in Gazebo: -->
-		<!-- <xacro:set_all_wheel_frictions prefix="${prefix}"/> -->
-		<!-- <xacro:macro name="diff_controller_plugin_gazebo" params="prefix left_wheel_joint right_wheel_joint wheel_separation wheel_radius">
-		<gazebo>
-			<plugin name="diff_drive_controller" filename="libgazebo_ros_diff_drive.so">
-				<legacyMode>false</legacyMode>
-				<alwaysOn>true</alwaysOn>
-				<updateRate>1000.0</updateRate>
-				<leftJoint>${left_wheel_joint}</leftJoint>
-				<rightJoint>${right_wheel_joint}</rightJoint>
-				<wheelSeparation>${wheel_separation}</wheelSeparation>
-				<wheelDiameter>${2*wheel_radius}</wheelDiameter>
-				<wheelTorque>10</wheelTorque>
-				<publishTf>1</publishTf>
-				<odometryFrame>map</odometryFrame>
-				<commandTopic>mobile_base_controller/cmd_vel</commandTopic>
-				<odometryTopic>mobile_base_controller/odom</odometryTopic>
-				<robotBaseFrame>base_footprint</robotBaseFrame>
-				<wheelAcceleration>2.8</wheelAcceleration>
-				<publishWheelJointState>true</publishWheelJointState>
-				<publishWheelTF>false</publishWheelTF>
-				<odometrySource>world</odometrySource>
-				<rosDebugLevel>Debug</rosDebugLevel>
-			</plugin>
-		</gazebo-->
-		<!-- <p3d_base_controller prefix="${tf_prefix}" /> -->
 	</xacro:macro>
 </robot>

File: mir/mir_description/urdf/mir_200/mir_200.gazebo.xacro (robot description, xacro)
@@ -48,72 +48,4 @@
 		<!-- Settings for the camera of the robot to work in the simulation environment-->
     	<xacro:gazebo_d435 camera_name="${robot_namespace_underscored}camera" reference_link="camera_link" topics_ns="${robot_namespace_slashed}camera" depth_optical_frame="${tf_prefix_slashed}camera_depth_optical_frame" color_optical_frame="${tf_prefix_slashed}camera_color_optical_frame" infrared1_optical_frame="${tf_prefix_slashed}camera_left_ir_optical_frame" infrared2_optical_frame="${tf_prefix_slashed}camera_right_ir_optical_frame" publish_pointcloud="true"/>
-		<!-- disabled, because it doesn't make a difference in Gazebo: -->
-		<!-- <xacro:set_all_wheel_frictions tf_prefix="${tf_prefix}"/> -->
-		<!-- This part of the file looks like it is not necessary for the correct function of the urdf files.-->
-		<!-- Remove this part in a second iteration when all functions are working like they are supposed to be-->
-		<!-- <xacro:macro name="diff_controller_plugin_gazebo" params="prefix left_wheel_joint right_wheel_joint wheel_separation wheel_radius">
-			<gazebo>
-			<plugin name="diff_drive_controller" filename="libgazebo_ros_diff_drive.so">
-				<legacyMode>false</legacyMode>
-				<alwaysOn>true</alwaysOn>
-				<updateRate>1000.0</updateRate>
-				<leftJoint>${left_wheel_joint}</leftJoint>
-				<rightJoint>${right_wheel_joint}</rightJoint>
-				<wheelSeparation>${wheel_separation}</wheelSeparation>
-				<wheelDiameter>${2*wheel_radius}</wheelDiameter>
-				<wheelTorque>10</wheelTorque>
-				<publishTf>1</publishTf>
-				<odometryFrame>map</odometryFrame>
-				<commandTopic>mobile_base_controller/cmd_vel</commandTopic>
-				<odometryTopic>mobile_base_controller/odom</odometryTopic>
-				<robotBaseFrame>base_footprint</robotBaseFrame>
-				<wheelAcceleration>2.8</wheelAcceleration>
-				<publishWheelJointState>true</publishWheelJointState>
-				<publishWheelTF>false</publishWheelTF>
-				<odometrySource>world</odometrySource>
-				<rosDebugLevel>Debug</rosDebugLevel>
-			</plugin>
-			</gazebo>
-		</xacro:macro> -->
-		<!-- <xacro:macro name="set_wheel_friction" params="link friction">
-			<gazebo reference="${link}">
-			<mu1 value="${friction}"/>
-			<mu2 value="${friction}"/>
-			<kp value="10000000.0"/>
-			<kd value="1.0"/>
-			</gazebo>
-		</xacro:macro>
-		<xacro:macro name="set_all_wheel_frictions" params="prefix">
-			<xacro:set_wheel_friction link="${prefix}left_wheel_link" friction="200"/>
-			<xacro:set_wheel_friction link="${prefix}right_wheel_link" friction="200"/>
-			<xacro:set_wheel_friction link="${prefix}fl_caster_wheel_link" friction="1"/>
-			<xacro:set_wheel_friction link="${prefix}fr_caster_wheel_link" friction="1"/>
-			<xacro:set_wheel_friction link="${prefix}bl_caster_wheel_link" friction="1"/>
-			<xacro:set_wheel_friction link="${prefix}br_caster_wheel_link" friction="1"/>
-		</xacro:macro> -->
-		<!-- <p3d_base_controller tf_prefix="${tf_prefix}" /> -->
-		<!-- Settings for the camera of the robot to work in the simulation environment-->
-		<!--gazebo reference="camera_link">
-			<sensor type="depth" name="camera">
-			<plugin name="kinect_camera_controller" filename="libgazebo_ros_openni_kinect.so">
-				<cameraName>camera</cameraName>
-				<alwaysOn>true</alwaysOn>
-				<updateRate>10</updateRate>
-				<imageTopicName>rgb/image_raw</imageTopicName>
-				<depthImageTopicName>depth/image_raw</depthImageTopicName>
-				<pointCloudTopicName>depth/points</pointCloudTopicName>
-				<cameraInfoTopicName>rgb/camera_info</cameraInfoTopicName>
-				<depthImageCameraInfoTopicName>depth/camera_info</depthImageCameraInfoTopicName>
-				<frameName>camera_link_optical</frameName>
-				<baseline>0.1</baseline>
-				<distortion_k1>0.0</distortion_k1>
-				<distortion_k2>0.0</distortion_k2>
-				<distortion_k3>0.0</distortion_k3>
-				<distortion_t1>0.0</distortion_t1>
-				<distortion_t2>0.0</distortion_t2>
-				<pointCloudCutoff>0.4</pointCloudCutoff>
-			</plugin>
-			</sensor>
-		</gazebo-->
 	</xacro:macro>
 </robot>

File: mir/mir_description/urdf/mir_200/mir_200.urdf.xacro (robot description, xacro)
@@ -114,41 +114,4 @@
 		<xacro:match_logo parent="base_link" locationprefix="left" location_dx="${mir_200_match_logo_dx}" location_dy="${mir_200_match_logo_dy}" location_dz="${mir_200_match_logo_dz}"/>
 		<xacro:match_logo parent="base_link" locationprefix="right" location_dx="${mir_200_match_logo_dx}" location_dy="${-1 * mir_200_match_logo_dy}" location_dz="${mir_200_match_logo_dz}" orientation="${pi}"/>
-		<!-- Camera -->
-		<!--link name="camera_link">
-		<collision>
-			<origin xyz="0 0 0" rpy="0 0 0"/>
-			<geometry>
-				<box size="0.1 0.1 0.1"/>
-			</geometry>
-		</collision>
-		<visual>
-			<origin xyz="0 0 0" rpy="0 0 0"/>
-			<geometry>
-				<mesh filename="package://mir_description/meshes/visual/realsense.dae" />
-			</geometry>
-		</visual>
-		<inertial>
-			<mass value="1e-5" />
-			<origin xyz="0 0 0" rpy="0 0 0"/>
-			<inertia ixx="1e-6" ixy="0" ixz="0" iyy="1e-6" iyz="0" izz="1e-6" />
-		</inertial>
-		</link>
-		<joint name="camera_joint" type="fixed">
-			<axis xyz="0 1 0" />
-			<origin xyz="0.42 0 0.27" rpy="0 0.2 0"/--> <!--set the position of the realsense-->
-			<!--parent link="${tf_prefix}base_link"/>
-			<child link="camera_link"/>
-		</joint-->
-		<!-- generate an optical frame http://www.ros.org/reps/rep-0103.html#suffix-frames
-			so that ros and opencv can operate on the camera frame correctly -->
-		<!--joint name="camera_optical_joint" type="fixed"-->
-			<!-- these values have to be these values otherwise the gazebo camera image
-				won't be aligned properly with the frame it is supposedly originating from -->
-			<!--origin xyz="0 0 0" rpy="-1.5708 0 -1.5708"/>
-			<parent link="camera_link"/>
-			<child link="camera_link_optical"/>
-		</joint>
-		<link name="camera_link_optical"-->
-		<!--/link-->
 	</xacro:macro>
 </robot>
