Commit message: mir600 rev 1.0

File: mir/mir_description/urdf/mir_600/mir_600.urdf.xacro (robot description, xacro)
@@ -19,6 +19,6 @@
 	<xacro:property name="mir_600_caster_wheel_dy" value="0" />
 	<xacro:property name="mir_600_caster_wheel_dz" value="-0.05" />
-	<xacro:property name="mir_600_front_caster_wheel_base_dx" value="0.5865" />
-	<xacro:property name="mir_600_back_caster_wheel_base_dx" value="-0.270154" />
+	<xacro:property name="mir_600_front_caster_wheel_base_dx" value="0.4915" />
+	<xacro:property name="mir_600_back_caster_wheel_base_dx" value="-0.4885" />
 	<xacro:property name="mir_600_caster_wheel_base_dy" value="0.3215" />
 	<xacro:property name="mir_600_caster_wheel_base_dz" value="${mir_600_caster_wheel_radius-mir_600_caster_wheel_dz}" />
@@ -40,5 +40,5 @@
 				<origin xyz="${mir_600_act_wheel_dx} 0 0" rpy="${pi * 0.5} 0 ${pi * 0.5}" />
 				<geometry>
-					<mesh filename="package://mir_description/meshes/visual/mir_600_base.stl" scale="0.001 0.001 0.001"/>
+					<mesh filename="package://mir_description/meshes/visual/mir_600_base.stl"/>
 				</geometry>
 				<xacro:insert_block name="material_white" />
@@ -47,5 +47,5 @@
 				<origin xyz="${mir_600_act_wheel_dx} 0 0" rpy="0 0 0" />
 				<geometry>
-					<mesh filename="package://mir_description/meshes/collision/mir_600_base.stl" scale="0.001 0.001 0.001" />
+					<mesh filename="package://mir_description/meshes/collision/mir_600_base.stl"/>
 				</geometry>
 			</collision>

File: mir/mir_description/urdf/mir_600/mir_600_wheels.urdf.xacro (robot description, xacro)
@@ -15,12 +15,12 @@
 			</xacro:cylinder_inertial>
 			<visual>
-				<origin xyz="0 0 0" rpy="0 0 0" />
+				<origin xyz="0 ${locationright * mir_600_act_wheel_width*0.5} 0" rpy="${pi * 0.5} 0 ${0.5 * pi * (1+ locationright)}" />
 				<geometry>
-					<mesh filename="package://mir_description/meshes/visual/wheel.stl" />
+					<mesh filename="package://mir_description/meshes/visual/mir_600_wheel.stl" />
 				</geometry>
 				<xacro:insert_block name="material_dark_grey" />
 			</visual>
 			<collision>
-				<origin xyz="0 0 0" rpy="0 0 0" />
+				<origin xyz="0 0 0" rpy="${pi * 0.5} 0 ${pi * -1}" />
 				<geometry>
 					<mesh filename="package://mir_description/meshes/visual/wheel.stl" />

Commit message: mir600 rev1.1

File: mir/mir_description/urdf/mir_600/mir_600.urdf.xacro (robot description, xacro)
@@ -11,5 +11,5 @@
 	<xacro:property name="mir_600_act_wheel_width" value="0.05" />
 	<xacro:property name="mir_600_act_wheel_mass" value="1.0" />
-	<xacro:property name="mir_600_act_wheel_dx" value="0.037646" />
+	<xacro:property name="mir_600_act_wheel_dx" value="0.0" />
 	<xacro:property name="mir_600_act_wheel_dy" value="0.330" />
 	<xacro:property name="mir_600_caster_wheel_radius" value="0.05" />
@@ -18,5 +18,5 @@
 	<xacro:property name="mir_600_caster_wheel_dx" value="-0.0382" />
 	<xacro:property name="mir_600_caster_wheel_dy" value="0" />
-	<xacro:property name="mir_600_caster_wheel_dz" value="-0.05" />
+	<xacro:property name="mir_600_caster_wheel_dz" value="-0.1" />
 	<xacro:property name="mir_600_front_caster_wheel_base_dx" value="0.4915" />
 	<xacro:property name="mir_600_back_caster_wheel_base_dx" value="-0.4885" />
@@ -45,5 +45,5 @@
 			</visual>
 			<collision>
-				<origin xyz="${mir_600_act_wheel_dx} 0 0" rpy="0 0 0" />
+				<origin xyz="${mir_600_act_wheel_dx} 0 0" rpy="${pi * 0.5} 0 ${pi * 0.5}" />
 				<geometry>
 					<mesh filename="package://mir_description/meshes/collision/mir_600_base.stl"/>
@@ -71,5 +71,5 @@
 			<parent link="base_link" />
 			<child link="front_laser_link" />
-			<origin xyz="0.4288 0.2358 0.1914" rpy="0.0 0.0 ${0.25 * pi}" />  <!-- from visually matching up the meshes of the MiR and the laser scanner -->
+			<origin xyz="0.58985 0.370 0.1914" rpy="0.0 0.0 ${0.25 * pi}" />  <!-- from visually matching up the meshes of the MiR and the laser scanner -->
 		</joint>
 		<xacro:sick_s300 link="front_laser_link" topic="f_scan" />
@@ -77,5 +77,5 @@
 			<parent link="base_link" />
 			<child link="back_laser_link" />
-			<origin xyz="-0.3548 -0.2352 0.1914" rpy="0.0 0.0 ${-0.75 * pi}" />  <!-- from visually matching up the meshes of the MiR and the laser scanner -->
+			<origin xyz="-0.58985 -0.370 0.1914" rpy="0.0 0.0 ${-0.75 * pi}" />  <!-- from visually matching up the meshes of the MiR and the laser scanner -->
 		</joint>
 		<xacro:sick_s300 link="back_laser_link" topic="b_scan" />
@@ -109,5 +109,5 @@
 		<!--Realsense_Intel_D435_Camera-->
 		<xacro:sensor_d435 name="camera" parent="base_link" use_nominal_extrinsics="true">
-    		<origin xyz="0.42 0 0.27" rpy="0 0 0" />
+    		<origin xyz="0.62335 0 0.24" rpy="0 0 0" />
   		</xacro:sensor_d435>
 		<!-- Insert a match logo on both sides of the mobile robot -->

File: mir/mir_description/urdf/mir_600/mir_600_wheels.urdf.xacro (robot description, xacro)
@@ -24,5 +24,5 @@
 				<origin xyz="0 0 0" rpy="${pi * 0.5} 0 ${pi * -1}" />
 				<geometry>
-					<mesh filename="package://mir_description/meshes/visual/wheel.stl" />
+					<mesh filename="package://mir_description/meshes/visual/mir_600_wheel.stl" />
 				</geometry>
 			</collision>
@@ -77,14 +77,14 @@
 			</xacro:cylinder_inertial>
 			<visual>
-				<origin xyz="0 0 0" rpy="0 0 0" />
+				<origin xyz="0 0 0" rpy="${pi * 0.5} 0 0" />
 				<geometry>
-					<mesh filename="package://mir_description/meshes/visual/wheel.stl" />
+					<mesh filename="package://mir_description/meshes/visual/mir_600_caster_wheel.stl" />
 				</geometry>
 				<xacro:insert_block name="material_dark_grey" />
 			</visual>
 			<collision>
-				<origin xyz="0 0 0" rpy="0 0 0" />
+				<origin xyz="0 0 0" rpy="${pi * 0.5} 0 0" />
 				<geometry>
-					<mesh filename="package://mir_description/meshes/visual/wheel.stl" />
+					<mesh filename="package://mir_description/meshes/visual/mir_600_caster_wheel.stl" />
 				</geometry>
 			</collision>

Commit message: added Urs

File: mir/mir_description/urdf/mir_600/mir_600.urdf.xacro (robot description, xacro)
@@ -114,4 +114,29 @@
 		<xacro:match_logo parent="base_link" locationprefix="left" location_dx="${mir_600_match_logo_dx}" location_dy="${mir_600_match_logo_dy}" location_dz="${mir_600_match_logo_dz}"/>
 		<xacro:match_logo parent="base_link" locationprefix="right" location_dx="${mir_600_match_logo_dx}" location_dy="${-1 * mir_600_match_logo_dy}" location_dz="${mir_600_match_logo_dz}" orientation="${pi}"/>
+		<!-- top module -->
+		<link name="top_module">
+			<xacro:box_inertial mass="${mir_600_base_mass}" x="0.9" y="0.58" z="0.3">
+				<origin xyz="${mir_600_act_wheel_dx} 0 0.20" rpy="0 0 0" />
+			</xacro:box_inertial>
+			<visual>
+				<origin xyz="${mir_600_act_wheel_dx} 0 0" rpy="${pi * 0.5} 0 ${pi * 0.5}" />
+				<geometry>
+					<mesh filename="package://mir_description/meshes/visual/mir_600_top_module.stl"/>
+				</geometry>
+				<xacro:insert_block name="material_white" />
+			</visual>
+			<collision>
+				<origin xyz="${mir_600_act_wheel_dx} 0 0" rpy="${pi * 0.5} 0 ${pi * 0.5}" />
+				<geometry>
+					<mesh filename="package://mir_description/meshes/collision/mir_600_top_module.stl"/>
+				</geometry>
+			</collision>
+		</link>
+		<joint name="top_module_joint" type="fixed">
+			<origin xyz="0 0 0.832" rpy="0 0 0" />
+			<parent link="base_link" />
+			<child link="top_module" />
+			<axis xyz="0 0 1" />
+		</joint>
 		<!-- Camera -->
 		<!--link name="camera_link">

Commit message: mur620 rev 1.0

File: mir/mir_description/urdf/mir_600/mir_600.urdf.xacro (robot description, xacro)
@@ -6,6 +6,9 @@
 	<xacro:include filename="$(find mir_description)/urdf/general/match_logo.urdf.xacro" />
 	<xacro:include filename="$(find mir_description)/urdf/general/_d435.urdf.xacro" />
+	<xacro:include filename="$(find mir_description)/urdf/mir_600/mir_600_top_module.urdf.xacro" />
 	<xacro:property name="deg_to_rad" value="${(1 / 360) * (2 * pi)}" />
-	<xacro:property name="mir_600_base_mass" value="58.0" />
+	<xacro:property name="mir_600_base_mass" value="300.0" />
+	<xacro:property name="mir_600_top_module_mass" value="100.0" />
+	<xacro:property name="mir_600_lift_mass" value="30.0" />
 	<xacro:property name="mir_600_act_wheel_radius" value="0.1" />
 	<xacro:property name="mir_600_act_wheel_width" value="0.05" />
@@ -114,29 +117,5 @@
 		<xacro:match_logo parent="base_link" locationprefix="left" location_dx="${mir_600_match_logo_dx}" location_dy="${mir_600_match_logo_dy}" location_dz="${mir_600_match_logo_dz}"/>
 		<xacro:match_logo parent="base_link" locationprefix="right" location_dx="${mir_600_match_logo_dx}" location_dy="${-1 * mir_600_match_logo_dy}" location_dz="${mir_600_match_logo_dz}" orientation="${pi}"/>
-		<!-- top module -->
-		<link name="top_module">
-			<xacro:box_inertial mass="${mir_600_base_mass}" x="0.9" y="0.58" z="0.3">
-				<origin xyz="${mir_600_act_wheel_dx} 0 0.20" rpy="0 0 0" />
-			</xacro:box_inertial>
-			<visual>
-				<origin xyz="${mir_600_act_wheel_dx} 0 0" rpy="${pi * 0.5} 0 ${pi * 0.5}" />
-				<geometry>
-					<mesh filename="package://mir_description/meshes/visual/mir_600_top_module.stl"/>
-				</geometry>
-				<xacro:insert_block name="material_white" />
-			</visual>
-			<collision>
-				<origin xyz="${mir_600_act_wheel_dx} 0 0" rpy="${pi * 0.5} 0 ${pi * 0.5}" />
-				<geometry>
-					<mesh filename="package://mir_description/meshes/collision/mir_600_top_module.stl"/>
-				</geometry>
-			</collision>
-		</link>
-		<joint name="top_module_joint" type="fixed">
-			<origin xyz="0 0 0.832" rpy="0 0 0" />
-			<parent link="base_link" />
-			<child link="top_module" />
-			<axis xyz="0 0 1" />
-		</joint>
+		<xacro:top_module/>
 		<!-- Camera -->
 		<!--link name="camera_link">

File: mur/mur_description/urdf/mur_620.gazebo.xacro (robot description, xacro)
@@ -23,10 +23,10 @@
 			<parent link="base_link" />
 			<child link="UR10l/base_link" />
-			<origin xyz="0.549 0.318 0.832" rpy="0 0 0" />
+			<origin xyz="0.549 0.318 0.892" rpy="0 0 0" />
 	</joint>
 	<joint name="plattform_manipulator_joint_r" type="fixed">
 			<parent link="base_link" />
 			<child link="UR10r/base_link" />
-			<origin xyz="0.549 -0.318 0.832" rpy="0 0 0" />
+			<origin xyz="0.549 -0.318 0.892" rpy="0 0 0" />
 	</joint>
 	<!-- <gazebo>

Commit message: fixed drift

File: mir/mir_description/urdf/mir_600/mir_600.urdf.xacro (robot description, xacro)
@@ -13,5 +13,5 @@
 	<xacro:property name="mir_600_act_wheel_radius" value="0.1" />
 	<xacro:property name="mir_600_act_wheel_width" value="0.05" />
-	<xacro:property name="mir_600_act_wheel_mass" value="1.0" />
+	<xacro:property name="mir_600_act_wheel_mass" value="10.0" /> <!-- the robot starts drifting if the wheels are to light -->
 	<xacro:property name="mir_600_act_wheel_dx" value="0.0" />
 	<xacro:property name="mir_600_act_wheel_dy" value="0.330" />

File: mir/mir_description/urdf/mir_600/mir_600_wheels.urdf.xacro (robot description, xacro)
@@ -86,5 +86,5 @@
 				<origin xyz="0 0 0" rpy="${pi * 0.5} 0 0" />
 				<geometry>
-					<mesh filename="package://mir_description/meshes/visual/mir_600_caster_wheel.stl" />
+					<cylinder radius="${mir_600_caster_wheel_radius}" length="${mir_600_caster_wheel_width}"/>
 				</geometry>
 			</collision>

Commit message: first working moveit version for one arm

File: mir/mir_description/urdf/mir_600/mir_600.urdf.xacro (robot description, xacro)
@@ -27,5 +27,5 @@
 	<xacro:property name="mir_600_caster_wheel_base_dz" value="${mir_600_caster_wheel_radius-mir_600_caster_wheel_dz}" />
 	<xacro:property name="mir_600_match_logo_dx" value="0.0" />
-	<xacro:property name="mir_600_match_logo_dy" value="0.2724435" />
+	<xacro:property name="mir_600_match_logo_dy" value="0.330" />
 	<xacro:property name="mir_600_match_logo_dz" value="0.27" />
 	<xacro:macro name="mir_600">
@@ -115,6 +115,6 @@
   		</xacro:sensor_d435>
 		<!-- Insert a match logo on both sides of the mobile robot -->
-		<xacro:match_logo parent="base_link" locationprefix="left" location_dx="${mir_600_match_logo_dx}" location_dy="${mir_600_match_logo_dy}" location_dz="${mir_600_match_logo_dz}"/>
-		<xacro:match_logo parent="base_link" locationprefix="right" location_dx="${mir_600_match_logo_dx}" location_dy="${-1 * mir_600_match_logo_dy}" location_dz="${mir_600_match_logo_dz}" orientation="${pi}"/>
+		<!-- <xacro:match_logo parent="base_link" locationprefix="left" location_dx="${mir_600_match_logo_dx}" location_dy="${mir_600_match_logo_dy}" location_dz="${mir_600_match_logo_dz}"/>
+		<xacro:match_logo parent="base_link" locationprefix="right" location_dx="${mir_600_match_logo_dx}" location_dy="${-1 * mir_600_match_logo_dy}" location_dz="${mir_600_match_logo_dz}" orientation="${pi}"/> -->
 		<xacro:top_module/>
 		<!-- Camera -->

File: mur/mur_description/urdf/mur_620.gazebo.xacro (robot description, xacro)
@@ -1,4 +1,4 @@
 <?xml version="1.0"?>
-<robot xmlns:xacro="http://wiki.ros.org/xacro" name="mur216" >
+<robot xmlns:xacro="http://wiki.ros.org/xacro" name="mur620" >
 	<xacro:arg name="robot_namespace" default=''/>
 	<xacro:arg name="tf_prefix" default=''/>

Commit message: added lift argument for prismatic joint

File: mir/mir_description/urdf/mir_600/mir_600.urdf.xacro (robot description, xacro)
@@ -1,4 +1,5 @@
 <?xml version="1.0"?>
 <robot xmlns:xacro="http://ros.org/wiki/xacro">
+	<xacro:property name="use_lift" value="$(arg use_lift)"/>
 	<xacro:include filename="$(find mir_description)/urdf/general/common_properties.urdf.xacro" />
 	<xacro:include filename="$(find mir_description)/urdf/general/sick_s300.urdf.xacro" />
@@ -7,4 +8,5 @@
 	<xacro:include filename="$(find mir_description)/urdf/general/_d435.urdf.xacro" />
 	<xacro:include filename="$(find mir_description)/urdf/mir_600/mir_600_top_module.urdf.xacro" />
+	<xacro:include filename="$(find mir_description)/urdf/mir_600/mir_600_top_lift.urdf.xacro" />
 	<xacro:property name="deg_to_rad" value="${(1 / 360) * (2 * pi)}" />
 	<xacro:property name="mir_600_base_mass" value="300.0" />
@@ -118,4 +120,8 @@
 		<xacro:match_logo parent="base_link" locationprefix="right" location_dx="${mir_600_match_logo_dx}" location_dy="${-1 * mir_600_match_logo_dy}" location_dz="${mir_600_match_logo_dz}" orientation="${pi}"/> -->
 		<xacro:top_module/>
+		<!-- <xacro:if value="${use_lift == 'true'}"> -->
+		<xacro:if value="${use_lift}">
+			<xacro:top_lift/>
+		</xacro:if>
 		<!-- Camera -->
 		<!--link name="camera_link">

File: mir/mir_description/urdf/mir_600/mir_600_top_module.urdf.xacro (robot description, xacro)
@@ -52,30 +52,4 @@
 			<axis xyz="0 0 1" />
 		</joint>
-		<link name="left_lift_top">
-			<xacro:box_inertial mass="1.0" x="0.2" y="0.2" z="0.3">
-				<origin xyz="0 0 0.15" rpy="0 0 0" />
-			</xacro:box_inertial>
-			<visual>
-				<origin xyz="0 0 0" rpy="${pi * 0.5} 0 ${pi * 0.0}" />
-				<geometry>
-					<mesh filename="package://mir_description/meshes/visual/mir_600_lift_top.stl"/>
-				</geometry>
-				<xacro:insert_block name="material_white" />
-			</visual>
-			<collision>
-				<origin xyz="0 0 0" rpy="${pi * 0.5} 0 ${pi * 0.0}" />
-				<geometry>
-					<mesh filename="package://mir_description/meshes/collision/mir_600_lift_top.stl"/>
-				</geometry>
-			</collision>
-		</link>
-		<joint name="left_lift_joint" type="prismatic">
-			<origin xyz="0.0 0.0 0.0" rpy="0 0 0" />
-			<parent link="left_lift_bottom" />
-			<child link="left_lift_top" />
-			<dynamics damping="1.0" friction="1.0"/>
-			<limit lower="0.0" upper="0.5" effort="1000000" velocity="1.0"/>
-			<axis xyz="0 0 1" />
-		</joint>
 		<link name="right_lift_bottom">
 			<xacro:box_inertial mass="${mir_600_lift_mass}" x="0.2" y="0.2" z="0.3">
@@ -102,50 +76,4 @@
 			<axis xyz="0 0 1" />
 		</joint>
-		<link name="right_lift_top">
-			<xacro:box_inertial mass="1.0" x="0.2" y="0.2" z="0.3">
-				<origin xyz="0 0 0.15" rpy="0 0 0" />
-			</xacro:box_inertial>
-			<visual>
-				<origin xyz="0 0 0" rpy="${pi * 0.5} 0 ${pi * 0.0}" />
-				<geometry>
-					<mesh filename="package://mir_description/meshes/visual/mir_600_lift_top.stl"/>
-				</geometry>
-				<xacro:insert_block name="material_white" />
-			</visual>
-			<collision>
-				<origin xyz="0 0 0" rpy="${pi * 0.5} 0 ${pi * 0.0}" />
-				<geometry>
-					<mesh filename="package://mir_description/meshes/collision/mir_600_lift_top.stl"/>
-				</geometry>
-			</collision>
-		</link>
-		<joint name="right_lift_joint" type="prismatic">
-			<origin xyz="0.0 0.0 0.0" rpy="0 0 0" />
-			<parent link="right_lift_bottom" />
-			<child link="right_lift_top" />
-			<dynamics damping="1.0" friction="1.0"/>
-			<limit lower="0.0" upper="0.5" effort="1000000" velocity="1.0"/>
-			<axis xyz="0 0 1" />
-		</joint>
-		<transmission name="left_lift_transmission">
-			<type>transmission_interface/SimpleTransmission</type>
-			<joint name="left_lift_joint">
-			  <hardwareInterface>hardware_interface/VelocityJointInterface</hardwareInterface>
-			</joint>
-			<actuator name="left_lift_joint_motor">
-			  <hardwareInterface>hardware_interface/VelocityJointInterface</hardwareInterface>
-			  <mechanicalReduction>1</mechanicalReduction>
-			</actuator>
-		</transmission>
-		<transmission name="right_lift_transmission">
-			<type>transmission_interface/SimpleTransmission</type>
-			<joint name="right_lift_joint">
-			  <hardwareInterface>hardware_interface/VelocityJointInterface</hardwareInterface>
-			</joint>
-			<actuator name="right_lift_joint_motor">
-			  <hardwareInterface>hardware_interface/VelocityJointInterface</hardwareInterface>
-			  <mechanicalReduction>1</mechanicalReduction>
-			</actuator>
-		</transmission>
 	</xacro:macro>
 </robot>

Commit message: mur620 sim with lift urdf as planned

File: mir/mir_description/urdf/mir_600/mir_600.urdf.xacro (robot description, xacro)
@@ -1,6 +1,4 @@
 <?xml version="1.0"?>
 <robot xmlns:xacro="http://ros.org/wiki/xacro">
-	<xacro:arg name="use_lift" default='true'/>
-	<xacro:property name="use_lift" value="$(arg use_lift)"/>
 	<xacro:include filename="$(find mir_description)/urdf/general/common_properties.urdf.xacro" />
 	<xacro:include filename="$(find mir_description)/urdf/general/sick_s300.urdf.xacro" />
@@ -9,5 +7,4 @@
 	<xacro:include filename="$(find mir_description)/urdf/general/_d435.urdf.xacro" />
 	<xacro:include filename="$(find mir_description)/urdf/mir_600/mir_600_top_module.urdf.xacro" />
-	<xacro:include filename="$(find mir_description)/urdf/mir_600/mir_600_top_lift.urdf.xacro" />
 	<xacro:property name="deg_to_rad" value="${(1 / 360) * (2 * pi)}" />
 	<xacro:property name="mir_600_base_mass" value="300.0" />
@@ -121,8 +118,4 @@
 		<xacro:match_logo parent="base_link" locationprefix="right" location_dx="${mir_600_match_logo_dx}" location_dy="${-1 * mir_600_match_logo_dy}" location_dz="${mir_600_match_logo_dz}" orientation="${pi}"/> -->
 		<xacro:top_module/>
-		<!-- <xacro:if value="${use_lift == 'true'}"> -->
-		<xacro:if value="${use_lift}">
-			<xacro:top_lift/>
-		</xacro:if>
 		<!-- Camera -->
 		<!--link name="camera_link">

File: mur/mur_description/urdf/mur_620.gazebo.xacro (robot description, xacro)
@@ -3,4 +3,6 @@
 	<xacro:arg name="robot_namespace" default=''/>
 	<xacro:arg name="tf_prefix" default=''/>
+	<xacro:arg name="use_lift" default='true'/>
+	<xacro:property name="use_lift" value="$(arg use_lift)"/>
 	<!-- MiR200 base -->
 	<xacro:include filename="$(find mir_description)/urdf/mir_600/mir_600.urdf.xacro" />
@@ -9,4 +11,6 @@
   	<xacro:include filename="$(find ur_description)/urdf/inc/ur16e_macro.xacro"/>
 	<xacro:include filename="$(find ur_description)/urdf/inc/ur10e_macro.xacro"/>
+	<!-- Lift modules -->
+	<xacro:include filename="$(find mir_description)/urdf/mir_600/mir_600_top_lift.urdf.xacro" />
 	<!-- Include plugin xacros -->
 	<xacro:include filename="$(find mir_description)/urdf/general/plugins.gazebo.xacro" />
@@ -23,14 +27,30 @@
 	<!-- Init the plugins that run the MiR in Gazebo -->
 	<xacro:controller_plugin_gazebo robot_namespace="$(arg robot_namespace)"/>
-	<joint name="plattform_manipulator_joint_l" type="fixed">
-			<parent link="left_lift_top" />
+	<!-- Init the lift macro -->
+	<xacro:if value="${use_lift}">
+		<xacro:top_lift/>
+		<joint name="plattform_manipulator_joint_l" type="fixed">
+				<parent link="left_lift_top" />
+				<child link="UR10_l/base_link" />
+				<origin xyz="0.0 0.0 0.555" rpy="0 0 0" />
+		</joint>
+		<joint name="plattform_manipulator_joint_r" type="fixed">
+				<parent link="right_lift_top" />
+				<child link="UR10_r/base_link" />
+				<origin xyz="0.0 0.0 0.555" rpy="0 0 0" />
+		</joint>
+	</xacro:if>
+	<xacro:unless value="${use_lift}">
+		<joint name="plattform_manipulator_joint_l" type="fixed">
+			<parent link="left_lift_bottom" />
 			<child link="UR10_l/base_link" />
 			<origin xyz="0.0 0.0 0.555" rpy="0 0 0" />
-	</joint>
-	<joint name="plattform_manipulator_joint_r" type="fixed">
-			<parent link="right_lift_top" />
+		</joint>
+		<joint name="plattform_manipulator_joint_r" type="fixed">
+			<parent link="right_lift_bottom" />
 			<child link="UR10_r/base_link" />
 			<origin xyz="0.0 0.0 0.555" rpy="0 0 0" />
-	</joint>
+		</joint>
+	</xacro:unless>
 	<xacro:schunk_emh_rp_045 tf_prefix="UR10_r"	tool_link="UR10_r/flange"/>
 	<xacro:schunk_emh_rp_045 tf_prefix="UR10_l"	tool_link="UR10_l/flange"/>
