Commit message: added colors/materials for gazebo

File: mir/mir_description/urdf/mir_600/mir_600_top_lift.urdf.xacro (robot description, xacro)
@@ -20,4 +20,7 @@
 			</collision>
 		</link>
+		<gazebo reference="left_lift_top">
+			<material>Gazebo/Grey</material>
+		</gazebo>
 		<joint name="left_lift_joint" type="prismatic">
 			<origin xyz="0.0 0.0 0.0" rpy="0 0 0" />
@@ -46,4 +49,7 @@
 			</collision>
 		</link>
+		<gazebo reference="right_lift_top">
+			<material>Gazebo/Grey</material>
+		</gazebo>
 		<joint name="right_lift_joint" type="prismatic">
 			<origin xyz="0.0 0.0 0.0" rpy="0 0 0" />
