Commit message: added lift modules

File: mir/mir_description/urdf/mir_600/mir_600_top_module.urdf.xacro (robot description, xacro)
@@ -70,8 +70,10 @@
 			</collision>
 		</link>
-		<joint name="left_lift_joint" type="fixed">
+		<joint name="left_lift_joint" type="prismatic">
 			<origin xyz="0.0 0.0 0.0" rpy="0 0 0" />
 			<parent link="left_lift_bottom" />
 			<child link="left_lift_top" />
+			<dynamics damping="1.0" friction="1.0"/>
+			<limit lower="0.0" upper="0.5" effort="1000000" velocity="1.0"/>
 			<axis xyz="0 0 1" />
 		</joint>
@@ -118,10 +120,32 @@
 			</collision>
 		</link>
-		<joint name="right_lift_joint" type="fixed">
+		<joint name="right_lift_joint" type="prismatic">
 			<origin xyz="0.0 0.0 0.0" rpy="0 0 0" />
 			<parent link="right_lift_bottom" />
 			<child link="right_lift_top" />
+			<dynamics damping="1.0" friction="1.0"/>
+			<limit lower="0.0" upper="0.5" effort="1000000" velocity="1.0"/>
 			<axis xyz="0 0 1" />
 		</joint>
+		<transmission name="left_lift_transmission">
+			<type>transmission_interface/SimpleTransmission</type>
+			<joint name="left_lift_joint">
+			  <hardwareInterface>hardware_interface/VelocityJointInterface</hardwareInterface>
+			</joint>
+			<actuator name="left_lift_joint_motor">
+			  <hardwareInterface>hardware_interface/VelocityJointInterface</hardwareInterface>
+			  <mechanicalReduction>1</mechanicalReduction>
+			</actuator>
+		</transmission>
+		<transmission name="right_lift_transmission">
+			<type>transmission_interface/SimpleTransmission</type>
+			<joint name="right_lift_joint">
+			  <hardwareInterface>hardware_interface/VelocityJointInterface</hardwareInterface>
+			</joint>
+			<actuator name="right_lift_joint_motor">
+			  <hardwareInterface>hardware_interface/VelocityJointInterface</hardwareInterface>
+			  <mechanicalReduction>1</mechanicalReduction>
+			</actuator>
+		</transmission>
 	</xacro:macro>
 </robot>

File: mur/mur_description/urdf/mur_620.gazebo.xacro (robot description, xacro)
@@ -21,12 +21,12 @@
 	<xacro:controller_plugin_gazebo robot_namespace="$(arg robot_namespace)"/>
 	<joint name="plattform_manipulator_joint_l" type="fixed">
-			<parent link="base_link" />
+			<parent link="left_lift_top" />
 			<child link="UR10l/base_link" />
-			<origin xyz="0.549 0.318 0.892" rpy="0 0 0" />
+			<origin xyz="0.0 0.0 0.555" rpy="0 0 0" />
 	</joint>
 	<joint name="plattform_manipulator_joint_r" type="fixed">
-			<parent link="base_link" />
+			<parent link="right_lift_top" />
 			<child link="UR10r/base_link" />
-			<origin xyz="0.549 -0.318 0.892" rpy="0 0 0" />
+			<origin xyz="0.0 0.0 0.555" rpy="0 0 0" />
 	</joint>
 	<!-- <gazebo>

Commit message: corrected top module orientation

File: mir/mir_description/urdf/mir_600/mir_600_top_module.urdf.xacro (robot description, xacro)
@@ -9,14 +9,14 @@
 			</xacro:box_inertial>
 			<visual>
-				<origin xyz="${mir_600_act_wheel_dx} 0 0" rpy="${pi * 0.5} 0 ${pi * 0.5}" />
+				<origin xyz="${mir_600_act_wheel_dx} 0 0" rpy="0 0 ${-pi * 0.5}" />
 				<geometry>
-					<mesh filename="package://mir_description/meshes/visual/mir_600_top_module.stl"/>
+					<mesh filename="package://mir_description/meshes/visual/mir_600_top_module.stl" scale="0.001 0.001 0.001"/>
 				</geometry>
 				<xacro:insert_block name="material_white" />
 			</visual>
 			<collision>
-				<origin xyz="${mir_600_act_wheel_dx} 0 0" rpy="${pi * 0.5} 0 ${pi * 0.5}" />
+				<origin xyz="${mir_600_act_wheel_dx} 0 0" rpy="0 0 ${-pi * 0.5}" />
 				<geometry>
-					<mesh filename="package://mir_description/meshes/collision/mir_600_top_module.stl"/>
+					<mesh filename="package://mir_description/meshes/collision/mir_600_top_module.stl" scale="0.001 0.001 0.001" />
 				</geometry>
 			</collision>

Commit message: added colors/materials for gazebo

File: mir/mir_description/urdf/mir_600/mir_600_top_module.urdf.xacro (robot description, xacro)
@@ -22,4 +22,7 @@
 			</collision>
 		</link>
+		<gazebo reference="top_module">
+			<material>Gazebo/Grey</material>
+		</gazebo>
 		<joint name="top_module_joint" type="fixed">
 			<origin xyz="0 0 0.832" rpy="0 0 0" />
@@ -46,4 +49,7 @@
 			</collision>
 		</link>
+		<gazebo reference="left_lift_bottom">
+			<material>Gazebo/DarkGrey</material>
+		</gazebo>
 		<joint name="left_lift_bottom_joint" type="fixed">
 			<origin xyz="0.549 0.318 -0.49" rpy="0 0 0" />
@@ -70,4 +76,7 @@
 			</collision>
 		</link>
+		<gazebo reference="right_lift_bottom">
+			<material>Gazebo/DarkGrey</material>
+		</gazebo>
 		<joint name="right_lift_bottom_joint" type="fixed">
 			<origin xyz="0.549 -0.318 -0.49" rpy="0 0 0" />

File: tools/schunk_emh_rp_45/urdf/schunk_emh_rp_045.urdf.xacro (robot description, xacro)
@@ -33,4 +33,7 @@
 			</collision>
 		</link>
+		<gazebo reference="${tf_prefix}/tcp">
+			<material>Gazebo/DarkGrey</material>
+		</gazebo>
 		<!-- the ft_sensor plugin will not work with fixed joints. This is why a prismatic joint with very small limits is added -->
 		<joint name="${tf_prefix}/tcp_joint" type="prismatic">

Commit message: Fix right lift bottom joint origin z-coordinate for accurate positioning

File: mir/mir_description/urdf/mir_600/mir_600_top_module.urdf.xacro (robot description, xacro)
@@ -80,5 +80,5 @@
 		</gazebo>
 		<joint name="right_lift_bottom_joint" type="fixed">
-			<origin xyz="0.549 -0.318 -0.49" rpy="0 0 0" />
+			<origin xyz="0.549 -0.318 -0.518" rpy="0 0 0" />
 			<parent link="top_module" />
 			<child link="right_lift_bottom" />
