Commit message: fixed ft_sensor noise issue

File: tools/schunk_emh_rp_45/urdf/schunk_emh_rp_045.urdf.xacro (robot description, xacro)
@@ -6,4 +6,16 @@
 		<link name="${tf_prefix}/gripper">
 			<xacro:cylinder_inertial mass="1.5" radius="0.32" length="0.128">
+				<origin xyz="0 0 0.06" rpy="0 0 0" />
+			</xacro:cylinder_inertial>
+		</link>
+		<joint name="${tf_prefix}/gripper_joint" type="fixed">
+			<origin xyz="0 0 0.0" rpy="0 0 0" />
+			<parent link="${tool_link}" />
+			<child link="${tf_prefix}/gripper" />
+			<axis xyz="0 0 1" />
+			<limit effort="1000" lower="-0.0001" upper="0.0001" velocity="10"/>
+		</joint>
+		<link name="${tf_prefix}/tcp">
+			<xacro:cylinder_inertial mass="0.01" radius="0.32" length="0.128">
 				<origin xyz="0 0 0.06" rpy="0 0 0" />
 			</xacro:cylinder_inertial>
@@ -16,5 +28,5 @@
 			</visual>
 			<collision>
-				<origin xyz="0 0 0" rpy="0 0 0" />
+				<origin xyz="0 0 0.128" rpy="${-pi * 0.5} 0 0" />
 				<geometry>
 					<mesh filename="package://schunk_emh_rp_45/meshes/collision/schunk_emh_rp_045.stl" scale="0.001 0.001 0.001" />
@@ -22,22 +34,21 @@
 			</collision>
 		</link>
-		<joint name="${tf_prefix}/gripper_joint" type="fixed">
+		<!-- the ft_sensor plugin will not work with fixed joints. This is why a prismatic joint with very small limits is added -->
+		<joint name="${tf_prefix}/tcp_joint" type="prismatic">
 			<origin xyz="0 0 0.0" rpy="0 0 0" />
-			<parent link="${tool_link}" />
-			<child link="${tf_prefix}/gripper" />
+			<parent link="${tf_prefix}/gripper" />
+			<child link="${tf_prefix}/tcp" />
 			<axis xyz="0 0 1" />
-			<sensor name="force_torque" type="force_torque">
-          		<update_rate>30</update_rate>
-        	</sensor>
+   			<limit effort="1000" lower="-0.0001" upper="0.0001" velocity="10"/>
 		</joint>
-		<gazebo reference="${tf_prefix}/wrist_3_joint">
+		<gazebo reference="${tf_prefix}/tcp_joint">
    			<provideFeedback>true</provideFeedback>
   		</gazebo>
 		<!-- The ft_sensor plugin  -->
 		<gazebo>
-			<plugin name="UR_ft_sensor" filename="libgazebo_ros_ft_sensor.so">
-			<updateRate>1000.0</updateRate>
+			<plugin name="ft_sensor" filename="libgazebo_ros_ft_sensor.so">
+			<updateRate>500.0</updateRate>
 			<topicName>${tf_prefix}/ft_sensor_topic</topicName>
-			<jointName>${tf_prefix}/wrist_3_joint</jointName>
+			<jointName>${tf_prefix}/tcp_joint</jointName>
 			<noise>
 			<type>gaussian</type>

Commit message: changed gripper tf

File: tools/schunk_emh_rp_45/urdf/schunk_emh_rp_045.urdf.xacro (robot description, xacro)
@@ -3,5 +3,4 @@
 	<xacro:include filename="$(find mir_description)/urdf/general/common_properties.urdf.xacro" />
 	<xacro:macro name="schunk_emh_rp_045" params="tool_link tf_prefix">
-		<!-- top module -->
 		<link name="${tf_prefix}/gripper">
 			<xacro:cylinder_inertial mass="1.5" radius="0.32" length="0.128">
@@ -10,5 +9,5 @@
 		</link>
 		<joint name="${tf_prefix}/gripper_joint" type="fixed">
-			<origin xyz="0 0 0.0" rpy="0 0 0" />
+			<origin xyz="0 0 0.0" rpy="${-pi * 0.5} ${-pi * 0.5} ${pi}" />
 			<parent link="${tool_link}" />
 			<child link="${tf_prefix}/gripper" />
@@ -21,5 +20,5 @@
 			</xacro:cylinder_inertial>
 			<visual>
-				<origin xyz="0 0 0.128" rpy="${-pi * 0.5} 0 0" />
+				<origin xyz="0 -0.128 0" rpy="0 0 0" />
 				<geometry>
 					<mesh filename="package://schunk_emh_rp_45/meshes/visual/schunk_emh_rp_045.stl" scale="0.001 0.001 0.001"/>
@@ -28,5 +27,5 @@
 			</visual>
 			<collision>
-				<origin xyz="0 0 0.128" rpy="${-pi * 0.5} 0 0" />
+				<origin xyz="0 -0.128 0" rpy="0 0 0" />
 				<geometry>
 					<mesh filename="package://schunk_emh_rp_45/meshes/collision/schunk_emh_rp_045.stl" scale="0.001 0.001 0.001" />
