Commit message: mur moveit finally working

File: mur/mur_moveit_config/config/mur.srdf.xacro (robot description, xacro)
@@ -4,5 +4,7 @@
     A URDF file must exist for this robot as well, where the joints and the links that are referenced are defined
 -->
-<robot name="mur216">
+<robot name="mur216"
+        xmlns:xacro="http://www.ros.org/wiki/xacro">
+    <xacro:arg name="prefix" default=""/>
     <!--GROUPS: Representation of a set of joints and links. This can be useful for specifying DOF to plan for, defining arms, end effectors, etc-->
     <!--LINKS: When a link is specified, the parent joint of that link (if it exists) is automatically included-->
@@ -11,70 +13,70 @@
     <!--SUBGROUPS: Groups can also be formed by referencing to already defined group names-->
     <group name="UR_arm">
-        <joint name="UR16/base_link-base_fixed_joint"/>
-        <joint name="UR16/base_link-base_link_inertia"/>
-        <joint name="UR16/shoulder_pan_joint"/>
-        <joint name="UR16/shoulder_lift_joint"/>
-        <joint name="UR16/elbow_joint"/>
-        <joint name="UR16/wrist_1_joint"/>
-        <joint name="UR16/wrist_2_joint"/>
-        <joint name="UR16/wrist_3_joint"/>
-        <joint name="UR16/wrist_3-flange"/>
-        <joint name="UR16/flange-tool0"/>
+        <joint name="$(arg prefix)base_link-base_fixed_joint"/>
+        <joint name="$(arg prefix)base_link-base_link_inertia"/>
+        <joint name="$(arg prefix)shoulder_pan_joint"/>
+        <joint name="$(arg prefix)shoulder_lift_joint"/>
+        <joint name="$(arg prefix)elbow_joint"/>
+        <joint name="$(arg prefix)wrist_1_joint"/>
+        <joint name="$(arg prefix)wrist_2_joint"/>
+        <joint name="$(arg prefix)wrist_3_joint"/>
+        <joint name="$(arg prefix)wrist_3-flange"/>
+        <joint name="$(arg prefix)flange-tool0"/>
     </group>
     <!--GROUP STATES: Purpose: Define a named state for a particular group, in terms of joint values. This is useful to define states like 'folded arms'-->
     <group_state name="Home_custom" group="UR_arm">
-        <joint name="UR16/elbow_joint" value="1.6141"/>
-        <joint name="UR16/shoulder_lift_joint" value="-1.5621"/>
-        <joint name="UR16/shoulder_pan_joint" value="-0.0347"/>
-        <joint name="UR16/wrist_1_joint" value="-1.7009"/>
-        <joint name="UR16/wrist_2_joint" value="-1.5621"/>
-        <joint name="UR16/wrist_3_joint" value="0"/>
+        <joint name="$(arg prefix)elbow_joint" value="1.6141"/>
+        <joint name="$(arg prefix)shoulder_lift_joint" value="-1.5621"/>
+        <joint name="$(arg prefix)shoulder_pan_joint" value="-0.0347"/>
+        <joint name="$(arg prefix)wrist_1_joint" value="-1.7009"/>
+        <joint name="$(arg prefix)wrist_2_joint" value="-1.5621"/>
+        <joint name="$(arg prefix)wrist_3_joint" value="0"/>
     </group_state>
     <!--END EFFECTOR: Purpose: Represent information about an end effector.-->
-    <end_effector name="hand" parent_link="UR16/tool0" group="UR_arm"/>
+    <end_effector name="hand" parent_link="$(arg prefix)tool0" group="UR_arm"/>
     <!--DISABLE COLLISIONS: By default it is assumed that any link of the robot could potentially come into collision with any other link in the robot. This tag disables collision checking between a specified pair of links. -->
-    <disable_collisions link1="UR16/base_link_inertia" link2="UR16/shoulder_link" reason="Adjacent"/>
-    <disable_collisions link1="UR16/base_link_inertia" link2="UR16/upper_arm_link" reason="Never"/>
-    <disable_collisions link1="UR16/base_link_inertia" link2="UR16/wrist_1_link" reason="Never"/>
-    <disable_collisions link1="UR16/base_link_inertia" link2="back_laser_link" reason="Never"/>
-    <disable_collisions link1="UR16/base_link_inertia" link2="base_link" reason="Adjacent"/>
-    <disable_collisions link1="UR16/base_link_inertia" link2="bl_caster_rotation_link" reason="Never"/>
-    <disable_collisions link1="UR16/base_link_inertia" link2="bl_caster_wheel_link" reason="Never"/>
-    <disable_collisions link1="UR16/base_link_inertia" link2="br_caster_rotation_link" reason="Never"/>
-    <disable_collisions link1="UR16/base_link_inertia" link2="br_caster_wheel_link" reason="Never"/>
-    <disable_collisions link1="UR16/base_link_inertia" link2="camera_link" reason="Never"/>
-    <disable_collisions link1="UR16/base_link_inertia" link2="fl_caster_rotation_link" reason="Never"/>
-    <disable_collisions link1="UR16/base_link_inertia" link2="fl_caster_wheel_link" reason="Never"/>
-    <disable_collisions link1="UR16/base_link_inertia" link2="fr_caster_rotation_link" reason="Never"/>
-    <disable_collisions link1="UR16/base_link_inertia" link2="fr_caster_wheel_link" reason="Never"/>
-    <disable_collisions link1="UR16/base_link_inertia" link2="front_laser_link" reason="Never"/>
-    <disable_collisions link1="UR16/base_link_inertia" link2="left_wheel_link" reason="Never"/>
-    <disable_collisions link1="UR16/base_link_inertia" link2="right_wheel_link" reason="Never"/>
-    <disable_collisions link1="UR16/forearm_link" link2="UR16/upper_arm_link" reason="Adjacent"/>
-    <disable_collisions link1="UR16/forearm_link" link2="UR16/wrist_1_link" reason="Adjacent"/>
-    <disable_collisions link1="UR16/shoulder_link" link2="UR16/upper_arm_link" reason="Adjacent"/>
-    <disable_collisions link1="UR16/shoulder_link" link2="UR16/wrist_1_link" reason="Never"/>
-    <disable_collisions link1="UR16/shoulder_link" link2="back_laser_link" reason="Never"/>
-    <disable_collisions link1="UR16/shoulder_link" link2="base_link" reason="Never"/>
-    <disable_collisions link1="UR16/shoulder_link" link2="bl_caster_rotation_link" reason="Never"/>
-    <disable_collisions link1="UR16/shoulder_link" link2="bl_caster_wheel_link" reason="Never"/>
-    <disable_collisions link1="UR16/shoulder_link" link2="br_caster_rotation_link" reason="Never"/>
-    <disable_collisions link1="UR16/shoulder_link" link2="br_caster_wheel_link" reason="Never"/>
-    <disable_collisions link1="UR16/shoulder_link" link2="camera_link" reason="Never"/>
-    <disable_collisions link1="UR16/shoulder_link" link2="fl_caster_rotation_link" reason="Never"/>
-    <disable_collisions link1="UR16/shoulder_link" link2="fl_caster_wheel_link" reason="Never"/>
-    <disable_collisions link1="UR16/shoulder_link" link2="fr_caster_rotation_link" reason="Never"/>
-    <disable_collisions link1="UR16/shoulder_link" link2="fr_caster_wheel_link" reason="Never"/>
-    <disable_collisions link1="UR16/shoulder_link" link2="front_laser_link" reason="Never"/>
-    <disable_collisions link1="UR16/shoulder_link" link2="left_wheel_link" reason="Never"/>
-    <disable_collisions link1="UR16/shoulder_link" link2="right_wheel_link" reason="Never"/>
-    <disable_collisions link1="UR16/upper_arm_link" link2="back_laser_link" reason="Never"/>
-    <disable_collisions link1="UR16/upper_arm_link" link2="bl_caster_rotation_link" reason="Never"/>
-    <disable_collisions link1="UR16/upper_arm_link" link2="bl_caster_wheel_link" reason="Never"/>
-    <disable_collisions link1="UR16/upper_arm_link" link2="br_caster_rotation_link" reason="Never"/>
-    <disable_collisions link1="UR16/upper_arm_link" link2="br_caster_wheel_link" reason="Never"/>
-    <disable_collisions link1="UR16/wrist_1_link" link2="UR16/wrist_2_link" reason="Adjacent"/>
-    <disable_collisions link1="UR16/wrist_1_link" link2="UR16/wrist_3_link" reason="Never"/>
-    <disable_collisions link1="UR16/wrist_2_link" link2="UR16/wrist_3_link" reason="Adjacent"/>
+    <disable_collisions link1="$(arg prefix)base_link_inertia" link2="$(arg prefix)shoulder_link" reason="Adjacent"/>
+    <disable_collisions link1="$(arg prefix)base_link_inertia" link2="$(arg prefix)upper_arm_link" reason="Never"/>
+    <disable_collisions link1="$(arg prefix)base_link_inertia" link2="$(arg prefix)wrist_1_link" reason="Never"/>
+    <disable_collisions link1="$(arg prefix)base_link_inertia" link2="back_laser_link" reason="Never"/>
+    <disable_collisions link1="$(arg prefix)base_link_inertia" link2="base_link" reason="Adjacent"/>
+    <disable_collisions link1="$(arg prefix)base_link_inertia" link2="bl_caster_rotation_link" reason="Never"/>
+    <disable_collisions link1="$(arg prefix)base_link_inertia" link2="bl_caster_wheel_link" reason="Never"/>
+    <disable_collisions link1="$(arg prefix)base_link_inertia" link2="br_caster_rotation_link" reason="Never"/>
+    <disable_collisions link1="$(arg prefix)base_link_inertia" link2="br_caster_wheel_link" reason="Never"/>
+    <disable_collisions link1="$(arg prefix)base_link_inertia" link2="camera_link" reason="Never"/>
+    <disable_collisions link1="$(arg prefix)base_link_inertia" link2="fl_caster_rotation_link" reason="Never"/>
+    <disable_collisions link1="$(arg prefix)base_link_inertia" link2="fl_caster_wheel_link" reason="Never"/>
+    <disable_collisions link1="$(arg prefix)base_link_inertia" link2="fr_caster_rotation_link" reason="Never"/>
+    <disable_collisions link1="$(arg prefix)base_link_inertia" link2="fr_caster_wheel_link" reason="Never"/>
+    <disable_collisions link1="$(arg prefix)base_link_inertia" link2="front_laser_link" reason="Never"/>
+    <disable_collisions link1="$(arg prefix)base_link_inertia" link2="left_wheel_link" reason="Never"/>
+    <disable_collisions link1="$(arg prefix)base_link_inertia" link2="right_wheel_link" reason="Never"/>
+    <disable_collisions link1="$(arg prefix)forearm_link" link2="$(arg prefix)upper_arm_link" reason="Adjacent"/>
+    <disable_collisions link1="$(arg prefix)forearm_link" link2="$(arg prefix)wrist_1_link" reason="Adjacent"/>
+    <disable_collisions link1="$(arg prefix)shoulder_link" link2="$(arg prefix)upper_arm_link" reason="Adjacent"/>
+    <disable_collisions link1="$(arg prefix)shoulder_link" link2="$(arg prefix)wrist_1_link" reason="Never"/>
+    <disable_collisions link1="$(arg prefix)shoulder_link" link2="back_laser_link" reason="Never"/>
+    <disable_collisions link1="$(arg prefix)shoulder_link" link2="base_link" reason="Never"/>
+    <disable_collisions link1="$(arg prefix)shoulder_link" link2="bl_caster_rotation_link" reason="Never"/>
+    <disable_collisions link1="$(arg prefix)shoulder_link" link2="bl_caster_wheel_link" reason="Never"/>
+    <disable_collisions link1="$(arg prefix)shoulder_link" link2="br_caster_rotation_link" reason="Never"/>
+    <disable_collisions link1="$(arg prefix)shoulder_link" link2="br_caster_wheel_link" reason="Never"/>
+    <disable_collisions link1="$(arg prefix)shoulder_link" link2="camera_link" reason="Never"/>
+    <disable_collisions link1="$(arg prefix)shoulder_link" link2="fl_caster_rotation_link" reason="Never"/>
+    <disable_collisions link1="$(arg prefix)shoulder_link" link2="fl_caster_wheel_link" reason="Never"/>
+    <disable_collisions link1="$(arg prefix)shoulder_link" link2="fr_caster_rotation_link" reason="Never"/>
+    <disable_collisions link1="$(arg prefix)shoulder_link" link2="fr_caster_wheel_link" reason="Never"/>
+    <disable_collisions link1="$(arg prefix)shoulder_link" link2="front_laser_link" reason="Never"/>
+    <disable_collisions link1="$(arg prefix)shoulder_link" link2="left_wheel_link" reason="Never"/>
+    <disable_collisions link1="$(arg prefix)shoulder_link" link2="right_wheel_link" reason="Never"/>
+    <disable_collisions link1="$(arg prefix)upper_arm_link" link2="back_laser_link" reason="Never"/>
+    <disable_collisions link1="$(arg prefix)upper_arm_link" link2="bl_caster_rotation_link" reason="Never"/>
+    <disable_collisions link1="$(arg prefix)upper_arm_link" link2="bl_caster_wheel_link" reason="Never"/>
+    <disable_collisions link1="$(arg prefix)upper_arm_link" link2="br_caster_rotation_link" reason="Never"/>
+    <disable_collisions link1="$(arg prefix)upper_arm_link" link2="br_caster_wheel_link" reason="Never"/>
+    <disable_collisions link1="$(arg prefix)wrist_1_link" link2="$(arg prefix)wrist_2_link" reason="Adjacent"/>
+    <disable_collisions link1="$(arg prefix)wrist_1_link" link2="$(arg prefix)wrist_3_link" reason="Never"/>
+    <disable_collisions link1="$(arg prefix)wrist_2_link" link2="$(arg prefix)wrist_3_link" reason="Adjacent"/>
     <disable_collisions link1="back_laser_link" link2="base_link" reason="Adjacent"/>
     <disable_collisions link1="back_laser_link" link2="bl_caster_rotation_link" reason="Never"/>

Commit message: fixed moveit get_jacobian issue

File: mur/mur_moveit_config/config/mur.srdf.xacro (robot description, xacro)
@@ -13,5 +13,4 @@
     <!--SUBGROUPS: Groups can also be formed by referencing to already defined group names-->
     <group name="UR_arm">
-        <joint name="$(arg prefix)base_link-base_fixed_joint"/>
         <joint name="$(arg prefix)base_link-base_link_inertia"/>
         <joint name="$(arg prefix)shoulder_pan_joint"/>
@@ -24,4 +23,13 @@
         <joint name="$(arg prefix)flange-tool0"/>
     </group>
+    <!--PASSIVE JOINT: Purpose: this element is used to mark joints that are not actuated-->
+    <passive_joint name="bl_caster_rotation_joint" />
+    <passive_joint name="bl_caster_wheel_joint" />
+    <passive_joint name="br_caster_rotation_joint" />
+    <passive_joint name="br_caster_wheel_joint" />
+    <passive_joint name="fl_caster_rotation_joint" />
+    <passive_joint name="fl_caster_wheel_joint" />
+    <passive_joint name="fr_caster_rotation_joint" />
+    <passive_joint name="fr_caster_wheel_joint" />
     <!--GROUP STATES: Purpose: Define a named state for a particular group, in terms of joint values. This is useful to define states like 'folded arms'-->
     <group_state name="Home_custom" group="UR_arm">
