Commit message: added group to control both arms simultaniously

File: mur/mur_moveit_config/config/mur620.srdf.xacro (robot description, xacro)
@@ -24,4 +24,24 @@
     </group>
 	<group name="UR_arm_r">
+        <joint name="$(arg prefix)_r/base_link-base_link_inertia"/>
+        <joint name="$(arg prefix)_r/shoulder_pan_joint"/>
+        <joint name="$(arg prefix)_r/shoulder_lift_joint"/>
+        <joint name="$(arg prefix)_r/elbow_joint"/>
+        <joint name="$(arg prefix)_r/wrist_1_joint"/>
+        <joint name="$(arg prefix)_r/wrist_2_joint"/>
+        <joint name="$(arg prefix)_r/wrist_3_joint"/>
+        <joint name="$(arg prefix)_r/wrist_3-flange"/>
+        <joint name="$(arg prefix)_r/flange-tool0"/>
+    </group>
+	<group name="UR_arm_both">
+		<joint name="$(arg prefix)_l/base_link-base_link_inertia"/>
+        <joint name="$(arg prefix)_l/shoulder_pan_joint"/>
+        <joint name="$(arg prefix)_l/shoulder_lift_joint"/>
+        <joint name="$(arg prefix)_l/elbow_joint"/>
+        <joint name="$(arg prefix)_l/wrist_1_joint"/>
+        <joint name="$(arg prefix)_l/wrist_2_joint"/>
+        <joint name="$(arg prefix)_l/wrist_3_joint"/>
+        <joint name="$(arg prefix)_l/wrist_3-flange"/>
+        <joint name="$(arg prefix)_l/flange-tool0"/>
         <joint name="$(arg prefix)_r/base_link-base_link_inertia"/>
         <joint name="$(arg prefix)_r/shoulder_pan_joint"/>
@@ -60,7 +80,23 @@
         <joint name="$(arg prefix)_r/wrist_3_joint" value="0"/>
     </group_state>
+	<group_state name="home" group="UR_arm_both">
+        <joint name="$(arg prefix)_l/elbow_joint" value="1.6141"/>
+        <joint name="$(arg prefix)_l/shoulder_lift_joint" value="-1.5621"/>
+        <joint name="$(arg prefix)_l/shoulder_pan_joint" value="-0.0347"/>
+        <joint name="$(arg prefix)_l/wrist_1_joint" value="-1.7009"/>
+        <joint name="$(arg prefix)_l/wrist_2_joint" value="-1.5621"/>
+        <joint name="$(arg prefix)_l/wrist_3_joint" value="0"/>
+        <joint name="$(arg prefix)_r/elbow_joint" value="1.6141"/>
+        <joint name="$(arg prefix)_r/shoulder_lift_joint" value="-1.5621"/>
+        <joint name="$(arg prefix)_r/shoulder_pan_joint" value="-0.0347"/>
+        <joint name="$(arg prefix)_r/wrist_1_joint" value="-1.7009"/>
+        <joint name="$(arg prefix)_r/wrist_2_joint" value="-1.5621"/>
+        <joint name="$(arg prefix)_r/wrist_3_joint" value="0"/>
+    </group_state>
     <!--END EFFECTOR: Purpose: Represent information about an end effector.-->
     <end_effector name="hand_l" parent_link="$(arg prefix)_l/tool0" group="UR_arm_l"/>
 	<end_effector name="hand_r" parent_link="$(arg prefix)_r/tool0" group="UR_arm_r"/>
+	<end_effector name="hand_l_both" parent_link="$(arg prefix)_l/tool0" group="UR_arm_both"/>
+	<end_effector name="hand_r_both" parent_link="$(arg prefix)_r/tool0" group="UR_arm_both"/>
     <!--DISABLE COLLISIONS: By default it is assumed that any link of the robot could potentially come into collision with any other link in the robot. This tag disables collision checking between a specified pair of links. -->
 	<disable_collisions link1="$(arg prefix)_l/base_link_inertia" link2="$(arg prefix)_l/shoulder_link" reason="Adjacent"/>

Commit message: added lift controller to moveit

File: mur/mur_moveit_config/config/mur620.srdf.xacro (robot description, xacro)
@@ -45,4 +45,50 @@
         <joint name="$(arg prefix)_l/flange-tool0"/>
         <joint name="$(arg prefix)_r/base_link-base_link_inertia"/>
+        <joint name="$(arg prefix)_r/shoulder_pan_joint"/>
+        <joint name="$(arg prefix)_r/shoulder_lift_joint"/>
+        <joint name="$(arg prefix)_r/elbow_joint"/>
+        <joint name="$(arg prefix)_r/wrist_1_joint"/>
+        <joint name="$(arg prefix)_r/wrist_2_joint"/>
+        <joint name="$(arg prefix)_r/wrist_3_joint"/>
+        <joint name="$(arg prefix)_r/wrist_3-flange"/>
+        <joint name="$(arg prefix)_r/flange-tool0"/>
+    </group>
+	<group name="UR_arm_lift_l">
+		<joint name="left_lift_joint"/>
+		<joint name="$(arg prefix)_l/base_link-base_link_inertia"/>
+        <joint name="$(arg prefix)_l/shoulder_pan_joint"/>
+        <joint name="$(arg prefix)_l/shoulder_lift_joint"/>
+        <joint name="$(arg prefix)_l/elbow_joint"/>
+        <joint name="$(arg prefix)_l/wrist_1_joint"/>
+        <joint name="$(arg prefix)_l/wrist_2_joint"/>
+        <joint name="$(arg prefix)_l/wrist_3_joint"/>
+        <joint name="$(arg prefix)_l/wrist_3-flange"/>
+        <joint name="$(arg prefix)_l/flange-tool0"/>
+    </group>
+	<group name="UR_arm_lift_r">
+		<joint name="right_lift_joint"/>
+        <joint name="$(arg prefix)_r/base_link-base_link_inertia"/>
+        <joint name="$(arg prefix)_r/shoulder_pan_joint"/>
+        <joint name="$(arg prefix)_r/shoulder_lift_joint"/>
+        <joint name="$(arg prefix)_r/elbow_joint"/>
+        <joint name="$(arg prefix)_r/wrist_1_joint"/>
+        <joint name="$(arg prefix)_r/wrist_2_joint"/>
+        <joint name="$(arg prefix)_r/wrist_3_joint"/>
+        <joint name="$(arg prefix)_r/wrist_3-flange"/>
+        <joint name="$(arg prefix)_r/flange-tool0"/>
+    </group>
+	<group name="UR_arm_all">
+		<joint name="left_lift_joint"/>
+		<joint name="$(arg prefix)_l/base_link-base_link_inertia"/>
+        <joint name="$(arg prefix)_l/shoulder_pan_joint"/>
+        <joint name="$(arg prefix)_l/shoulder_lift_joint"/>
+        <joint name="$(arg prefix)_l/elbow_joint"/>
+        <joint name="$(arg prefix)_l/wrist_1_joint"/>
+        <joint name="$(arg prefix)_l/wrist_2_joint"/>
+        <joint name="$(arg prefix)_l/wrist_3_joint"/>
+        <joint name="$(arg prefix)_l/wrist_3-flange"/>
+        <joint name="$(arg prefix)_l/flange-tool0"/>
+        <joint name="right_lift_joint"/>
+		<joint name="$(arg prefix)_r/base_link-base_link_inertia"/>
         <joint name="$(arg prefix)_r/shoulder_pan_joint"/>
         <joint name="$(arg prefix)_r/shoulder_lift_joint"/>

Commit message: changed home pose

File: mur/mur_moveit_config/config/mur620.srdf.xacro (robot description, xacro)
@@ -129,5 +129,5 @@
         <joint name="$(arg prefix)_l/elbow_joint" value="1.6141"/>
         <joint name="$(arg prefix)_l/shoulder_lift_joint" value="-1.5621"/>
-        <joint name="$(arg prefix)_l/shoulder_pan_joint" value="-0.0347"/>
+        <joint name="$(arg prefix)_l/shoulder_pan_joint" value="3.14"/>
         <joint name="$(arg prefix)_l/wrist_1_joint" value="-1.7009"/>
         <joint name="$(arg prefix)_l/wrist_2_joint" value="-1.5621"/>

Commit message: added move_UR_to_home

File: mur/mur_moveit_config/config/mur620.srdf.xacro (robot description, xacro)
@@ -111,5 +111,5 @@
     <!--GROUP STATES: Purpose: Define a named state for a particular group, in terms of joint values. This is useful to define states like 'folded arms'-->
     <group_state name="Home_custom" group="UR_arm_l">
-        <joint name="$(arg prefix)_l/elbow_joint" value="1.6141"/>
+        <joint name="$(arg prefix)_l/elbow_joint" value="-1.6141"/>
         <joint name="$(arg prefix)_l/shoulder_lift_joint" value="-1.5621"/>
         <joint name="$(arg prefix)_l/shoulder_pan_joint" value="-0.0347"/>

Commit message: changed default pose fixed move_UR_to_home

File: mur/mur_moveit_config/config/mur620.srdf.xacro (robot description, xacro)
@@ -111,9 +111,9 @@
     <!--GROUP STATES: Purpose: Define a named state for a particular group, in terms of joint values. This is useful to define states like 'folded arms'-->
     <group_state name="Home_custom" group="UR_arm_l">
-        <joint name="$(arg prefix)_l/elbow_joint" value="-1.6141"/>
-        <joint name="$(arg prefix)_l/shoulder_lift_joint" value="-1.5621"/>
-        <joint name="$(arg prefix)_l/shoulder_pan_joint" value="-0.0347"/>
-        <joint name="$(arg prefix)_l/wrist_1_joint" value="-1.7009"/>
-        <joint name="$(arg prefix)_l/wrist_2_joint" value="-1.5621"/>
+        <joint name="$(arg prefix)_l/elbow_joint" value="-1.57079632679 "/>
+        <joint name="$(arg prefix)_l/shoulder_lift_joint" value="-1.57079632679 "/>
+        <joint name="$(arg prefix)_l/shoulder_pan_joint" value="-0.0"/>
+        <joint name="$(arg prefix)_l/wrist_1_joint" value="-1.57079632679 "/>
+        <joint name="$(arg prefix)_l/wrist_2_joint" value="1.57079632679 "/>
         <joint name="$(arg prefix)_l/wrist_3_joint" value="0"/>
     </group_state>

Commit message: added global tcp pose publisher for right ur

File: mur/mur_moveit_config/config/mur620.srdf.xacro (robot description, xacro)
@@ -119,9 +119,9 @@
     </group_state>
 	<group_state name="Home_custom" group="UR_arm_r">
-        <joint name="$(arg prefix)_r/elbow_joint" value="1.6141"/>
-        <joint name="$(arg prefix)_r/shoulder_lift_joint" value="-1.5621"/>
-        <joint name="$(arg prefix)_r/shoulder_pan_joint" value="-0.0347"/>
-        <joint name="$(arg prefix)_r/wrist_1_joint" value="-1.7009"/>
-        <joint name="$(arg prefix)_r/wrist_2_joint" value="-1.5621"/>
+        <joint name="$(arg prefix)_r/elbow_joint" value="1.57079632679"/>
+        <joint name="$(arg prefix)_r/shoulder_lift_joint" value="-1.57079632679"/>
+        <joint name="$(arg prefix)_r/shoulder_pan_joint" value="-0.0"/>
+        <joint name="$(arg prefix)_r/wrist_1_joint" value="-1.57079632679"/>
+        <joint name="$(arg prefix)_r/wrist_2_joint" value="-1.57079632679"/>
         <joint name="$(arg prefix)_r/wrist_3_joint" value="0"/>
     </group_state>

Commit message: improved UR enable added dual arm collision avoidance

File: mur/mur_moveit_config/config/mur620.srdf.xacro (robot description, xacro)
@@ -124,4 +124,20 @@
         <joint name="$(arg prefix)_r/wrist_1_joint" value="-1.57079632679"/>
         <joint name="$(arg prefix)_r/wrist_2_joint" value="-1.57079632679"/>
+        <joint name="$(arg prefix)_r/wrist_3_joint" value="0"/>
+    </group_state>
+    <group_state name="handling_position" group="UR_arm_l">
+        <joint name="$(arg prefix)_l/elbow_joint" value="1.57079632679 "/>
+        <joint name="$(arg prefix)_l/shoulder_lift_joint" value="-1.57079632679 "/>
+        <joint name="$(arg prefix)_l/shoulder_pan_joint" value="-0.0"/>
+        <joint name="$(arg prefix)_l/wrist_1_joint" value="-1.57079632679 "/>
+        <joint name="$(arg prefix)_l/wrist_2_joint" value="-1.57079632679 "/>
+        <joint name="$(arg prefix)_l/wrist_3_joint" value="0"/>
+    </group_state>
+    <group_state name="handling_position" group="UR_arm_r">
+        <joint name="$(arg prefix)_r/elbow_joint" value="-1.57079632679"/>
+        <joint name="$(arg prefix)_r/shoulder_lift_joint" value="-1.57079632679"/>
+        <joint name="$(arg prefix)_r/shoulder_pan_joint" value="-0.0"/>
+        <joint name="$(arg prefix)_r/wrist_1_joint" value="-1.57079632679"/>
+        <joint name="$(arg prefix)_r/wrist_2_joint" value="1.57079632679"/>
         <joint name="$(arg prefix)_r/wrist_3_joint" value="0"/>
     </group_state>

Commit message: added calibration params

File: mur/mur_moveit_config/config/mur620.srdf.xacro (robot description, xacro)
@@ -126,5 +126,5 @@
         <joint name="$(arg prefix)_r/wrist_3_joint" value="0"/>
     </group_state>
-    <group_state name="handling_position" group="UR_arm_l">
+    <group_state name="handling_position_wide" group="UR_arm_l">
         <joint name="$(arg prefix)_l/elbow_joint" value="1.57079632679 "/>
         <joint name="$(arg prefix)_l/shoulder_lift_joint" value="-1.57079632679 "/>
@@ -134,8 +134,56 @@
         <joint name="$(arg prefix)_l/wrist_3_joint" value="0"/>
     </group_state>
-    <group_state name="handling_position" group="UR_arm_r">
+    <group_state name="handling_position_wide" group="UR_arm_r">
         <joint name="$(arg prefix)_r/elbow_joint" value="-1.57079632679"/>
         <joint name="$(arg prefix)_r/shoulder_lift_joint" value="-1.57079632679"/>
         <joint name="$(arg prefix)_r/shoulder_pan_joint" value="-0.0"/>
+        <joint name="$(arg prefix)_r/wrist_1_joint" value="-1.57079632679"/>
+        <joint name="$(arg prefix)_r/wrist_2_joint" value="1.57079632679"/>
+        <joint name="$(arg prefix)_r/wrist_3_joint" value="0"/>
+    </group_state>
+    <group_state name="handling_position_narrow" group="UR_arm_l">
+        <joint name="$(arg prefix)_l/elbow_joint" value="-1.57079632679 "/>
+        <joint name="$(arg prefix)_l/shoulder_lift_joint" value="-1.57079632679 "/>
+        <joint name="$(arg prefix)_l/shoulder_pan_joint" value="3.14159265359 "/>
+        <joint name="$(arg prefix)_l/wrist_1_joint" value="-1.57079632679 "/>
+        <joint name="$(arg prefix)_l/wrist_2_joint" value="1.57079632679 "/>
+        <joint name="$(arg prefix)_l/wrist_3_joint" value="0"/>
+    </group_state>
+    <group_state name="handling_position_narrow" group="UR_arm_r">
+        <joint name="$(arg prefix)_r/elbow_joint" value="1.57079632679"/>
+        <joint name="$(arg prefix)_r/shoulder_lift_joint" value="-1.57079632679"/>
+        <joint name="$(arg prefix)_r/shoulder_pan_joint" value="3.14159265359 "/>
+        <joint name="$(arg prefix)_r/wrist_1_joint" value="-1.57079632679"/>
+        <joint name="$(arg prefix)_r/wrist_2_joint" value="-1.57079632679"/>
+        <joint name="$(arg prefix)_r/wrist_3_joint" value="0"/>
+    </group_state>
+    <group_state name="handling_position_narrow_lift" group="UR_arm_l">
+        <joint name="$(arg prefix)_l/elbow_joint" value="-1.57079632679 "/>
+        <joint name="$(arg prefix)_l/shoulder_lift_joint" value="-1.57079632679 "/>
+        <joint name="$(arg prefix)_l/shoulder_pan_joint" value="3.378002286996061"/>
+        <joint name="$(arg prefix)_l/wrist_1_joint" value="-1.57079632679 "/>
+        <joint name="$(arg prefix)_l/wrist_2_joint" value="1.57079632679 "/>
+        <joint name="$(arg prefix)_l/wrist_3_joint" value="0"/>
+    </group_state>
+    <group_state name="handling_position_narrow_lift" group="UR_arm_r">
+        <joint name="$(arg prefix)_r/elbow_joint" value="1.57079632679"/>
+        <joint name="$(arg prefix)_r/shoulder_lift_joint" value="-1.57079632679"/>
+        <joint name="$(arg prefix)_r/shoulder_pan_joint" value="3.378002286996061 "/>
+        <joint name="$(arg prefix)_r/wrist_1_joint" value="-1.57079632679"/>
+        <joint name="$(arg prefix)_r/wrist_2_joint" value="-1.57079632679"/>
+        <joint name="$(arg prefix)_r/wrist_3_joint" value="0"/>
+    </group_state>
+    <group_state name="handling_position_wide_lift" group="UR_arm_l">
+        <joint name="$(arg prefix)_l/elbow_joint" value="1.57079632679 "/>
+        <joint name="$(arg prefix)_l/shoulder_lift_joint" value="-1.57079632679 "/>
+        <joint name="$(arg prefix)_l/shoulder_pan_joint" value="0.23640963340626803"/>
+        <joint name="$(arg prefix)_l/wrist_1_joint" value="-1.57079632679 "/>
+        <joint name="$(arg prefix)_l/wrist_2_joint" value="-1.57079632679 "/>
+        <joint name="$(arg prefix)_l/wrist_3_joint" value="0"/>
+    </group_state>
+    <group_state name="handling_position_wide_lift" group="UR_arm_r">
+        <joint name="$(arg prefix)_r/elbow_joint" value="-1.57079632679"/>
+        <joint name="$(arg prefix)_r/shoulder_lift_joint" value="-1.57079632679"/>
+        <joint name="$(arg prefix)_r/shoulder_pan_joint" value="0.23640963340626803"/>
         <joint name="$(arg prefix)_r/wrist_1_joint" value="-1.57079632679"/>
         <joint name="$(arg prefix)_r/wrist_2_joint" value="1.57079632679"/>

Commit message: Enhance teleoperation configuration and add custom home state
- Introduced a new group state `Home_custom_teleop` in `mur620.srdf.xacro` for the right arm, providing a predefined pose for teleoperation.
- Adjusted force and torque reflection scales in `master_real_mur620b_ur10_l.yaml` to improve feedback responsiveness.
- Increased the force deadband in `slave_real_mur620b_ur10_r.yaml` for enhanced stability during operation.
- Updated launch file `master_slave_mur620b_real.launch` to clarify the base frame parameters for the slave arm.

File: mur/mur_moveit_config/config/mur620.srdf.xacro (robot description, xacro)
@@ -126,4 +126,12 @@
         <joint name="$(arg prefix)_r/wrist_1_joint" value="-1.57079632679"/>
         <joint name="$(arg prefix)_r/wrist_2_joint" value="-1.57079632679"/>
+        <joint name="$(arg prefix)_r/wrist_3_joint" value="0"/>
+    </group_state>
+    <group_state name="Home_custom_teleop" group="UR_arm_r">
+        <joint name="$(arg prefix)_r/elbow_joint" value="-1.57079632679 "/>
+        <joint name="$(arg prefix)_r/shoulder_lift_joint" value="-1.57079632679 "/>
+        <joint name="$(arg prefix)_r/shoulder_pan_joint" value="-0.0"/>
+        <joint name="$(arg prefix)_r/wrist_1_joint" value="-1.57079632679 "/>
+        <joint name="$(arg prefix)_r/wrist_2_joint" value="1.57079632679 "/>
         <joint name="$(arg prefix)_r/wrist_3_joint" value="0"/>
     </group_state>

Commit message: Aggiunta posa Aggiunto esponente per modificarte funzione di variazione della massa e dello smorzamento

File: mur/mur_moveit_config/config/mur620.srdf.xacro (robot description, xacro)
@@ -118,4 +118,12 @@
         <joint name="$(arg prefix)_l/wrist_1_joint" value="-1.57079632679 "/>
         <joint name="$(arg prefix)_l/wrist_2_joint" value="1.57079632679 "/>
+        <joint name="$(arg prefix)_l/wrist_3_joint" value="0"/>
+    </group_state>
+    <group_state name="Home_custom_teleop" group="UR_arm_l">
+        <joint name="$(arg prefix)_l/elbow_joint" value="1.57079632679"/>
+        <joint name="$(arg prefix)_l/shoulder_lift_joint" value="-1.57079632679"/>
+        <joint name="$(arg prefix)_l/shoulder_pan_joint" value="-0.0"/>
+        <joint name="$(arg prefix)_l/wrist_1_joint" value="-1.57079632679"/>
+        <joint name="$(arg prefix)_l/wrist_2_joint" value="-1.57079632679"/>
         <joint name="$(arg prefix)_l/wrist_3_joint" value="0"/>
     </group_state>

Commit message: Aggiunta rotazione su asse z a causa del diverso montaggio dei robot

File: mur/mur_moveit_config/config/mur620.srdf.xacro (robot description, xacro)
@@ -128,4 +128,12 @@
         <joint name="$(arg prefix)_l/wrist_3_joint" value="0"/>
     </group_state>
+    <group_state name="home_custom_teleop_slave" group="UR_arm_l">
+        <joint name="$(arg prefix)_l/elbow_joint" value="1.57079632679"/>
+        <joint name="$(arg prefix)_l/shoulder_lift_joint" value="-1.57079632679"/>
+        <joint name="$(arg prefix)_l/shoulder_pan_joint" value="0.2305469980736988"/>
+        <joint name="$(arg prefix)_l/wrist_1_joint" value="-1.57079632679"/>
+        <joint name="$(arg prefix)_l/wrist_2_joint" value="-1.57079632679"/>
+        <joint name="$(arg prefix)_l/wrist_3_joint" value="0"/>
+    </group_state>
 	<group_state name="Home_custom" group="UR_arm_r">
         <joint name="$(arg prefix)_r/elbow_joint" value="1.57079632679"/>
@@ -140,4 +148,12 @@
         <joint name="$(arg prefix)_r/shoulder_lift_joint" value="-1.57079632679 "/>
         <joint name="$(arg prefix)_r/shoulder_pan_joint" value="-0.0"/>
+        <joint name="$(arg prefix)_r/wrist_1_joint" value="-1.57079632679 "/>
+        <joint name="$(arg prefix)_r/wrist_2_joint" value="1.57079632679 "/>
+        <joint name="$(arg prefix)_r/wrist_3_joint" value="0"/>
+    </group_state>
+    <group_state name="home_custom_teleop_slave" group="UR_arm_r">
+        <joint name="$(arg prefix)_r/elbow_joint" value="-1.57079632679 "/>
+        <joint name="$(arg prefix)_r/shoulder_lift_joint" value="-1.57079632679 "/>
+        <joint name="$(arg prefix)_r/shoulder_pan_joint" value="0.22812032433233884"/>
         <joint name="$(arg prefix)_r/wrist_1_joint" value="-1.57079632679 "/>
         <joint name="$(arg prefix)_r/wrist_2_joint" value="1.57079632679 "/>
