Commit message: Update gripper_joint origin position and rotation in URDF

File: tools/keyence_lj_x/urdf/keyence_lj_x.urdf.xacro (robot description, xacro)
@@ -9,5 +9,5 @@
 		</link>
 		<joint name="${tf_prefix}/gripper_joint" type="fixed">
-			<origin xyz="0 0 0.0" rpy="${-pi * 0.5} ${pi * 0.0} ${pi * 0.0}" />
+			<origin xyz="0.05 0 0.0" rpy="${-pi * 0.0} ${pi * 0.0} ${pi * 0.0}" />
 			<parent link="${tool_link}" />
 			<child link="${tf_prefix}/gripper" />
