Commit message: Fix joint origins and adjust visual/collision properties in bauschaum_ee URDF

File: tools/bauschaum_ee/urdf/bauschaum_ee.urdf.xacro (robot description, xacro)
@@ -9,5 +9,5 @@
 		</link>
 		<joint name="${tf_prefix}/gripper_joint" type="fixed">
-			<origin xyz="0.5 -0.13 0.0" rpy="${-pi * 0.5} ${pi * 0.0} ${pi * 0.0}" />
+			<origin xyz="0.13 0 0.50" rpy="${-pi * 0.0} ${-pi * 0.5} ${pi * 0.0}" />
 			<parent link="${tool_link}" />
 			<child link="${tf_prefix}/gripper" />
@@ -20,5 +20,5 @@
 			</xacro:cylinder_inertial>
 			<visual>
-				<origin xyz="0.0 0.0 0" rpy="0 ${pi * 0.5} ${pi * 0.0}" />
+				<origin xyz="0.01 0.0 0.0" rpy="0 ${pi * 0.5} ${pi * 0.0}" />
 				<geometry>
 					<mesh filename="package://bauschaum_ee/meshes/visual/bauschaum_ee.stl" scale="0.001 0.001 0.001"/>
@@ -27,5 +27,5 @@
 			</visual>
 			<collision>
-				<origin xyz="0.0 0.0 0" rpy="0 ${pi * 0.5} ${pi * 0.0}" />
+				<origin xyz="0.01 0.0 0.0" rpy="0 ${pi * 0.5} ${pi * 0.0}" />
 				<geometry>
 					<mesh filename="package://bauschaum_ee/meshes/collision/bauschaum_ee.stl" scale="0.001 0.001 0.001"/>
@@ -35,5 +35,5 @@
 		<!-- the ft_sensor plugin will not work with fixed joints. This is why a prismatic joint with very small limits is added -->
 		<joint name="${tf_prefix}/tcp_joint" type="prismatic">
-			<origin xyz="-0.5 0.0 0.13" rpy="0 0 0" />
+			<origin xyz="-0.50 0.0 0.13" rpy="0 0 0" />
 			<parent link="${tf_prefix}/gripper" />
 			<child link="${tf_prefix}/tcp" />

Commit message: Refactor bauschaum_ee integration: update URDF and launch files, add BMS node, and improve gripper joint definitions

File: tools/bauschaum_ee/urdf/bauschaum_ee.urdf.xacro (robot description, xacro)
@@ -9,5 +9,5 @@
 		</link>
 		<joint name="${tf_prefix}/gripper_joint" type="fixed">
-			<origin xyz="0.5 -0.13 0.0" rpy="${-pi * 0.5} ${pi * 0.0} ${pi * 0.0}" />
+			<origin xyz="0.13 0 0.50" rpy="${-pi * 0.0} ${-pi * 0.5} ${pi * 0.0}" />
 			<parent link="${tool_link}" />
 			<child link="${tf_prefix}/gripper" />
@@ -20,5 +20,5 @@
 			</xacro:cylinder_inertial>
 			<visual>
-				<origin xyz="0.0 0.0 0" rpy="0 ${pi * 0.5} ${pi * 0.0}" />
+				<origin xyz="0.01 0.0 0.0" rpy="0 ${pi * 0.5} ${pi * 0.0}" />
 				<geometry>
 					<mesh filename="package://bauschaum_ee/meshes/visual/bauschaum_ee.stl" scale="0.001 0.001 0.001"/>
@@ -26,11 +26,14 @@
 				<xacro:insert_block name="material_white" />
 			</visual>
+			<collision>
+				<origin xyz="0.01 0.0 0.0" rpy="0 ${pi * 0.5} ${pi * 0.0}" />
+				<geometry>
+					<mesh filename="package://bauschaum_ee/meshes/collision/bauschaum_ee.stl" scale="0.001 0.001 0.001"/>
+				</geometry>
+			</collision>
 		</link>
-		<gazebo reference="${tf_prefix}/tcp">
-			<material>Gazebo/DarkGrey</material>
-		</gazebo>
 		<!-- the ft_sensor plugin will not work with fixed joints. This is why a prismatic joint with very small limits is added -->
 		<joint name="${tf_prefix}/tcp_joint" type="prismatic">
-			<origin xyz="-0.5 0.0 0.13" rpy="0 0 0" />
+			<origin xyz="-0.50 0.0 0.13" rpy="0 0 0" />
 			<parent link="${tf_prefix}/gripper" />
 			<child link="${tf_prefix}/tcp" />
@@ -38,43 +41,4 @@
    			<limit effort="1000" lower="-0.0001" upper="0.0001" velocity="10"/>
 		</joint>
-		<!-- Gazebo Plugin for Line Laser -->
-		<gazebo reference="${tf_prefix}/gripper">
-			<sensor type="ray" name="line_laser">
-			<pose>0 0 0 0.0 0 0</pose>
-			<visualize>true</visualize>
-			<update_rate>20.0</update_rate>
-			<ray>
-				<scan>
-				<!-- Horizontal range parameters -->
-				<horizontal>
-					<samples>1000</samples> <!-- Number of laser beams -->
-					<resolution>1</resolution>
-					<min_angle>-0.27317277996474193</min_angle> <!-- Start angle in radians -->
-					<max_angle>0.27317277996474193</max_angle> <!-- End angle in radians -->
-				</horizontal>
-				<!-- Vertical range parameters (set min and max equal for a line) -->
-				<vertical>
-					<samples>1</samples> <!-- Single vertical beam -->
-					<min_angle>0.0</min_angle>
-					<max_angle>0.0</max_angle>
-				</vertical>
-				</scan>
-				<range>
-				<min>0.285</min> <!-- Minimum range in meters -->
-				<max>0.600</max> <!-- Maximum range in meters -->
-				<resolution>0.0001707329874779637</resolution> <!-- Range resolution -->
-				</range>
-				<noise>
-				<type>gaussian</type>
-				<mean>0.00005</mean>
-				<stddev>0.0005</stddev>
-				</noise>
-			</ray>
-			<plugin name="gazebo_ros_laser" filename="libgazebo_ros_laser.so">
-				<topicName>${tf_prefix}/line_laser/scan</topicName> <!-- ROS topic -->
-				<frameName>mur620a/${tf_prefix}/gripper</frameName> <!-- Frame for the laser -->
-			</plugin>
-			</sensor>
-		</gazebo>
 	</xacro:macro>
 </robot>

Commit message: Fix gripper_joint origin position for correct alignment

File: tools/bauschaum_ee/urdf/bauschaum_ee.urdf.xacro (robot description, xacro)
@@ -9,5 +9,5 @@
 		</link>
 		<joint name="${tf_prefix}/gripper_joint" type="fixed">
-			<origin xyz="0.13 0 0.50" rpy="${-pi * 0.0} ${-pi * 0.5} ${pi * 0.0}" />
+			<origin xyz="0.0 0.0605 0.50" rpy="${-pi * 0.0} ${-pi * 0.5} ${pi * 0.0}" />
 			<parent link="${tool_link}" />
 			<child link="${tf_prefix}/gripper" />
